File: Flash1MB/Flash1MB.kicad_pcb (KiCad board)
At the start: 2 copper layers, 102.2 x 69.2 mm, 12 parts, among them J1 Conn_02x04_Odd_Even, J2 Conn_01x01_Pin, J3 Conn_01x01_Pin, J4 Conn_01x01_Pin, J5 Conn_01x01_Pin, J6 Conn_01x01_Pin, J7 Conn_01x01_Pin, J8 Conn_01x01_Pin

Commit message: masse
Parts:
- H1, H2, H3, H4: footprint MountingHole:MountingHole_2.5mm_Pad -> MountingHole:MountingHole_2.2mm_M2_DIN965_Pad
- moved H3 0.50 mm to (200.0, 123.0)
- moved H4 0.50 mm to (104.0, 123.0)
Connections:
- J1 pad 8: Net-(J1-Pin_8) -> unconnected-(J1-Pin_8-Pad8)
Other:
- board size 102.2 x 69.2 mm -> 101.7 x 69.2 mm
Changed lines of the file:
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@@
 	(net 5 "Net-(J1-Pin_5)")
 	(net 6 "Net-(J1-Pin_7)")
-	(net 7 "Net-(J1-Pin_8)")
+	(net 7 "unconnected-(J1-Pin_8-Pad8)")
 	(net 8 "Net-(J1-Pin_2)")
 	(net 9 "unconnected-(H1-Pad1)")
@@
 		)
 	)
-	(footprint "MountingHole:MountingHole_2.5mm_Pad"
+	(footprint "MountingHole:MountingHole_2.2mm_M2_DIN965_Pad"
 		(layer "F.Cu")
-		(at 104 122.5)
-		(descr "Mounting Hole 2.5mm")
-		(tags "mounting hole 2.5mm")
+		(at 104 123)
+		(descr "Mounting Hole 2.2mm, M2, DIN965")
+		(tags "mounting hole 2.2mm m2 din965")
 		(property "Reference" "H4"
-			(at 0 -3.5 0)
+			(at 0 -2.9 0)
 			(layer "F.SilkS")
 			(effects
@@
 		)
 		(property "Value" "MountingHole_Pad"
-			(at 0 3.5 0)
-			(layer "F.Fab")
-			(effects
-				(font
-					(size 1 1)
-					(thickness 0.15)
-				)
-			)
-		)
-		(property "Footprint" "MountingHole:MountingHole_2.5mm_Pad"
+			(at 0 2.9 0)
+			(layer "F.Fab")
+			(effects
+				(font
+					(size 1 1)
+					(thickness 0.15)
+				)
+			)
+		)
+		(property "Footprint" "MountingHole:MountingHole_2.2mm_M2_DIN965_Pad"
 			(at 0 0 0)
 			(unlocked yes)
@@
 		(fp_circle
 			(center 0 0)
-			(end 2.5 0)
+			(end 1.9 0)
 			(stroke
 				(width 0.15)
@@
 		(fp_circle
 			(center 0 0)
-			(end 2.75 0)
+			(end 2.15 0)
 			(stroke
 				(width 0.05)
@@
 		(pad "1" thru_hole circle
 			(at 0 0)
-			(size 5 5)
-			(drill 2.5)
+			(size 3.8 3.8)
+			(drill 2.2)
 			(layers "*.Cu" "*.Mask")
 			(remove_unused_layers no)
@@
 			(layers "*.Cu" "*.Mask")
 			(remove_unused_layers no)
-			(net 7 "Net-(J1-Pin_8)")
+			(net 7 "unconnected-(J1-Pin_8-Pad8)")
 			(pinfunction "Pin_8")
-			(pintype "passive")
+			(pintype "passive+no_connect")
 		)
 		(model "${KICAD8_3DMODEL_DIR}/Connector_PinHeader_2.54mm.3dshapes/PinHeader_2x04_P2.54mm_Vertical.wrl"
@@
 		)
 	)
-	(footprint "MountingHole:MountingHole_2.5mm_Pad"
+	(footprint "MountingHole:MountingHole_2.2mm_M2_DIN965_Pad"
 		(layer "F.Cu")
-		(at 200 122.5)
-		(descr "Mounting Hole 2.5mm")
-		(tags "mounting hole 2.5mm")
+		(at 200 123)
+		(descr "Mounting Hole 2.2mm, M2, DIN965")
+		(tags "mounting hole 2.2mm m2 din965")
 		(property "Reference" "H3"
-			(at 0 -3.5 0)
+			(at 0 -2.9 0)
 			(layer "F.SilkS")
 			(effects
@@
 		)
 		(property "Value" "MountingHole_Pad"
-			(at 0 3.5 0)
-			(layer "F.Fab")
-			(effects
-				(font
-					(size 1 1)
-					(thickness 0.15)
-				)
-			)
-		)
-		(property "Footprint" "MountingHole:MountingHole_2.5mm_Pad"
+			(at 0 2.9 0)
+			(layer "F.Fab")
+			(effects
+				(font
+					(size 1 1)
+					(thickness 0.15)
+				)
+			)
+		)
+		(property "Footprint" "MountingHole:MountingHole_2.2mm_M2_DIN965_Pad"
 			(at 0 0 0)
 			(unlocked yes)
@@
 		(fp_circle
 			(center 0 0)
-			(end 2.5 0)
+			(end 1.9 0)
 			(stroke
 				(width 0.15)
@@
 		(fp_circle
 			(center 0 0)
-			(end 2.75 0)
+			(end 2.15 0)
 			(stroke
 				(width 0.05)
@@
 		(pad "1" thru_hole circle
 			(at 0 0)
-			(size 5 5)
-			(drill 2.5)
+			(size 3.8 3.8)
+			(drill 2.2)
 			(layers "*.Cu" "*.Mask")
 			(remove_unused_layers no)
@@
 		)
 	)
-	(footprint "MountingHole:MountingHole_2.5mm_Pad"
+	(footprint "MountingHole:MountingHole_2.2mm_M2_DIN965_Pad"
 		(layer "F.Cu")
 		(at 200 59.5)
-		(descr "Mounting Hole 2.5mm")
-		(tags "mounting hole 2.5mm")
+		(descr "Mounting Hole 2.2mm, M2, DIN965")
+		(tags "mounting hole 2.2mm m2 din965")
 		(property "Reference" "H2"
-			(at 0 -3.5 0)
+			(at 0 -2.9 0)
 			(layer "F.SilkS")
 			(effects
@@
 		)
 		(property "Value" "MountingHole_Pad"
-			(at 0 3.5 0)
-			(layer "F.Fab")
-			(effects
-				(font
-					(size 1 1)
-					(thickness 0.15)
-				)
-			)
-		)
-		(property "Footprint" "MountingHole:MountingHole_2.5mm_Pad"
+			(at 0 2.9 0)
+			(layer "F.Fab")
+			(effects
+				(font
+					(size 1 1)
+					(thickness 0.15)
+				)
+			)
+		)
+		(property "Footprint" "MountingHole:MountingHole_2.2mm_M2_DIN965_Pad"
 			(at 0 0 0)
 			(unlocked yes)
@@
 		(fp_circle
 			(center 0 0)
-			(end 2.5 0)
+			(end 1.9 0)
 			(stroke
 				(width 0.15)
@@
 		(fp_circle
 			(center 0 0)
-			(end 2.75 0)
+			(end 2.15 0)
 			(stroke
 				(width 0.05)
@@
 		(pad "1" thru_hole circle
 			(at 0 0)
-			(size 5 5)
-			(drill 2.5)
+			(size 3.8 3.8)
+			(drill 2.2)
 			(layers "*.Cu" "*.Mask")
 			(remove_unused_layers no)
@@
 		)
 	)
-	(footprint "MountingHole:MountingHole_2.5mm_Pad"
+	(footprint "MountingHole:MountingHole_2.2mm_M2_DIN965_Pad"
 		(layer "F.Cu")
 		(at 104 59.5)
-		(descr "Mounting Hole 2.5mm")
-		(tags "mounting hole 2.5mm")
+		(descr "Mounting Hole 2.2mm, M2, DIN965")
+		(tags "mounting hole 2.2mm m2 din965")
 		(property "Reference" "H1"
-			(at 0 -3.5 0)
+			(at 0 -2.9 0)
 			(layer "F.SilkS")
 			(effects
@@
 		)
 		(property "Value" "MountingHole_Pad"
-			(at 0 3.5 0)
-			(layer "F.Fab")
-			(effects
-				(font
-					(size 1 1)
-					(thickness 0.15)
-				)
-			)
-		)
-		(property "Footprint" "MountingHole:MountingHole_2.5mm_Pad"
+			(at 0 2.9 0)
+			(layer "F.Fab")
+			(effects
+				(font
+					(size 1 1)
+					(thickness 0.15)
+				)
+			)
+		)
+		(property "Footprint" "MountingHole:MountingHole_2.2mm_M2_DIN965_Pad"
 			(at 0 0 0)
 			(unlocked yes)
@@
 		(fp_circle
 			(center 0 0)
-			(end 2.5 0)
+			(end 1.9 0)
 			(stroke
 				(width 0.15)
@@
 		(fp_circle
 			(center 0 0)
-			(end 2.75 0)
+			(end 2.15 0)
 			(stroke
 				(width 0.05)
@@
 		(pad "1" thru_hole circle
 			(at 0 0)
-			(size 5 5)
-			(drill 2.5)
+			(size 3.8 3.8)
+			(drill 2.2)
 			(layers "*.Cu" "*.Mask")
 			(remove_unused_layers no)
@@
 	(gr_rect
 		(start 100.965 56.515)
-		(end 203.2 125.73)
+		(end 202.7 125.73)
 		(stroke
 			(width 0.05)

Commit message: polygon
Routing:
- added copper zone on B.Cu, net (none)
- added copper zone on F.Cu, net (none)
Changed lines of the file:
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@@
 		(net 8)
 	)
+	(zone
+		(net 0)
+		(net_name "")
+		(layers "F&B.Cu")
+		(hatch edge 0.5)
+		(connect_pads
+			(clearance 0.5)
+		)
+		(min_thickness 0.25)
+		(filled_areas_thickness no)
+		(fill yes
+			(thermal_gap 0.5)
+			(thermal_bridge_width 0.5)
+			(island_removal_mode 1)
+			(island_area_min 10)
+		)
+		(polygon
+			(pts
+				(xy 101.5 57) (xy 202 57) (xy 202 125) (xy 101.5 125)
+			)
+		)
+	)
 )
