File: Soundkarte/Soundkarte.kicad_pcb (KiCad board)
At the start: 2 copper layers, 114.9 x 67.3 mm, 6 parts, among them J1 Conn_01x09_Pin, J2 Conn_02x03_Counter_Clockwise

Commit message: masse
Parts:
- H1, H2, H3, H4: footprint MountingHole:MountingHole_3mm_Pad -> MountingHole:MountingHole_4mm_Pad
Changed lines of the file:
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@@
 		)
 	)
-	(footprint "MountingHole:MountingHole_3mm_Pad"
+	(footprint "MountingHole:MountingHole_4mm_Pad"
 		(layer "F.Cu")
 		(at 206.375 145.415 90)
-		(descr "Mounting Hole 3mm")
-		(tags "mounting hole 3mm")
+		(descr "Mounting Hole 4mm")
+		(tags "mounting hole 4mm")
 		(property "Reference" "H3"
-			(at 0 -4 90)
+			(at 0 -5 90)
 			(layer "F.SilkS")
 			(effects
@@
 		)
 		(property "Value" "MountingHole_Pad"
-			(at 0 4 90)
-			(layer "F.Fab")
-			(effects
-				(font
-					(size 1 1)
-					(thickness 0.15)
-				)
-			)
-		)
-		(property "Footprint" "MountingHole:MountingHole_3mm_Pad"
+			(at 0 5 90)
+			(layer "F.Fab")
+			(effects
+				(font
+					(size 1 1)
+					(thickness 0.15)
+				)
+			)
+		)
+		(property "Footprint" "MountingHole:MountingHole_4mm_Pad"
 			(at 0 0 90)
 			(unlocked yes)
@@
 		(fp_circle
 			(center 0 0)
-			(end 3 0)
+			(end 4 0)
 			(stroke
 				(width 0.15)
@@
 		(fp_circle
 			(center 0 0)
-			(end 3.25 0)
+			(end 4.25 0)
 			(stroke
 				(width 0.05)
@@
 		(pad "1" thru_hole circle
 			(at 0 0 90)
-			(size 6 6)
-			(drill 3)
+			(size 8 8)
+			(drill 4)
 			(layers "*.Cu" "*.Mask")
 			(remove_unused_layers no)
@@
 		)
 	)
-	(footprint "MountingHole:MountingHole_3mm_Pad"
+	(footprint "MountingHole:MountingHole_4mm_Pad"
 		(layer "F.Cu")
 		(at 100.965 87.63 90)
-		(descr "Mounting Hole 3mm")
-		(tags "mounting hole 3mm")
+		(descr "Mounting Hole 4mm")
+		(tags "mounting hole 4mm")
 		(property "Reference" "H1"
-			(at 0 -4 90)
+			(at 0 -5 90)
 			(layer "F.SilkS")
 			(effects
@@
 		)
 		(property "Value" "MountingHole_Pad"
-			(at 0 4 90)
-			(layer "F.Fab")
-			(effects
-				(font
-					(size 1 1)
-					(thickness 0.15)
-				)
-			)
-		)
-		(property "Footprint" "MountingHole:MountingHole_3mm_Pad"
+			(at 0 5 90)
+			(layer "F.Fab")
+			(effects
+				(font
+					(size 1 1)
+					(thickness 0.15)
+				)
+			)
+		)
+		(property "Footprint" "MountingHole:MountingHole_4mm_Pad"
 			(at 0 0 90)
 			(unlocked yes)
@@
 		(fp_circle
 			(center 0 0)
-			(end 3 0)
+			(end 4 0)
 			(stroke
 				(width 0.15)
@@
 		(fp_circle
 			(center 0 0)
-			(end 3.25 0)
+			(end 4.25 0)
 			(stroke
 				(width 0.05)
@@
 		(pad "1" thru_hole circle
 			(at 0 0 90)
-			(size 6 6)
-			(drill 3)
+			(size 8 8)
+			(drill 4)
 			(layers "*.Cu" "*.Mask")
 			(remove_unused_layers no)
@@
 		)
 	)
-	(footprint "MountingHole:MountingHole_3mm_Pad"
+	(footprint "MountingHole:MountingHole_4mm_Pad"
 		(layer "F.Cu")
 		(at 100.965 145.415 90)
-		(descr "Mounting Hole 3mm")
-		(tags "mounting hole 3mm")
+		(descr "Mounting Hole 4mm")
+		(tags "mounting hole 4mm")
 		(property "Reference" "H4"
-			(at 0 -4 90)
+			(at 0 -5 90)
 			(layer "F.SilkS")
 			(effects
@@
 		)
 		(property "Value" "MountingHole_Pad"
-			(at 0 4 90)
-			(layer "F.Fab")
-			(effects
-				(font
-					(size 1 1)
-					(thickness 0.15)
-				)
-			)
-		)
-		(property "Footprint" "MountingHole:MountingHole_3mm_Pad"
+			(at 0 5 90)
+			(layer "F.Fab")
+			(effects
+				(font
+					(size 1 1)
+					(thickness 0.15)
+				)
+			)
+		)
+		(property "Footprint" "MountingHole:MountingHole_4mm_Pad"
 			(at 0 0 90)
 			(unlocked yes)
@@
 		(fp_circle
 			(center 0 0)
-			(end 3 0)
+			(end 4 0)
 			(stroke
 				(width 0.15)
@@
 		(fp_circle
 			(center 0 0)
-			(end 3.25 0)
+			(end 4.25 0)
 			(stroke
 				(width 0.05)
@@
 		(pad "1" thru_hole circle
 			(at 0 0 90)
-			(size 6 6)
-			(drill 3)
+			(size 8 8)
+			(drill 4)
 			(layers "*.Cu" "*.Mask")
 			(remove_unused_layers no)
@@
 		)
 	)
-	(footprint "MountingHole:MountingHole_3mm_Pad"
+	(footprint "MountingHole:MountingHole_4mm_Pad"
 		(layer "F.Cu")
 		(at 206.375 86.995 90)
-		(descr "Mounting Hole 3mm")
-		(tags "mounting hole 3mm")
+		(descr "Mounting Hole 4mm")
+		(tags "mounting hole 4mm")
 		(property "Reference" "H2"
-			(at 0 -4 90)
+			(at 0 -5 90)
 			(layer "F.SilkS")
 			(effects
@@
 		)
 		(property "Value" "MountingHole_Pad"
-			(at 0 4 90)
-			(layer "F.Fab")
-			(effects
-				(font
-					(size 1 1)
-					(thickness 0.15)
-				)
-			)
-		)
-		(property "Footprint" "MountingHole:MountingHole_3mm_Pad"
+			(at 0 5 90)
+			(layer "F.Fab")
+			(effects
+				(font
+					(size 1 1)
+					(thickness 0.15)
+				)
+			)
+		)
+		(property "Footprint" "MountingHole:MountingHole_4mm_Pad"
 			(at 0 0 90)
 			(unlocked yes)
@@
 		(fp_circle
 			(center 0 0)
-			(end 3 0)
+			(end 4 0)
 			(stroke
 				(width 0.15)
@@
 		(fp_circle
 			(center 0 0)
-			(end 3.25 0)
+			(end 4.25 0)
 			(stroke
 				(width 0.05)
@@
 		(pad "1" thru_hole circle
 			(at 0 0 90)
-			(size 6 6)
-			(drill 3)
+			(size 8 8)
+			(drill 4)
 			(layers "*.Cu" "*.Mask")
 			(remove_unused_layers no)
