File: SoundkartenProg/SoundkartenProg.kicad_sch (KiCad schematic)
At the start: 5 parts, among them J1 TTL, J2 Soundkarte, J3 Messgerät, J4 12-16V, U1 74HC14

Commit message: kicad10
Parts:
- J3: value Messgerät -> 12V
- J4: value 12-16V -> Messgerät
Other:
- moved on the sheet: U1A, U1B
