File: LPTastatur/LPTastatur.kicad_pcb (KiCad board)
At the start: 2 copper layers, 84 x 54 mm, 23 parts, among them J1 Conn_01x04, Q1 BC556, SW1 SW_Push_Dual, SW2 SW_Push_Dual, SW3 SW_Push_Dual, U1 L7805, U2 NE555P

Commit message: upsi
Parts:
- moved R7 1.00 mm to (122.0, 85.0)
- moved SW1 0.50 mm to (99.5, 65.0)
- moved SW3 0.50 mm to (151.5, 65.0)
Connections:
- R7 pad 2: VCC -> Net-(D1-K)
Routing:
- net Net-(D1-K): track 38.7 -> 40.1 mm
- net VCC: track 109.3 -> 110.3 mm
- net Net-(U2-R): track 23.7 -> 24.7 mm
- net Net-(D3-A): track 15.5 -> 16.0 mm
- net Net-(D1-A): track 8.07 -> 8.57 mm
Changed lines of the file:
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@@
 		)
 		(fp_text user "K"
-			(at 0 -1.9 90)
+			(at -1.34 0 90)
 			(layer "F.SilkS")
 			(effects
@@
 		(tags "THT DIP DIL PDIP 2.54mm 7.62mm 300mil")
 		(property "Reference" "U2"
-			(at 3.81 -2.33 0)
+			(at 3.5 10.5 0)
 			(layer "F.SilkS")
 			(effects
@@
 	(footprint "Button_Switch_THT:Push_E-Switch_KS01Q01"
 		(layer "F.Cu")
-		(at 151 65)
+		(at 151.5 65)
 		(descr "E-Switch KS01Q01 http://spec_sheets.e-switch.com/specs/29-KS01Q01.pdf")
 		(tags "Push Button")
@@
 		(tags "Resistor Axial_DIN0207 series Axial Horizontal pin pitch 10.16mm 0.25W = 1/4W length 6.3mm diameter 2.5mm")
 		(property "Reference" "R3"
-			(at 5.08 -2.37 0)
+			(at 10 -2.37 0)
 			(layer "F.SilkS")
 			(effects
@@
 	(footprint "Button_Switch_THT:Push_E-Switch_KS01Q01"
 		(layer "F.Cu")
-		(at 100 65)
+		(at 99.5 65)
 		(descr "E-Switch KS01Q01 http://spec_sheets.e-switch.com/specs/29-KS01Q01.pdf")
 		(tags "Push Button")
@@
 		)
 		(fp_text user "K"
-			(at 0 -1.9 90)
+			(at 0 2 90)
 			(layer "F.SilkS")
 			(effects
@@
 	(footprint "Resistor_THT:R_Axial_DIN0207_L6.3mm_D2.5mm_P10.16mm_Horizontal"
 		(layer "F.Cu")
-		(at 122 86 90)
+		(at 122 85 90)
 		(descr "Resistor, Axial_DIN0207 series, Axial, Horizontal, pin pitch=10.16mm, 0.25W = 1/4W, length*diameter=6.3*2.5mm^2, http://cdn-reichelt.de/documents/datenblatt/B400/1_4W%23YAG.pdf")
 		(tags "Resistor Axial_DIN0207 series Axial Horizontal pin pitch 10.16mm 0.25W = 1/4W length 6.3mm diameter 2.5mm")
@@
 			(layers "*.Cu" "*.Mask")
 			(remove_unused_layers no)
-			(net 8 "VCC")
+			(net 14 "Net-(D1-K)")
 			(pintype "passive")
 		)
@@
 		)
 		(fp_text user "K"
-			(at 0 -1.9 90)
+			(at -1.34 0 90)
 			(layer "F.SilkS")
 			(effects
@@
 		)
 	)
+	(dimension
+		(type aligned)
+		(layer "User.1")
+		(pts
+			(xy 87 54) (xy 171 54)
+		)
+		(height -7.2)
+		(gr_text "84,0000 mm"
+			(at 129 45.65 0)
+			(layer "User.1")
+			(effects
+				(font
+					(size 1 1)
+					(thickness 0.15)
+				)
+			)
+		)
+		(format
+			(prefix "")
+			(suffix "")
+			(units 3)
+			(units_format 1)
+			(precision 4)
+		)
+		(style
+			(thickness 0.1)
+			(arrow_length 1.27)
+			(text_position_mode 0)
+			(extension_height 0.58642)
+			(extension_offset 0.5) keep_text_aligned)
+	)
+	(dimension
+		(type aligned)
+		(layer "User.1")
+		(pts
+			(xy 171 108) (xy 171 54)
+		)
+		(height 7.1)
+		(gr_text "54,0000 mm"
+			(at 176.95 81 90)
+			(layer "User.1")
+			(effects
+				(font
+					(size 1 1)
+					(thickness 0.15)
+				)
+			)
+		)
+		(format
+			(prefix "")
+			(suffix "")
+			(units 3)
+			(units_format 1)
+			(precision 4)
+		)
+		(style
+			(thickness 0.1)
+			(arrow_length 1.27)
+			(text_position_mode 0)
+			(extension_height 0.58642)
+			(extension_offset 0.5) keep_text_aligned)
+	)
 	(segment
 		(start 117 92)
@@
 	)
 	(segment
-		(start 148 68)
-		(end 151 65)
+		(start 128 68)
+		(end 148 68)
+		(width 1)
+		(layer "B.Cu")
+		(net 8)
+	)
+	(segment
+		(start 125 65)
+		(end 128 68)
 		(width 1)
 		(layer "B.Cu")
@@
 	)
 	(segment
+		(start 148 68)
+		(end 151 65)
+		(width 1)
+		(layer "B.Cu")
+		(net 8)
+	)
+	(segment
 		(start 100 65)
 		(end 102 67)
@@
 	)
 	(segment
+		(start 99.5 65)
+		(end 100 65)
+		(width 1)
+		(layer "B.Cu")
+		(net 8)
+	)
+	(segment
 		(start 106.31 82)
 		(end 111 82)
@@
 	)
 	(segment
-		(start 128 68)
-		(end 148 68)
-		(width 1)
-		(layer "B.Cu")
-		(net 8)
-	)
-	(segment
 		(start 103 68)
 		(end 122 68)
@@
 	)
 	(segment
-		(start 125 65)
-		(end 128 68)
+		(start 151 65)
+		(end 151.5 65)
 		(width 1)
 		(layer "B.Cu")
@@
 	)
 	(segment
-		(start 105 65)
+		(start 104.5 65)
 		(end 112.84 65)
 		(width 1)
@@
 	)
 	(segment
+		(start 143 65)
+		(end 146 65)
+		(width 1)
+		(layer "B.Cu")
+		(net 12)
+	)
+	(segment
 		(start 149 62)
 		(end 153 62)
@@
 	)
 	(segment
-		(start 143 65)
-		(end 146 65)
+		(start 146 65)
+		(end 149 62)
 		(width 1)
 		(layer "B.Cu")
@@
 	)
 	(segment
-		(start 153 62)
-		(end 156 65)
+		(start 156 65)
+		(end 156.5 65)
 		(width 1)
 		(layer "B.Cu")
@@
 	)
 	(segment
-		(start 146 65)
-		(end 149 62)
+		(start 153 62)
+		(end 156 65)
 		(width 1)
 		(layer "B.Cu")
@@
 	)
 	(segment
-		(start 113 73.5)
-		(end 138.5 73.5)
-		(width 1)
-		(layer "B.Cu")
-		(net 14)
-	)
-	(segment
 		(start 113 75)
 		(end 113 73.5)
@@
 	)
 	(segment
+		(start 122 74.84)
+		(end 122 73.5)
+		(width 1)
+		(layer "B.Cu")
+		(net 14)
+	)
+	(segment
+		(start 113 73.5)
+		(end 122 73.5)
+		(width 1)
+		(layer "B.Cu")
+		(net 14)
+	)
+	(segment
 		(start 138.5 73.5)
 		(end 139 73)
@@
 	)
 	(segment
+		(start 122 73.5)
+		(end 138.5 73.5)
+		(width 1)
+		(layer "B.Cu")
+		(net 14)
+	)
+	(segment
 		(start 128.96 94.5)
 		(end 122 94.5)
@@
 	)
 	(segment
-		(start 122 86)
-		(end 124.66 88.66)
+		(start 122 85)
+		(end 122 86)
 		(width 1)
 		(layer "F.Cu")
@@
 		(width 1)
 		(layer "F.Cu")
+		(net 19)
+	)
+	(segment
+		(start 122 86)
+		(end 124.66 88.66)
+		(width 1)
+		(layer "F.Cu")

Commit message: warnungen weg
Parts:
- Q1: value BC556 -> BC556B
- moved R1 1.00 mm to (114.5, 103.5)
- moved D1 0.67 mm to (113.7, 75.0)
- moved R6 0.49 mm to (110.5, 75.0)
- moved R3 0.44 mm to (114.5, 99.1)
- moved R4 0.12 mm to (142.9, 75.2)
- moved R5 0.11 mm to (135.9, 75.2)
Routing:
- net GND: track 86.1 -> 101.5 mm
- net Net-(D1-K): track 40.1 -> 38.8 mm
- net Net-(U2-R): track 24.7 -> 24.0 mm
- net VCC: track 110.3 -> 109.6 mm
- net Net-(D1-A): track 8.57 -> 9.23 mm
- net Net-(Q1-B): track 8.22 -> 8.73 mm
Other:
- board text added: "JLCJLCJLCJLC"

Commit message: sieht besser aus im 3d render
Parts:
- J1: footprint Connector_PinSocket_2.54mm:PinSocket_1x04_P2.54mm_Vertical -> Connector_PinHeader_2.54mm:PinHeader_1x04_P2.54mm_Horizontal
