File: LPTastatur/LPTastatur.kicad_sch (KiCad schematic)
At the start: 23 parts, among them J1 Conn_01x04, Q1 BC556, SW1 SW_Push_Dual, SW2 SW_Push_Dual, SW3 SW_Push_Dual, U1 L7805, U2 NE555P

Commit message: upsi
Connections:
- net VCC: no longer R7.2
- net at D1.1 (K), D2.1 (K), D3.1 (K): now also R7.2
Other:
- moved on the sheet: C4, C5, U1
Changed lines of the file:
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@@
 	)
 	(junction
-		(at 55.88 80.01)
+		(at 34.29 91.44)
 		(diameter 0)
 		(color 0 0 0 0)
@@
 	)
 	(junction
+		(at 60.96 49.53)
+		(diameter 0)
+		(color 0 0 0 0)
+	)
+	(junction
 		(at 85.09 45.72)
 		(diameter 0)
@@
 	)
 	(junction
-		(at 40.64 80.01)
+		(at 19.05 91.44)
 		(diameter 0)
 		(color 0 0 0 0)
@@
 	)
 	(junction
-		(at 48.26 87.63)
+		(at 26.67 99.06)
 		(diameter 0)
 		(color 0 0 0 0)
@@
 	(wire
 		(pts
+			(xy 52.07 49.53) (xy 60.96 49.53)
+		)
+		(stroke
+			(width 0)
+			(type default)
+		)
+	)
+	(wire
+		(pts
 			(xy 120.65 45.72) (xy 85.09 45.72)
 		)
@@
 	(wire
 		(pts
-			(xy 40.64 87.63) (xy 48.26 87.63)
+			(xy 19.05 99.06) (xy 26.67 99.06)
 		)
 		(stroke
@@
 	(wire
 		(pts
-			(xy 48.26 87.63) (xy 55.88 87.63)
+			(xy 26.67 99.06) (xy 34.29 99.06)
 		)
 		(stroke
@@
 		(pts
 			(xy 80.01 140.97) (xy 91.44 140.97)
+		)
+		(stroke
+			(width 0)
+			(type default)
+		)
+	)
+	(wire
+		(pts
+			(xy 52.07 157.48) (xy 52.07 49.53)
 		)
 		(stroke
@@
 	(symbol
 		(lib_id "power:LINE")
-		(at 40.64 80.01 90)
+		(at 19.05 91.44 90)
 		(unit 1)
 		(exclude_from_sim no)
@@
 		(fields_autoplaced yes)
 		(property "Reference" "#PWR02"
-			(at 44.45 80.01 0)
+			(at 22.86 91.44 0)
 			(effects
 				(font
@@
 		)
 		(property "Value" "LINE"
-			(at 36.83 80.0099 90)
+			(at 15.24 91.4399 90)
 			(effects
 				(font
@@
 		)
 		(property "Footprint" ""
-			(at 40.64 80.01 0)
+			(at 19.05 91.44 0)
 			(effects
 				(font
@@
 		)
 		(property "Datasheet" ""
-			(at 40.64 80.01 0)
+			(at 19.05 91.44 0)
 			(effects
 				(font
@@
 		)
 		(property "Description" "Power symbol creates a global label with name \"LINE\""
-			(at 40.64 80.01 0)
+			(at 19.05 91.44 0)
 			(effects
 				(font
@@
 	(symbol
 		(lib_id "power:GND")
-		(at 48.26 87.63 0)
+		(at 26.67 99.06 0)
 		(unit 1)
 		(exclude_from_sim no)
@@
 		(fields_autoplaced yes)
 		(property "Reference" "#PWR04"
-			(at 48.26 93.98 0)
+			(at 26.67 105.41 0)
 			(effects
 				(font
@@
 		)
 		(property "Value" "GND"
-			(at 48.26 92.71 0)
+			(at 26.67 104.14 0)
 			(effects
 				(font
@@
 		)
 		(property "Footprint" ""
-			(at 48.26 87.63 0)
+			(at 26.67 99.06 0)
 			(effects
 				(font
@@
 		)
 		(property "Datasheet" ""
-			(at 48.26 87.63 0)
+			(at 26.67 99.06 0)
 			(effects
 				(font
@@
 		)
 		(property "Description" "Power symbol creates a global label with name \"GND\" , ground"
-			(at 48.26 87.63 0)
+			(at 26.67 99.06 0)
 			(effects
 				(font
@@
 	(symbol
 		(lib_id "power:VCC")
-		(at 55.88 80.01 270)
+		(at 34.29 91.44 270)
 		(unit 1)
 		(exclude_from_sim no)
@@
 		(fields_autoplaced yes)
 		(property "Reference" "#PWR03"
-			(at 52.07 80.01 0)
+			(at 30.48 91.44 0)
 			(effects
 				(font
@@
 		)
 		(property "Value" "VCC"
-			(at 59.69 80.0099 90)
+			(at 38.1 91.4399 90)
 			(effects
 				(font
@@
 		)
 		(property "Footprint" ""
-			(at 55.88 80.01 0)
+			(at 34.29 91.44 0)
 			(effects
 				(font
@@
 		)
 		(property "Datasheet" ""
-			(at 55.88 80.01 0)
+			(at 34.29 91.44 0)
 			(effects
 				(font
@@
 		)
 		(property "Description" "Power symbol creates a global label with name \"VCC\""
-			(at 55.88 80.01 0)
+			(at 34.29 91.44 0)
 			(effects
 				(font
@@
 	(symbol
 		(lib_id "power:VCC")
-		(at 52.07 157.48 90)
-		(unit 1)
-		(exclude_from_sim no)
-		(in_bom yes)
-		(on_board yes)
-		(dnp no)
-		(fields_autoplaced yes)
-		(property "Reference" "#PWR015"
-			(at 55.88 157.48 0)
-			(effects
-				(font
-					(size 1.27 1.27)
-				)
-				(hide yes)
-			)
-		)
-		(property "Value" "VCC"
-			(at 48.26 157.4799 90)
-			(effects
-				(font
-					(size 1.27 1.27)
-				)
-				(justify left)
-			)
-		)
-		(property "Footprint" ""
-			(at 52.07 157.48 0)
-			(effects
-				(font
-					(size 1.27 1.27)
-				)
-				(hide yes)
-			)
-		)
-		(property "Datasheet" ""
-			(at 52.07 157.48 0)
-			(effects
-				(font
-					(size 1.27 1.27)
-				)
-				(hide yes)
-			)
-		)
-		(property "Description" "Power symbol creates a global label with name \"VCC\""
-			(at 52.07 157.48 0)
-			(effects
-				(font
-					(size 1.27 1.27)
-				)
-				(hide yes)
-			)
-		)
-		(pin "1"
-		)
-		(instances
-			(project "LPTastatur"
-				(path "/c514f48a-b774-46ff-af59-98c8eb075295"
-					(reference "#PWR015")
-					(unit 1)
-				)
-			)
-		)
-	)
-	(symbol
-		(lib_id "power:VCC")
 		(at 104.14 130.81 0)
 		(unit 1)
@@
 	(symbol
 		(lib_id "Device:C")
-		(at 55.88 83.82 0)
+		(at 34.29 95.25 0)
 		(unit 1)
 		(exclude_from_sim no)
@@
 		(fields_autoplaced yes)
 		(property "Reference" "C4"
-			(at 59.69 82.5499 0)
+			(at 38.1 93.9799 0)
 			(effects
 				(font
@@
 		)
 		(property "Value" "4,7u 10V"
-			(at 59.69 85.0899 0)
+			(at 38.1 96.5199 0)
 			(effects
 				(font
@@
 		)
 		(property "Footprint" "Capacitor_THT:CP_Radial_Tantal_D4.5mm_P5.00mm"
-			(at 56.8452 87.63 0)
+			(at 35.2552 99.06 0)
 			(effects
 				(font
@@
 		)
 		(property "Datasheet" "~"
-			(at 55.88 83.82 0)
+			(at 34.29 95.25 0)
 			(effects
 				(font
@@
 		)
 		(property "Description" "Unpolarized capacitor"
-			(at 55.88 83.82 0)
+			(at 34.29 95.25 0)
 			(effects
 				(font
@@
 	(symbol
 		(lib_id "Device:C")
-		(at 40.64 83.82 0)
+		(at 19.05 95.25 0)
 		(mirror y)
 		(unit 1)
@@
 		(dnp no)
 		(property "Reference" "C5"
-			(at 36.83 82.5499 0)
+			(at 15.24 93.9799 0)
 			(effects
 				(font
@@
 		)
 		(property "Value" "0,1uF"
-			(at 36.83 85.0899 0)
+			(at 15.24 96.5199 0)
 			(effects
 				(font
@@
 		)
 		(property "Footprint" "Capacitor_THT:C_Rect_L7.0mm_W2.0mm_P5.00mm"
-			(at 39.6748 87.63 0)
+			(at 18.0848 99.06 0)
 			(effects
 				(font
@@
 		)
 		(property "Datasheet" "~"
-			(at 40.64 83.82 0)
+			(at 19.05 95.25 0)
 			(effects
 				(font
@@
 		)
 		(property "Description" "Unpolarized capacitor"
-			(at 40.64 83.82 0)
+			(at 19.05 95.25 0)
 			(effects
 				(font
@@
 	(symbol
 		(lib_id "Regulator_Linear:L7805")
-		(at 48.26 80.01 0)
+		(at 26.67 91.44 0)
 		(unit 1)
 		(exclude_from_sim no)
@@
 		(fields_autoplaced yes)
 		(property "Reference" "U1"
-			(at 48.26 73.66 0)
+			(at 26.67 85.09 0)
 			(effects
 				(font
@@
 		)
 		(property "Value" "L7805"
-			(at 48.26 76.2 0)
+			(at 26.67 87.63 0)
 			(effects
 				(font
@@
 		)
 		(property "Footprint" "Package_TO_SOT_THT:TO-220-3_Horizontal_TabDown"
-			(at 48.895 83.82 0)
+			(at 27.305 95.25 0)
 			(effects
 				(font
@@
 		)
 		(property "Datasheet" "http://www.st.com/content/ccc/resource/technical/document/datasheet/41/4f/b3/b0/12/d4/47/88/CD00000444.pdf/files/CD00000444.pdf/jcr:content/translations/en.CD00000444.pdf"
-			(at 48.26 81.28 0)
+			(at 26.67 92.71 0)
 			(effects
 				(font
@@
 		)
 		(property "Description" "Positive 1.5A 35V Linear Regulator, Fixed Output 5V, TO-220/TO-263/TO-252"
-			(at 48.26 80.01 0)
-			(effects
-				(font
+			(at 26.67 91.44 0)
+			(effects
+				(font

Commit message: din a5
Parts:
- Q1: value BC556 -> BC556B
Other:
- moved on the sheet: C1, C2, C3, C4, C5, C6, D1, D2, D3, J1, Q1, R1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

Commit message: sieht besser aus im 3d render
Parts:
- J1: footprint Connector_PinSocket_2.54mm:PinSocket_1x04_P2.54mm_Vertical -> Connector_PinHeader_2.54mm:PinHeader_1x04_P2.54mm_Horizontal
Changed lines of the file:
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@@
 			)
 		)
-		(property "Footprint" "Connector_PinSocket_2.54mm:PinSocket_1x04_P2.54mm_Vertical"
+		(property "Footprint" "Connector_PinHeader_2.54mm:PinHeader_1x04_P2.54mm_Horizontal"
 			(at 151.13 66.04 0)
 			(effects
