File: DBV/Adapter/Adapter.kicad_pcb (KiCad board)
At the start: 2 copper layers, 8 parts, among them J1 USB_B, U2 STM32C071CBUx, U3 AMS1117-3.3

Commit message: plcc68
Parts:
- removed D1: SK6812MINI, LED_SMD:LED_SK6812MINI_PLCC4_3.5x3.5mm_P1.75mm
- added R1: 1k, Resistor_SMD:R_0603_1608Metric, F.Cu at (73.7, 72.8)
- added R2: 1k, Resistor_SMD:R_0603_1608Metric, F.Cu at (71.9, 72.8)
- added U1: MC68000FN, PLCCaussen:PLCC-68_out, F.Cu at (72.0, 78.7)
- added U4: TCA9555PWR, Package_SO:TSSOP-24_4.4x7.8mm_P0.65mm, F.Cu at (65.7, 84.9)
- added U5: TCA9555PWR, Package_SO:TSSOP-24_4.4x7.8mm_P0.65mm, F.Cu at (79.0, 85.3)
- C1, C3: value 4.7uF -> C; footprint Capacitor_SMD:C_0805_2012Metric -> Capacitor_SMD:C_0603_1608Metric; moved to F.Cu
- C2, C4: value 100nF -> C; footprint Capacitor_SMD:C_0805_2012Metric -> Capacitor_SMD:C_0603_1608Metric; moved to F.Cu
- J1: value USB_B -> Conn_01x04_MountingPin; footprint Connector_USB:USB_B_TE_5787834_Vertical -> Connector_JST:JST_SH_BM04B-SRSS-TB_1x04-1MP_P1.00mm_Vertical
- U2: value STM32C071CBUx -> TCA9555PWR; footprint Package_DFN_QFN:QFN-48-1EP_7x7mm_P0.5mm_EP5.6x5.6mm -> Package_SO:TSSOP-24_4.4x7.8mm_P0.65mm
- U3: value AMS1117-3.3 -> TCA9555PWR; footprint Package_TO_SOT_SMD:SOT-223-3_TabPin2 -> Package_SO:TSSOP-24_4.4x7.8mm_P0.65mm
- moved C3 43.3 mm to (67.8, 77.1)
- moved U3 39.7 mm to (65.6, 72.4)
- moved C2 36.6 mm to (79.2, 77.1), turned to 0 degrees
- moved C1 33.6 mm to (73.5, 84.5), turned to 90 degrees
- moved C4 30.1 mm to (67.7, 79.9), turned to 180 degrees
- moved J1 27.7 mm to (73.7, 78.8), turned to 0 degrees
- moved U2 20.8 mm to (78.4, 72.0), turned to 180 degrees
Connections:
- C1 pad 1: +3.3V -> VCC
- C2 pad 1: +3.3V -> VCC
- C3 pad 1: +3.3V -> VCC
- C4 pad 1: +3.3V -> VCC
- J1 pad 1: +5V -> GND
- J1 pad 2: Net-(J1-D-) -> VCC
- J1 pad 3: Net-(J1-D+) -> SDA
- J1 pad 4: GND -> SCL
- U2 pad 10: unconnected-(U2-PF2-Pad10) -> Net-(U1-A11)
- U2 pad 11: unconnected-(U2-PA0-Pad11) -> Net-(U1-A12)
- U2 pad 12: unconnected-(U2-PA1-Pad12) -> GND
- U2 pad 13: unconnected-(U2-PA2-Pad13) -> Net-(U1-A19)
- U2 pad 14: unconnected-(U2-PA3-Pad14) -> Net-(U1-A20)
- U2 pad 15: unconnected-(U2-PA4-Pad15) -> Net-(U1-A18)
- U2 pad 17: unconnected-(U2-PA6-Pad17) -> Net-(U1-A16)
- U2 pad 18: unconnected-(U2-PA7-Pad18) -> Net-(U1-A15)
- U2 pad 19: unconnected-(U2-PB0-Pad19) -> Net-(U1-A14)
- U2 pad 2: unconnected-(U2-PC14-Pad2) -> GND
- U2 pad 20: unconnected-(U2-PB1-Pad20) -> Net-(U1-A13)
- U2 pad 21: unconnected-(U2-PB2-Pad21) -> GND
- U2 pad 22: unconnected-(U2-PB10-Pad22) -> SCL
- U2 pad 23: unconnected-(U2-PB11-Pad23) -> SDA
- U2 pad 24: unconnected-(U2-PB12-Pad24) -> VCC
- U2 pad 3: unconnected-(U2-PC15-Pad3) -> GND
- U2 pad 4: unconnected-(U2-PF3-Pad4) -> Net-(U1-A5)
- U2 pad 5: unconnected-(U2-VREF+-Pad5) -> Net-(U1-A6)
- U2 pad 6: +3.3V -> Net-(U1-A7)
- U2 pad 7: GND -> Net-(U1-A8)
- U2 pad 8: unconnected-(U2-PF0-Pad8) -> Net-(U1-A9)
- U2 pad 9: unconnected-(U2-PF1-Pad9) -> Net-(U1-A10)
- U3 pad 1: GND -> unconnected-(U3-~{INT}-Pad1)
- U3 pad 2: +3.3V -> GND
- U3 pad 3: +5V -> GND
Routing:
- net GND: track 0.00 -> 136.4 mm, vias 0 -> 17
- net VCC: track 0.00 -> 102.5 mm, vias 0 -> 10
- net SDA: track 0.00 -> 50.9 mm, vias 0 -> 4
- net SCL: track 0.00 -> 50.2 mm, vias 0 -> 3
- net Net-(U1-D10): track 0.00 -> 11.8 mm
- net Net-(U1-D9): track 0.00 -> 10.2 mm
- net Net-(U1-DTACK): track 0.00 -> 10.2 mm
- net Net-(U1-A4): track 0.00 -> 10.1 mm
- net Net-(U1-A13): track 0.00 -> 9.86 mm
- net Net-(U1-BG): track 0.00 -> 9.05 mm
- net Net-(U1-A3): track 0.00 -> 8.89 mm
- net Net-(U1-VMA): track 0.00 -> 8.81 mm
- net Net-(U1-D3): track 0.00 -> 8.50 mm
- net Net-(U1-D8): track 0.00 -> 8.49 mm
- net Net-(U1-A14): track 0.00 -> 8.36 mm
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- added copper zone on B.Cu, net GND
- added copper zone on F.Cu, net GND
Other:
- board outline added: 25.1 x 25.1 mm

Commit message: bom
Parts:
- C1, C2, C3, C4: value C -> 100nF
- J1: value Conn_01x04_MountingPin -> BM04B-SRSS-TB
Other:
- board text added: "Edge plate"
Changed lines of the file:
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@@
 			)
 		)
-		(property "Value" "C"
+		(property "Value" "100nF"
 			(at 0 1.43 90)
 			(layer "F.Fab")
@@
 			)
 		)
-		(property "Value" "C"
+		(property "Value" "100nF"
 			(at 0 1.43 0)
 			(layer "F.Fab")
@@
 			)
 		)
-		(property "Value" "Conn_01x04_MountingPin"
+		(property "Value" "BM04B-SRSS-TB"
 			(at 0 3.3 0)
 			(layer "F.Fab")
@@
 			)
 		)
-		(property "Value" "C"
+		(property "Value" "100nF"
 			(at 0 1.43 0)
 			(layer "F.Fab")
@@
 			)
 		)
-		(property "Value" "C"
+		(property "Value" "100nF"
 			(at 0 1.43 0)
 			(layer "F.Fab")
@@
 		(layer "Edge.Cuts")
 	)
+	(gr_rect
+		(start 60.96 91.059)
+		(end 83.185 92.075)
+		(stroke
+			(width 0.1)
+			(type default)
+		)
+		(fill none)
+		(layer "User.2")
+	)
+	(gr_rect
+		(start 60.96 65.405)
+		(end 83.185 66.421)
+		(stroke
+			(width 0.1)
+			(type default)
+		)
+		(fill none)
+		(layer "User.2")
+	)
+	(gr_rect
+		(start 84.328 67.564)
+		(end 85.217 89.535)
+		(stroke
+			(width 0.1)
+			(type default)
+		)
+		(fill none)
+		(layer "User.2")
+	)
+	(gr_rect
+		(start 58.42 67.183)
+		(end 59.69 89.916)
+		(stroke
+			(width 0.1)
+			(type default)
+		)
+		(fill none)
+		(layer "User.2")
+	)
+	(gr_text "Edge plate"
+		(at 67.945 64.77 0)
+		(layer "User.2")
+		(effects
+			(font
+				(size 1 1)
+				(thickness 0.15)
+			)
+			(justify left bottom)
+		)
+	)
 	(segment
