File: ST25/ST25.kicad_pcb (KiCad board)
At the start: 2 copper layers, 51.4 x 126.4 mm, 41 parts, among them J1 Conn_01x13, J2 Conn_01x13, J3 Conn_01x13, J4 Conn_01x08, J5 Conn_01x08, SW1 [1], SW10 [*], SW11 [0], SW12 [#], SW13 [1], SW14 [2], SW15 [3], SW16 [4], SW17 [5], SW18 [6], SW19 [7], SW2 [2], SW20 [8], SW21 [9], SW22 [*], SW23 [0], SW24 [#], SW3 [3], SW4 [4], SW5 [5], SW6 [6], SW7 [7], SW8 [8], SW9 [9], U1 HEF4094B, U2 HEF4094B

Commit message: led und ffc
Parts:
- removed J2, J3: Conn_01x13, Connector_PinHeader_2.54mm:PinHeader_1x13_P2.54mm_Vertical
- added D3: LED, LED_SMD:LED_0603_1608Metric, F.Cu at (118.8, 70.0)
- added H1: MountingHole, MountingHole:MountingHole_3mm, F.Cu at (79.5, 62.5)
- added H2: MountingHole, MountingHole:MountingHole_3mm, F.Cu at (126.8, 62.5)
- added J6: Conn_01x13_MountingPin, Connector_FFC-FPC:TE_1-84952-3_1x13-1MP_P1.0mm_Horizontal, F.Cu at (102.5, 58.8)
- added J7: Conn_01x13_MountingPin, Connector_FFC-FPC:TE_1-84953-3_1x13-1MP_P1.0mm_Horizontal, F.Cu at (102.5, 70.0)
- added R3: 47k, Resistor_SMD:R_0603_1608Metric, F.Cu at (122.9, 70.0)
- moved J1 8.85 mm to (102.5, 45.0)
Routing:
- net VCC: track 69.7 -> 97.0 mm, vias 3 -> 5
- net GND: track 201.3 -> 177.5 mm, vias 2 -> 18
- net Net-(J1-Pin_12): track 166.3 -> 186.6 mm, vias 3 -> 4
- net Net-(J1-Pin_4): track 186.3 -> 206.5 mm, vias 2 -> 4
- net Net-(J1-Pin_2): track 184.6 -> 203.4 mm, vias 1 -> 3
- net STROBE: track 44.3 -> 59.9 mm, vias 0 -> 1
- net Net-(J1-Pin_8): track 146.4 -> 161.7 mm, vias 2 -> 4
- net Net-(J1-Pin_11): track 12.7 -> 25.8 mm, vias 0 -> 1
- net /BOTK: track 211.8 -> 223.0 mm, vias 1 -> 4
- net Net-(J1-Pin_10): track 146.7 -> 156.8 mm, vias 3 -> 4
- net DATAin: track 26.3 -> 35.9 mm, vias 0 -> 1
- net CLK: track 62.1 -> 71.7 mm, vias 4 -> 5
- net +5V: track 49.0 -> 57.6 mm, vias 2 -> 3
- net Net-(J1-Pin_6): track 186.3 -> 190.9 mm, vias 3 -> 4
- net Net-(D3-A): track 0.00 -> 2.52 mm
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Other:
- board size 51.4 x 126.4 mm -> 51.4 x 134.6 mm

Commit message: loecher dann doch
Parts:
- added J2: Conn_01x13, Connector_PinHeader_2.54mm:PinHeader_1x13_P2.54mm_Vertical, F.Cu at (87.3, 53.2)
- moved J1 2.38 mm to (102.5, 42.6)
- moved H2 2.21 mm to (126.4, 60.3)
- moved H1 2.17 mm to (79.5, 60.3)
Routing:
- net GND: track 177.5 -> 187.7 mm, vias 18 -> 26
- net /TOPK: vias 1 -> 3
- net (no net): vias 69 -> 95
Other:
- board size 51.4 x 134.6 mm -> 51.4 x 137 mm
