File: ProgrammierStation/ProgrammierStation.kicad_sch (KiCad schematic)
At the start: 22 parts, among them J1 DB, J2 DB, J3 Conn_02x03_Counter_Clockwise, J7 ZLK intern, J9 Conn_02x04_Counter_Clockwise, SW1 SW_DPDT_x2, SW2 SW_Push, SW3 SW_Push, U2 74HC14

Commit message: ps
Parts:
- added D4: 1N4001, Diode_THT:D_DO-41_SOD81_P10.16mm_Horizontal, symbol Diode:1N4001
Changed lines of the file:
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@@
+	)
+	(symbol
+		(lib_id "Diode:1N4001")
+		(at 180.34 127 0)
+		(unit 1)
+		(exclude_from_sim no)
+		(in_bom yes)
+		(on_board yes)
+		(dnp no)
+		(fields_autoplaced yes)
+		(property "Reference" "D4"
+			(at 180.34 120.65 0)
+			(effects
+				(font
+					(size 1.27 1.27)
+				)
+			)
+		)
+		(property "Value" "1N4001"
+			(at 180.34 123.19 0)
+			(effects
+				(font
+					(size 1.27 1.27)
+				)
+			)
+		)
+		(property "Footprint" "Diode_THT:D_DO-41_SOD81_P10.16mm_Horizontal"
+			(at 180.34 127 0)
+			(effects
+				(font
+					(size 1.27 1.27)
+				)
+				(hide yes)
+			)
+		)
+		(property "Datasheet" "http://www.vishay.com/docs/88503/1n4001.pdf"
+			(at 180.34 127 0)
+			(effects
+				(font
+					(size 1.27 1.27)
+				)
+				(hide yes)
+			)
+		)
+		(property "Description" "50V 1A General Purpose Rectifier Diode, DO-41"
+			(at 180.34 127 0)
+			(effects
+				(font
+					(size 1.27 1.27)
+				)
+				(hide yes)
+			)
+		)
+		(property "Sim.Device" "D"
+			(at 180.34 127 0)
+			(effects
+				(font
+					(size 1.27 1.27)
+				)
+				(hide yes)
+			)
+		)
+		(property "Sim.Pins" "1=K 2=A"
+			(at 180.34 127 0)
+			(effects
+				(font
+					(size 1.27 1.27)
+				)
+				(hide yes)
+			)
+		)
+		(pin "2"
+		)
+		(pin "1"
+		)
+		(instances
+			(project ""
+				(path "/8791464e-45ca-4793-8042-4a41a8adeea1"
+					(reference "D4")
+					(unit 1)
+				)
+			)
+		)
 	)
 	(symbol

Commit message: beschriftung hinten
Parts:
- added C4, C5, C6: 100uF, Capacitor_Tantalum_SMD:CP_EIA-7132-20_AVX-U, symbol Device:C_Polarized
- added FID1: Fiducial, Symbol:WEEE-Logo_8.4x12mm_SilkScreen, symbol Mechanical:Fiducial
- added R7, R8, R9: 330, Resistor_SMD:R_0603_1608Metric, symbol Device:R
- added U3: 74HC14, Package_SO:SO-14_3.9x8.65mm_P1.27mm, symbol 74xx:74HC14
- J3: value Conn_02x03_Counter_Clockwise -> Sound
- J9: value Conn_02x04_Counter_Clockwise -> ATMEL/Flash
- Nano-3: renamed from A1; value Arduino_Nano_v3.x -> ISP
- SW1: value SW_DPDT_x2 -> Sound
- SW2, SW3: value SW_Push -> Reset
Connections:
- net CS: now also J9.3 (Pin_3)
- net GND: now also C4.2, C5.2, C6.2, R7.2, R8.2, R9.2, U3.7 (GND); no longer D1.1 (K), D2.1 (K), D3.1 (K)
- net MISO: now also J9.5 (Pin_5)
- net MOSI: now also J9.4 (Pin_4)
- net SCK: now also J9.6 (Pin_6)
- net at R2.1: now also D2.1 (K), R8.1
- net at U2.8: now also U3.8
- net at U2.9: now also U3.9
- net at U2.10: now also U3.10
- net at U2.11: now also U3.11
- net at R1.1: now also D3.1 (K), R9.1
- net at C2.1: now also C5.1
- net at C3.1: now also C6.1
- net at C1.1: now also C4.1
- net +12V: now reaches J9.8 (Pin_8)
- net +12V: now also J3.6 (Pin_6), J7.8 (Pin_8)
- net at U2.5: now also U3.5
- net at U2.6: now also U3.6
- net at U2.14 (VCC): now also U3.14 (VCC)
- net at U2.1: now also U3.1
- net at U2.2: now also U3.2
- net at R3.1: now also D1.1 (K), R7.1
- net at U2.12: now also U3.12
- net at U2.13: now also U3.13
- net at U2.3: now also U3.3
- net at U2.4: now also U3.4
Other:
- moved on the sheet: R1, R2, R3

Commit message: halbzeit
Parts:
- added J4: CP2102, Connector_PinHeader_2.54mm:PinHeader_1x06_P2.54mm_Vertical, symbol Connector_Generic:Conn_01x06
- added J5: INA226, Connector_PinHeader_2.54mm:PinHeader_1x08_P2.54mm_Vertical, symbol Connector_Generic:Conn_01x08
- added PS1: MEE1S0512SC, Modules:MT3608, symbol Converter_DCDC:MEE1S0512SC
- added R10: 1, Resistor_SMD:R_0603_1608Metric, symbol Device:R
- C4, C5, C6: footprint Capacitor_Tantalum_SMD:CP_EIA-7132-20_AVX-U -> Capacitor_Tantalum_SMD:CP_EIA-6032-20_AVX-F
- D4: footprint Diode_THT:D_DO-41_SOD81_P10.16mm_Horizontal -> Diode_THT:D_DO-41_SOD81_P7.62mm_Horizontal
Connections:
- net +12V: now also J1.c6 (Pin_c6), PS1.4 (+Vout); no longer J3.6 (Pin_6)
- net +3.3V: now also J9.7 (Pin_7); no longer J7.7 (Pin_7)
- net +5V: now also C2.1, C5.1, D4.2 (A), Nano-3.6 (D3), R5.1, R6.2, U2.14 (VCC), U3.14 (VCC), J4.1 (Pin_1); no longer J1.a1 (Pin_a1)
- net +5VA: now also C3.1, C6.1, D4.1 (K), J9.2 (Pin_2), J5.8 (Pin_8), PS1.2 (+Vin); no longer J7.2 (Pin_2)
- net GND: now also J1.a4 (Pin_a4), J4.2 (Pin_2), J5.7 (Pin_7), PS1.1 (-Vin), PS1.3 (-Vout)
- net RX: now also J2.b8 (Pin_b8), Nano-3.5 (D2), SW1.5 (B), J4.4 (Pin_4); no longer J1.b8 (Pin_b8)
- net TX: now also J2.c7 (Pin_c7), SW1.2 (B), J4.3 (Pin_3); no longer J1.c7 (Pin_c7)
- net at U3.10: no longer U2.10
- net at U3.11: no longer U2.11
- net at J1.a7 (Pin_a7): now also J1.a1 (Pin_a1), J2.a1 (Pin_a1), J2.a7 (Pin_a7), R5.2
- net RESET: now reaches SW3.2
- net RESET: now also Nano-3.28 (~{RESET}), SW2.1
- net at U2.8: no longer U3.8
- net at U2.9: no longer U3.9
- net at U2.3, U3.3: now also J3.1 (Pin_1)
- net at R4.1: now also R10.1
- net at R4.2: now also J2.b5 (Pin_b5), R10.2
- net SDA: now reaches Nano-3.23 (A4)
- net SDA: now also J5.5 (Pin_5)
- net SCL: now reaches Nano-3.24 (A5)
- net SCL: now also J5.6 (Pin_6)
- net ALE: now reaches Nano-3.7 (D4)
- net ALE: now also J5.4 (Pin_4)
- net at J3.4 (Pin_4): now also U2.2, U3.2
- net at U3.5: no longer U2.5
- net at U3.6: no longer U2.6
- net at U3.12: no longer U2.12
- net at U3.13: no longer U2.13
- new net: J3.6 (Pin_6), J5.2 (Pin_2)
- no-connect marks 20 -> 81
Other:
- moved on the sheet: J1B, J1C, J2B, J2C, J3, R4, R5, R6, SW3, U2A, U2B, U2E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

Commit message: rev1
Parts:
- added D5: 1N4001, Diode_SMD:D_SOD-123, symbol Diode:1N4001
- added R11: 1, Resistor_SMD:R_0603_1608Metric, symbol Device:R
- added R12: 10k, Resistor_SMD:R_0603_1608Metric, symbol Device:R
Connections:
- net +5V: now also D5.2 (A), R11.1, R12.2
- net +5VA: now also C1.1, C4.1, D5.1 (K)
- net at J1.a1 (Pin_a1), J1.a7 (Pin_a7), J2.a1 (Pin_a1)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: now also R11.2
- net at SW1.3 (C): now also U2.1, U3.1
- net at U2.4, U3.4: now also SW1.6 (C)
- net at R10.1, R4.1: now also J2.b9 (Pin_b9)
- net at R10.2, R4.2: now also J1.b5 (Pin_b5); no longer J2.b5 (Pin_b5)
- net at R6.1: now also J2.b5 (Pin_b5), R12.1
Other:
- moved on the sheet: D4, J3, J5, R10, R4, R6, SW1A, SW1B, U2A, U2B, U3A, U3B

Commit message: zweite reihe
Parts:
- added J6: INA226, Connector_PinHeader_2.54mm:PinHeader_1x08_P2.54mm_Vertical, symbol Connector_Generic:Conn_01x08
Connections:
- net +12V: now also C1.1, C4.1, J5.1 (Pin_1), J6.8 (Pin_8)
- net +5VA: now also J6.1 (Pin_1); no longer C1.1, C4.1
- net ALE: now also J6.5 (Pin_5)
- net GND: now also J6.2 (Pin_2)
- net SCL: now also J6.4 (Pin_4)
- net SDA: now also J6.3 (Pin_3)
- net at J3.6 (Pin_6), J5.2 (Pin_2): now also J6.7 (Pin_7)
- no-connect marks 81 -> 83

Commit message: stromleitungen
Connections:
- no-connect marks 83 -> 85

Commit message: DATENBANK
Parts:
- PS1: value MEE1S0512SC -> MT3608
Changed lines of the file:
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@@
 			)
 		)
-		(property "Value" "MEE1S0512SC"
+		(property "Value" "MT3608"
 			(at 54.61 173.99 0)
 			(effects

Commit message: jumper
Parts:
- added J8: Conn_01x06, Connector_PinHeader_2.54mm:PinHeader_1x06_P2.54mm_Vertical, symbol Connector_Generic:Conn_01x06
- added JP1, JP2, JP3, JP4, JP5, JP6, JP7, JP8, JP9: Jumper_2_Bridged, Jumper:SolderJumper-2_P1.3mm_Bridged_Pad1.0x1.5mm, symbol Jumper:Jumper_2_Bridged
Connections:
- net GND: now also J8.2 (Pin_2)
- net at SW1.1 (A): now also JP9.2 (B)
- net 12V_SOUND: now reaches J3.6 (Pin_6), J5.2 (Pin_2), J6.7 (Pin_7)
- net 12V_SOUND: now also J8.6 (Pin_6)
- net DSP REPLY: now reaches J3.1 (Pin_1), U2.3, U3.3
- net DSP REPLY: now also J8.1 (Pin_1), JP8.1 (A)
- net at R12.1, R6.1: now also JP3.1 (A); no longer J2.b5 (Pin_b5)
- net at R10.1, R4.1: now also JP2.2 (B); no longer J2.b9 (Pin_b9)
- net at R10.2, R4.2: now also JP1.1 (A); no longer J1.b5 (Pin_b5)
- net DSP DATEN: now reaches J3.4 (Pin_4), U2.2, U3.2
- net DSP DATEN: now also J8.4 (Pin_4), JP9.1 (A)
- net at SW1.4 (A): now also JP8.2 (B)
- new net: J1.a1 (Pin_a1), JP4.2 (B)
- new net: J1.a7 (Pin_a7), JP5.2 (B)
- new net: J2.b9 (Pin_b9), JP2.1 (A)
- new net: JP4.1 (A), JP5.1 (A), JP6.1 (A), JP7.1 (A), R11.2, R5.2
- new net: J2.a1 (Pin_a1), JP6.2 (B)
- new net: J2.a7 (Pin_a7), JP7.2 (B)
- new net: J2.b5 (Pin_b5), JP3.2 (B)
- new net: J1.b5 (Pin_b5), JP1.2 (B)
- no-connect marks 85 -> 84
Other:
- moved on the sheet: J1A, J1B, J1C, J2A, J2B, J2C, R10, R12, R4, R6
