File: DB1MBRedesign/DB1MB.kicad_sch (KiCad schematic)
At the start: 53 parts, among them J1 Conn_01x10_Socket, J2 Conn_01x10_Socket, J3 Conn_01x10_Socket, J4 Conn_01x10_Socket, J5 Conn_01x10_Socket, J6 Conn_01x10_Socket, U1 MC68331, U2 ATmega48V-10A, U3 CY62157, U4 74LS573, U5 74LS245, U6 74LS573, U7 74LS573, U8 74LS245, U9 74LS28

Commit message: we
Parts:
- added C12, C13, C14, C15, C16: C, Capacitor_SMD:C_0805_2012Metric, symbol Device:C
Connections:
- net A15: now also U3.22 (A14)
- net A16: now also U3.21 (A15)
- net A17: now also U3.20 (A16)
- net A18: now also U3.19 (A17)
- net D0: now also U7.2 (D0), U8.9 (A7)
- net D1: now also U7.3 (D1), U8.8 (A6)
- net D10: now also U4.7 (D5), U5.7 (A5); no longer U4.17 (Q2), U5.17 (B1)
- net D11: now also U4.6 (D4), U5.6 (A4); no longer U4.16 (Q3), U5.16 (B2)
- net D12: now also U4.5 (D3), U5.5 (A3); no longer U4.15 (Q4), U5.15 (B3)
- net D13: now also U4.4 (D2), U5.4 (A2); no longer U4.14 (Q5), U5.14 (B4)
- net D14: now also U4.3 (D1), U5.3 (A1); no longer U4.13 (Q6), U5.13 (B5)
- net D15: now also U4.2 (D0), U5.2 (A0); no longer U4.12 (Q7), U5.12 (B6)
- net D2: now also U7.4 (D2), U8.7 (A5)
- net D3: now also U7.5 (D3), U8.6 (A4)
- net D4: now also U7.6 (D4), U8.5 (A3)
- net D5: now also U7.7 (D5), U8.4 (A2)
- net D6: now also U7.8 (D6), U8.3 (A1)
- net D7: now also U7.9 (D7), U8.2 (A0)
- net D8: now also U4.9 (D7), U5.9 (A7); no longer U4.19 (Q0), U5.19 (CE)
- net D9: now also U4.8 (D6), U5.8 (A6); no longer U4.18 (Q1), U5.18 (B0)
- net GND: now also U1.22 (PAI), U1.30 (PGP3), U1.31 (PGP2), U1.32 (PGP1), U9.12, U9.6, C12.2, C13.2, C14.2, C15.2, C16.2
- net VDD: now also J3.1 (Pin_1), U2.4 (VCC), U2.6 (VCC), U4.20 (VCC), U5.20 (VCC), U8.20 (VCC), C12.1, C13.1, C14.1, C15.1, C16.1
- net at U9.11: now also U9.5, U9.8
- net at U8.11 (B7): now also U7.19 (Q0)
- net at U8.12 (B6): now also U7.18 (Q1)
- net at U8.13 (B5): now also U7.17 (Q2)
- net at U8.14 (B4): now also U7.16 (Q3)
- net at U8.15 (B3): now also U7.15 (Q4)
- net at U8.16 (B2): now also U7.14 (Q5)
- net at U8.17 (B1): now also U7.13 (Q6)
- net at U8.18 (B0): now also U7.12 (Q7)
- net at RN8.1 (R1.1): now also RN2.7 (R2.2)
- net at RN8.2 (R2.1): now also RN2.5 (R4.2)
- net at RN8.5 (R4.2): now also RN8.6 (R3.2), RN8.7 (R2.2), RN8.8 (R1.2)
- net at U9.3: now also U9.9
- net at U2.10 (PD6): now also U1.77 (DSO)
- net A19: now reaches U3.18 (A18)
- net A19: now also U1.6 (A19)
- net A20: now reaches RN3.7 (R2.2)
- net A20: now also U1.7 (A20)
- net A23: now reaches U1.10 (A23)
- net A21: now reaches U1.8 (A21)
- net A22: now reaches U1.9 (A22)
- net A22: now also RN1.7 (R2.2)
- net at J3.10 (Pin_10): now also J3.4 (Pin_4)
- net at U5.11 (B7): now also J3.2 (Pin_2), U4.12 (Q7)
- new net: J1.2 (Pin_2), U4.14 (Q5), U5.13 (B5)
- new net: J1.3 (Pin_3), U4.17 (Q2), U5.16 (B2)
- new net: J1.4 (Pin_4), U4.19 (Q0), U5.18 (B0)
- new net: J2.2 (Pin_2), U4.13 (Q6), U5.12 (B6)
- new net: J2.3 (Pin_3), U4.16 (Q3), U5.15 (B3)
- new net: J2.4 (Pin_4), U4.18 (Q1), U5.17 (B1)
- new net: J3.3 (Pin_3), U4.15 (Q4), U5.14 (B4)
- now unconnected: U5.1 (A->B)
- no-connect marks 7 -> 11
Other:
- moved on the sheet: RN8, U5, U7, U8, U9A, U9B, U9C, U9D

Commit message: db
Parts:
- removed U9: 74LS28, Package_SO:TSSOP-14_4.4x5mm_P0.65mm, symbol 74xx:74LS28
- added C17, C18, C19, C20, C21, C22, C23: C, Capacitor_SMD:C_0805_2012Metric, symbol Device:C
- added D1, D2, D3, D4, D5: BAS40-05, Package_TO_SOT_SMD:SOT-23-3, symbol Device:D_Schottky_Dual_CommonCathode_AAK
- added D6, D7: LED, LED_SMD:LED_ASMB-KTF0-0A306, symbol Device:LED
- added J7: Conn_01x04_Socket, ADP:Deckel, symbol Connector:Conn_01x04_Socket
- added JP1: Jumper_2_Open, Jumper:SolderJumper-2_P1.3mm_Open_Pad1.0x1.5mm, symbol Jumper:Jumper_2_Open
- added Q1: Q_Photo_NPN_CBE, OptoDevice:Osram_SMD-SmartDIL, symbol Device:Q_Photo_NPN_CBE
- added TP10, TP11, TP12, TP13, TP14, TP15, TP8, TP9: TestPoint, TestPoint:TestPoint_Pad_D1.0mm, symbol Connector:TestPoint
- added U11: 74LS08, Package_SO:TSSOP-14_4.4x5mm_P0.65mm, symbol 74xx:74LS08
- added U9: 74LS20, Package_SO:TSSOP-14_4.4x5mm_P0.65mm, symbol 74xx:74LS20
- RN1, RN3: value R_Pack04 -> 330
- RN2: value R_Pack04 -> 750
- RN6, RN7, RN8: value R_Pack04 -> 822
Connections:
- net A19: now also D3.2 (A)
- net A21: now also U11.10, U11.5, U11.9
- net GND: now also J3.10 (Pin_10), J3.4 (Pin_4), J6.10 (Pin_10), C17.2, C18.2, C19.2, C20.2, C21.2, C22.2, C23.2, JP1.2 (B), U11.7 (GND), U9.7 (GND); no longer RN5.2 (R2.1), RN5.3 (R3.1), RN5.4 (R4.1), RN6.1 (R1.1), RN6.2 (R2.1), RN6.3 (R3.1), RN6.4 (R4.1)
- net VDD: now also RN13.5 (R4.2), RN13.6 (R3.2), RN13.7 (R2.2), RN13.8 (R1.2), RN5.2 (R2.1), RN5.3 (R3.1), RN5.4 (R4.1), RN6.1 (R1.1), RN6.2 (R2.1), RN6.3 (R3.1), RN6.4 (R4.1), U10.14 (Vdd), U6.20 (VCC), U7.20 (VCC), C17.1, C18.1, C19.1, C20.1, C21.1, C22.1, C23.1, D1.3 (K), U11.14 (VCC), U9.13, U9.14 (VCC), U9.5
- net at TP1.1, U1.81 (FREEZE/QUOT): now also U2.14 (PB2)
- net at J1.8 (Pin_8): now also RN12.6 (R3.2)
- net at RN12.1 (R1.1): now also U1.69 (PQS4)
- net at RN12.2 (R2.1): now also J3.9 (Pin_9)
- net at RN12.4 (R4.1): now also J6.5 (Pin_5)
- net at RN12.5 (R4.2): now also U1.103 (R/~{W})
- net at RN12.7 (R2.2): now also U11.8
- net at RN5.5 (R4.2): now also RN4.7 (R2.2), U1.101 (PF1)
- net at J2.8 (Pin_8): now also RN11.8 (R1.2)
- net MOSI: now reaches U10.11 (DATA)
- net MOSI: now also RN7.8 (R1.2), U10.6 (WR), U2.15 (PB3), TP12.1
- net SCK: now reaches U10.12 (CLK)
- net at RN11.1 (R1.1): now also U1.75 (PQS7/TXD)
- net at RN13.1 (R1.1): now also U1.95 (PF7)
- net at RN13.2 (R2.1): now also RN10.3 (R3.1), U1.100 (PF2)
- net at RN13.3 (R3.1): now also RN10.2 (R2.1), U1.99 (PF3)
- net at RN13.4 (R4.1): now also RN10.1 (R1.1), U1.113 (PE1)
- net at TP7.1, U1.102 (PF0): now also RN6.7 (R2.2)
- net at RN10.6 (R3.2): now also J5.1 (Pin_1)
- net at RN10.7 (R2.2): now also J4.1 (Pin_1)
- net at RN10.8 (R1.2): now also J5.5 (Pin_5)
- net at U7.17 (Q2), U8.13 (B5): now also J4.2 (Pin_2)
- net at U7.12 (Q7), U8.18 (B0): now also J4.4 (Pin_4)
- net CE: now reaches U8.19 (CE)
- net CE: now also U5.19 (CE), TP15.1, U11.6
- net at U6.12 (Q7): now also J4.8 (Pin_8)
- net at U6.13 (Q6): now also J6.9 (Pin_9)
- net at U6.14 (Q5): now also J5.9 (Pin_9)
- net at U6.15 (Q4): now also J4.9 (Pin_9)
- net at U6.16 (Q3): now also J5.8 (Pin_8)
- net at U6.17 (Q2): now also J6.8 (Pin_8)
- net at U6.18 (Q1): now also J4.7 (Pin_7)
- net at U6.19 (Q0): now also J5.7 (Pin_7)
- net at U2.13 (PB1): now also RN7.7 (R2.2)
- net MISO: now reaches U2.16 (PB4)
- net MISO: now also TP13.1
- net at U2.17 (PB5): now also RN7.6 (R3.2)
- net at U2.23 (PC0): now also RN9.1 (R1.1), TP4.1, U1.79 (DSCLK)
- net at TP2.1, U1.78 (DSI), U2.26 (PC3): now also RN9.2 (R2.1)
- net at U2.30 (PD0): now also TP14.1
- net at U3.17 (~{WE}): now also D2.2 (A)
- net at U3.39 (~{BLE}): now also D1.1 (A)
- net at U3.41 (~{OE}): now also D1.2 (A)
- net OE: now reaches U7.1 (OE)
- net OE: now also U4.1 (OE), U9.6
- net at BT1.2 (-), BT2.2 (-), TP3.1: now also JP1.1 (A)
- net at U4.11 (Load): now also TP10.1, U9.8
- net at RN9.3 (R3.1): now also RN9.7 (R2.2), RN9.8 (R1.2)
- net at RN6.5 (R4.2), TP6.1: now also U1.112 (PE2)
- net at RN4.6 (R3.2), U1.65 (PQS0): now also RN6.8 (R1.2)
- net at U1.114 (PE0): now also RN6.6 (R3.2)
- net at U1.3 (FC0): now also D2.1 (A)
- net at U1.5 (FC2): now also TP11.1, U11.12, U11.13, U11.4, U9.1, U9.12, U9.4
- new net: U11.1, U11.2, U9.9
- new net: TP9.1, U9.10, U9.2
- new net: D2.3 (K), D3.3 (K)
- new net: J7.1 (Pin_1), TP8.1
- new net: D4.1 (A), D4.2 (A)
- no-connect marks 11 -> 16
Other:
- moved on the sheet: BT1, BT2, H1, H2, H3, H4, J4, J5, J6, RN10, RN11, RN12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

Commit message: db
Parts:
- added D8: LED, LED_SMD:LED_ASMB-KTF0-0A306, symbol Device:LED
- added FID1: Fiducial, Fiducial:Fiducial_0.75mm_Mask2.25mm, symbol Mechanical:Fiducial
- added Q2: Q_Photo_NPN_CBE, OptoDevice:Osram_SMD-SmartDIL, symbol Device:Q_Photo_NPN_CBE
- added TP16, TP17, TP18, TP19: TestPoint, TestPoint:TestPoint_Pad_D1.0mm, symbol Connector:TestPoint
Connections:
- net at RN5.6 (R3.2): now also U1.94 (~{BERR})
- net at RN5.7 (R2.2): now also U1.93 (~{HALT})
- net at U10.8 (CE): now also RN7.7 (R2.2), U2.13 (PB1)
- net at U11.3: now also RN1.8 (R1.2)
- net at U6.11 (Load): now also U1.106 (PE4)
- net at RN2.7 (R2.2), RN8.1 (R1.1): now also U1.76 (RXD)
- net at U2.1 (PD3): now also TP17.1
- net at U2.19 (ADC6): now also D8.2 (A)
- net at U2.2 (PD4): now also TP16.1
- net at U2.24 (PC1): now also TP18.1
- net at U2.31 (PD1): now also D8.1 (K), TP19.1
- net at U2.9 (PD5): now also Q2.1 (C)
- net at U1.71 (PQS6): now also RN1.6 (R3.2)
Other:
- moved on the sheet: U10

Commit message: kicad9 update
Parts:
- removed J1, J2, J3, J4, J5, J6: Conn_01x10_Socket, Connector_PinSocket_2.54mm:PinSocket_1x10_P2.54mm_Vertical, symbol Connector:Conn_01x10_Socket
- added C24: C, Capacitor_SMD:C_1206_3216Metric, symbol Device:C
- added C25: C, Capacitor_SMD:C_0805_2012Metric, symbol Device:C
- added D10: BAV70, Package_TO_SOT_SMD:SOT-23, symbol Diode:BAV70
- added D9: D_Zener, Diode_SMD:D_SOD-123, symbol Device:D_Zener
- added J8, J9: DIN41612_03x10_ABC, Connector_DIN:DIN41612_R3_3x10_Male_Vertical_THT, symbol DIN41612:DIN41612_03x10_ABC
- added Q3: BSS84, Package_TO_SOT_SMD:SOT-23-3, symbol Transistor_FET:BSS84
- added Q4: IRF7313, Package_SO:SOIC-8_3.9x4.9mm_P1.27mm, symbol Transistor_FET:IRF7309IPBF
- added R1: 10, Resistor_SMD:R_0805_2012Metric, symbol Device:R
- added R2: 1, Resistor_SMD:R_0805_2012Metric, symbol Device:R
- added R4, R5, R6, R7: R, Resistor_SMD:R_0603_1608Metric, symbol Device:R
- added TP20, TP21, TP24: TestPoint, TestPoint:TestPoint_Pad_D1.0mm, symbol Connector:TestPoint
- added TP22, TP23: TestPoint, TestPoint:TestPoint_Pad_1.0x1.0mm, symbol Connector:TestPoint
- added Y1: Crystal_GND23, Crystal:Crystal_SMD_SeikoEpson_MC306-4Pin_8.0x3.2mm, symbol Device:Crystal_GND23
Connections:
- net GND: now also D9.2 (A), J8.a1 (Pin_a1), J8.a7 (Pin_a7), J9.a1 (Pin_a1), J9.a7 (Pin_a7), Q4.1 (S), Q4.3 (1)
- net PF1: now also J8.a5 (Pin_a5)
- net VDD: now also U2.18 (AVCC), D9.1 (K), J8.a10 (Pin_a10), J9.a10 (Pin_a10)
- net at RN3.2 (R2.1): now also J8.c10 (Pin_c10)
- net at RN1.3 (R3.1): now also J8.c1 (Pin_c1)
- net at U4.14 (Q5), U5.13 (B5): now also J8.c9 (Pin_c9)
- net at U4.17 (Q2), U5.16 (B2): now also J8.c8 (Pin_c8)
- net at U4.19 (Q0), U5.18 (B0): now also J8.c7 (Pin_c7)
- net at RN3.1 (R1.1): now also J8.c6 (Pin_c6)
- net at RN2.2 (R2.1): now also J8.c4 (Pin_c4)
- net at RN12.6 (R3.2): now also J8.c3 (Pin_c3)
- net at RN1.1 (R1.1): now also J8.c2 (Pin_c2)
- net at D5.1 (A): now also Q3.2 (S), R1.1, R2.2
- net at RN12.2 (R2.1): now also J8.a2 (Pin_a2)
- net at RN12.4 (R4.1): now also J9.a6 (Pin_a6)
- net at RN1.4 (R4.1): now also J8.b1 (Pin_b1)
- net at U4.13 (Q6), U5.12 (B6): now also J8.b9 (Pin_b9)
- net at U4.16 (Q3), U5.15 (B3): now also J8.b8 (Pin_b8)
- net at U4.18 (Q1), U5.17 (B1): now also J8.b7 (Pin_b7)
- net at RN2.1 (R1.1): now also J8.b5 (Pin_b5)
- net at RN2.3 (R3.1): now also J8.b4 (Pin_b4)
- net at RN11.8 (R1.2): now also J8.b3 (Pin_b3)
- net at RN1.2 (R2.1): now also J8.b2 (Pin_b2)
- net at RN6.7 (R2.2), TP7.1, U1.102 (PF0): now also TP23.1
- net at RN10.6 (R3.2): now also J9.b10 (Pin_b10)
- net at RN10.7 (R2.2): now also J9.c10 (Pin_c10)
- net at RN10.8 (R1.2): now also J9.b6 (Pin_b6)
- net at U7.17 (Q2), U8.13 (B5): now also J9.c9 (Pin_c9)
- net at U7.12 (Q7), U8.18 (B0): now also J9.c7 (Pin_c7)
- net at U6.12 (Q7): now also J9.c3 (Pin_c3)
- net at U6.13 (Q6): now also J9.a2 (Pin_a2)
- net at U6.14 (Q5): now also J9.b2 (Pin_b2)
- net at U6.15 (Q4): now also J9.c2 (Pin_c2)
- net at U6.16 (Q3): now also J9.b3 (Pin_b3)
- net at U6.17 (Q2): now also J9.a3 (Pin_a3)
- net at U6.18 (Q1): now also J9.c4 (Pin_c4)
- net at U6.19 (Q0): now also J9.b4 (Pin_b4)
- net +BATT: now reaches BT1.1 (+), BT2.1 (+), TP5.1
- net +BATT: now also R2.1, TP22.1
- net at U2.11 (PD7): now also TP24.1
- net at D8.2 (A), U2.19 (ADC6): now also C24.1
- net at RN3.3 (R3.1): now also J8.a6 (Pin_a6)
- net -BATT: now reaches BT1.2 (-), BT2.2 (-), JP1.1 (A), TP3.1
- net at U4.12 (Q7), U5.11 (B7): now also J8.a9 (Pin_a9)
- net at U4.15 (Q4), U5.14 (B4): now also J8.a8 (Pin_a8)
- net at RN2.4 (R4.1): now also J8.a3 (Pin_a3)
- net at U1.85 (EXTAL): now also Y1.4
- net at U1.96 (PF6): now also D10.1 (A), R7.2
- net at D4.1 (A), D4.2 (A): now also Q3.3 (D)
- net at RN7.5 (R4.2): now also TP21.1
- new net: D10.3 (K), R5.1
- new net: J9.c5 (Pin_c5), R7.1
- new net: C25.1, R6.2
- new net: Q3.1 (G), Q4.2 (G), Q4.5 (D), Q4.6 (D), R1.2, TP20.1
- new net: Q4.7 (D), Q4.8 (D)
- new net: R5.2, R6.1
- no-connect marks 16 -> 18
Other:
- moved on the sheet: D4, D5

Commit message: vias
Parts:
- added C26, C27: C, Capacitor_SMD:C_0805_2012Metric, symbol Device:C
- added TP25, TP26, TP27, TP28: TestPoint, TestPoint:TestPoint_Pad_D1.0mm, symbol Connector:TestPoint
- Q3: footprint Package_TO_SOT_SMD:SOT-23-3 -> Package_TO_SOT_SMD:SOT-23
- Y1: value Crystal_GND23 -> 32.768k
Connections:
- net GND: now also C27.2
- net SCK: now also RN7.6 (R3.2), U2.17 (PB5), TP25.1
- net VDD: now also D10.3 (K), R5.1
- net at RN12.3 (R3.1): now also U11.11
- net at RN12.8 (R1.2): now also J9.c1 (Pin_c1)
- net at U2.28 (PC5): now also TP27.1
- net at U2.29 (~{RESET}/PC6): now also C26.1, TP26.1
- net at D2.1 (A), U1.3 (FC0): now also U3.40 (~{BHE})
- net at D1.1 (A), U3.39 (~{BLE}): now also U1.4 (FC1)
- net at Q4.7 (D), Q4.8 (D): now also C27.1
- net at D4.3 (K): now also TP28.1
Other:
- moved on the sheet: C25, R5, R6

Commit message: led
Parts:
- removed D6, D7, D8: LED, LED_SMD:LED_ASMB-KTF0-0A306, symbol Device:LED
- added C28, C29: C, Capacitor_SMD:C_0805_2012Metric, symbol Device:C
- added D6, D7: LED_RBGA, LED_SMD:LED_Cree-PLCC4_3.2x2.8mm_CCW, symbol Device:LED_RBGA
- added R8: R, Resistor_SMD:R_0603_1608Metric, symbol Device:R
- added TP29: TestPoint, TestPoint:TestPoint_Pad_D1.0mm, symbol Connector:TestPoint
- R7: value R -> 10k
Connections:
- net GND: now also C24.2, C28.1, C29.1, D6.1 (RK), D6.2 (BK), D6.3 (GK), D7.1 (RK), D7.2 (BK), D7.3 (GK)
- net PF1: now also RN4.7 (R2.2), RN5.5 (R4.2), U1.101 (PF1); no longer J8.a5 (Pin_a5), RN4.2 (R2.1)
- net PQS0: now also RN4.6 (R3.2), RN6.8 (R1.2), U1.65 (PQS0); no longer RN4.3 (R3.1)
- net VDD: now also C29.2
- net PQS4: now reaches RN12.1 (R1.1), U1.69 (PQS4)
- net RW: now reaches RN12.5 (R4.2), U1.103 (R/~{W})
- net cPQS4: now reaches J9.c1 (Pin_c1), RN12.8 (R1.2)
- net BERR: now reaches RN5.6 (R3.2), U1.94 (~{BERR})
- net HALT: now reaches RN5.7 (R2.2), U1.93 (~{HALT})
- net cPQS2: now reaches J8.a6 (Pin_a6), RN3.3 (R3.1)
- net TXD: now reaches RN11.1 (R1.1), U1.75 (PQS7/TXD)
- net CLKOUT: now reaches RN11.2 (R2.1)
- net CLKOUT: now also U1.90 (CLKOUT)
- net at RN11.3 (R3.1): now also R4.1, TP29.1
- net at RN11.6 (R3.2): now also J9.c6 (Pin_c6)
- net at RN11.7 (R2.2): now also R8.1
- net cTXD: now reaches J8.b3 (Pin_b3), RN11.8 (R1.2)
- net FC2: now reaches TP11.1, U1.5 (FC2), U11.12, U11.13, U11.4, U9.1, U9.12, U9.4
- net PF7: now reaches RN13.1 (R1.1), U1.95 (PF7)
- net PF2: now reaches RN10.3 (R3.1), RN13.2 (R2.1), U1.100 (PF2)
- net PF3: now reaches RN10.2 (R2.1), RN13.3 (R3.1), U1.99 (PF3)
- net PF0: now reaches RN6.7 (R2.2), TP23.1, TP7.1, U1.102 (PF0)
- net cPF2: now reaches J9.b10 (Pin_b10), RN10.6 (R3.2)
- net cPF3: now reaches J9.c10 (Pin_c10), RN10.7 (R2.2)
- net at U7.19 (Q0), U8.11 (B7): now also J9.a9 (Pin_a9)
- net at U7.18 (Q1), U8.12 (B6): now also J9.b9 (Pin_b9)
- net at U7.16 (Q3), U8.14 (B4): now also J9.a8 (Pin_a8)
- net at U7.15 (Q4), U8.15 (B3): now also J9.b8 (Pin_b8)
- net at U7.14 (Q5), U8.16 (B2): now also J9.c8 (Pin_c8)
- net at U7.13 (Q6), U8.17 (B1): now also J9.b7 (Pin_b7)
- net 12Vin: now reaches D10.1 (A), R7.2, U1.96 (PF6)
- net cPQS5: now reaches J8.b1 (Pin_b1), RN1.4 (R4.1)
- net cA22: now reaches J8.b2 (Pin_b2), RN1.2 (R2.1)
- net cPQS0: now reaches J8.b6 (Pin_b6)
- net cPQS0: now also RN4.3 (R3.1)
- net RXD: now reaches RN2.7 (R2.2), RN8.1 (R1.1), U1.76 (RXD)
- net cCLKOUT: now reaches J9.a5 (Pin_a5)
- net cCLKOUT: now also R8.2
- net c12V: now reaches J9.c5 (Pin_c5), R7.1
- net at U2.20 (AREF): now also C28.2
- net FC0: now reaches D2.1 (A), U1.3 (FC0), U3.40 (~{BHE})
- net FC1: now reaches D1.1 (A), U1.4 (FC1), U3.39 (~{BLE})
- net cPQS1: now reaches J8.c6 (Pin_c6), RN3.1 (R1.1)
- net cA20: now reaches J8.c10 (Pin_c10), RN3.2 (R2.1)
- net PQS2: now reaches RN3.6 (R3.2)
- net PQS2: now also U1.67 (PQS2)
- net PQS1: now reaches RN3.8 (R1.2)
- net PQS1: now also U1.66 (PQS1)
- net at RN9.6 (R3.2): now also U1.80 (TSC)
- net cPQS6: now reaches J8.c1 (Pin_c1), RN1.3 (R3.1)
- net cRXD: now reaches J8.c4 (Pin_c4), RN2.2 (R2.1)
- net PF4: now reaches RN2.6 (R3.2)
- net PF4: now also U1.98 (PF4)
- net CS0: now reaches U1.141 (~{CS0})
- net PGP7: now reaches U1.23 (PGP7)
- net PGP6: now reaches U1.24 (PGP6)
- net PGP5: now reaches U1.28 (PGP5)
- net PGP4: now reaches U1.29 (PGP4)
- net PGP0: now reaches U1.33 (PGP0)
- net PQS3: now reaches U1.68 (PQS3)
- net PQS5: now reaches U1.70 (PQS5)
- net PQS5: now also RN1.5 (R4.2)
- net PQS6: now reaches RN1.6 (R3.2), U1.71 (PQS6)
- net RESET: now reaches U1.92 (~{RESET})
- net PF5: now reaches U1.97 (PF5)
- new net cPF1: J8.a5 (Pin_a5), RN4.2 (R2.1)
- no-connect marks 18 -> 20
Other:
- moved on the sheet: R4, RN4, RN8

Commit message: widerstand
Parts:
- added C30, C31, C32, C33, C34, C35, C36, C37, C39: C, Capacitor_SMD:C_0805_2012Metric, symbol Device:C
- added C38: C, Capacitor_SMD:C_1206_3216Metric, symbol Device:C
- added D11, D8: BAS28, Package_TO_SOT_SMD:SOT-143, symbol DualDiode:BAS28
- added FID2, FID3: Fiducial, Fiducial:Fiducial_0.75mm_Mask2.25mm, symbol Mechanical:Fiducial
- added R10, R11, R16, R17, R18, R19, R20, R21, R9: ~, Resistor_SMD:R_0603_1608Metric, symbol Device:R
- added R12, R13, R15: R, Resistor_SMD:R_0603_1608Metric, symbol Device:R
- added R14: R, Resistor_SMD:R_1206_3216Metric, symbol Device:R
- added TP30, TP34, TP35: TestPoint, TestPoint:TestPoint_Pad_D1.0mm, symbol Connector:TestPoint
- added TP31, TP33: TestPoint, TestPoint:TestPoint_Pad_1.0x1.0mm, symbol Connector:TestPoint
- added TP32: TestPoint, TestPoint:TestPoint_Pad_D1.5mm, symbol Connector:TestPoint
Connections:
- net D2: now also TP33.1
- net D3: now also R15.1
- net GND: now also C30.1, C32.2, C33.2, C34.2, C35.2, C36.2, C37.2, R21.2, TP31.1, TP32.1
- net MOSI: now also D8.1 (K)
- net PF5: now also RN2.5 (R4.2), RN8.2 (R2.1)
- net PGP4: now also D8.3 (A)
- net PGP5: now also D8.4 (A)
- net PGP6: now also D11.4 (A)
- net PGP7: now also D11.3 (A)
- net PQS3: now also RN11.4 (R4.1)
- net RESET: now also R4.1, RN11.3 (R3.1), TP29.1
- net SCK: now also D8.2 (K)
- net VDD: now also C30.2, C31.1, C33.1, C34.1, C36.1, C39.1, TP34.1
- net FREEZE: now reaches TP1.1, U1.81 (FREEZE/QUOT), U2.14 (PB2)
- net cRW: now reaches J9.a6 (Pin_a6), RN12.4 (R4.1)
- net at C24.1, U2.19 (ADC6): now also R11.1
- net at R8.1, RN11.7 (R2.2): now also C35.1
- net cPF5: now reaches J8.a3 (Pin_a3), RN2.4 (R4.1)
- net cD11: now reaches J8.a8 (Pin_a8), U4.15 (Q4), U5.14 (B4)
- net cD8: now reaches J8.a9 (Pin_a9), U4.12 (Q7), U5.11 (B7)
- net at RN7.7 (R2.2), U10.8 (CE), U2.13 (PB1): now also D11.1 (K)
- net cPQS3: now reaches RN11.5 (R4.2)
- net cRESET: now reaches J9.c6 (Pin_c6), RN11.6 (R3.2)
- net PE1: now reaches RN10.1 (R1.1), RN13.4 (R4.1), U1.113 (PE1)
- net cPE1: now reaches J9.b6 (Pin_b6), RN10.8 (R1.2)
- net cD0: now reaches J9.a9 (Pin_a9), U7.19 (Q0), U8.11 (B7)
- net cD1: now reaches J9.b9 (Pin_b9), U7.18 (Q1), U8.12 (B6)
- net cD2: now reaches J9.c9 (Pin_c9), U7.17 (Q2), U8.13 (B5)
- net cD3: now reaches J9.a8 (Pin_a8), U7.16 (Q3), U8.14 (B4)
- net cD4: now reaches J9.b8 (Pin_b8), U7.15 (Q4), U8.15 (B3)
- net cD5: now reaches J9.c8 (Pin_c8), U7.14 (Q5), U8.16 (B2)
- net cD6: now reaches J9.b7 (Pin_b7), U7.13 (Q6), U8.17 (B1)
- net cD7: now reaches J9.c7 (Pin_c7), U7.12 (Q7), U8.18 (B0)
- net PE4: now reaches U1.106 (PE4), U6.11 (Load)
- net cA5: now reaches J9.c3 (Pin_c3), U6.12 (Q7)
- net cA6: now reaches J9.a2 (Pin_a2), U6.13 (Q6)
- net cA7: now reaches J9.b2 (Pin_b2), U6.14 (Q5)
- net cA8: now reaches J9.c2 (Pin_c2), U6.15 (Q4)
- net cA3: now reaches J9.b3 (Pin_b3), U6.16 (Q3)
- net cA2: now reaches J9.a3 (Pin_a3), U6.17 (Q2)
- net cA1: now reaches J9.c4 (Pin_c4), U6.18 (Q1)
- net cA0: now reaches J9.b4 (Pin_b4), U6.19 (Q0)
- net cD14: now reaches J8.b7 (Pin_b7), U4.18 (Q1), U5.17 (B1)
- net cD12: now reaches J8.b8 (Pin_b8), U4.16 (Q3), U5.15 (B3)
- net cD9: now reaches J8.b9 (Pin_b9), U4.13 (Q6), U5.12 (B6)
- net DSO: now reaches U1.77 (DSO), U2.10 (PD6)
- net at TP24.1, U2.11 (PD7): now also R19.1
- net at U2.22 (ADC7): now also R20.1, R21.1
- net DSCLK: now reaches RN9.1 (R1.1), TP4.1, U1.79 (DSCLK), U2.23 (PC0)
- net at TP18.1, U2.24 (PC1): now also R18.1
- net at U2.25 (PC2): now also R16.1, R17.1, TP35.1
- net DSI: now reaches RN9.2 (R2.1), TP2.1, U1.78 (DSI), U2.26 (PC3)
- net at TP19.1, U2.31 (PD1): now also R10.1, R9.1
- net cD10: now reaches J8.c9 (Pin_c9), U4.14 (Q5), U5.13 (B5)
- net cD13: now reaches J8.c8 (Pin_c8), U4.17 (Q2), U5.16 (B2)
- net cD15: now reaches J8.c7 (Pin_c7), U4.19 (Q0), U5.18 (B0)
- net at RN7.5 (R4.2), TP21.1: now also D11.2 (K)
- net TSC: now reaches RN9.6 (R3.2), U1.80 (TSC)
- net TSC: now also TP30.1
- net at C26.2: now also R16.2
- net at Y1.1: now also C32.1, R12.1
- net at U1.85 (EXTAL), Y1.4: now also C37.1, R14.2
- net PE2: now reaches RN6.5 (R4.2), TP6.1, U1.112 (PE2)
- net PE7: now reaches U1.104 (PE7)
- net PE6: now reaches U1.105 (PE6)
- net PE5: now reaches U1.110 (PE5)
- net PE3: now reaches U1.111 (PE3)
- net PE0: now reaches RN6.6 (R3.2), U1.114 (PE0)
- net at U1.83 (XTAL): now also R12.2, R14.1
- net XFC: now reaches U1.87 (XFC)
- net XFC: now also C31.2, R13.1
- new net: C39.2, R13.2
- new net: R18.2, R19.2
Other:
- moved on the sheet: FID1, R4, R8, RN11, RN7, TP12, TP18, TP21, TP24, TP29
