File: DB1MBRedesign/DB1MB.kicad_sch (KiCad schematic)
At the start: 147 parts, among them J7 Conn_01x04_Socket, J8 DIN41612_03x10_ABC, J9 DIN41612_03x10_ABC, Q1 Q_Photo_NPN_CBE, Q2 Q_Photo_NPN_CBE, Q3 BSS84, Q4 IRF7313, U1 MC68331, U11 74LS08, U2 ATmega48V-10A, U3 CY62157, U4 74LS573, U5 74LS245, U6 74LS573, U7 74LS573, U8 74LS245, U9 74LS20, Y1 32.768k

Commit message: inner
Parts:
- removed FID3: Fiducial, Fiducial:Fiducial_0.75mm_Mask2.25mm, symbol Mechanical:Fiducial
- added C40: C, Capacitor_SMD:C_1206_3216Metric, symbol Device:C
- added D12, D13: BAS40-06, Package_TO_SOT_SMD:TSOT-23, symbol Device:D_Dual_CommonAnode_KKA
- added Q5: BC807-40W, Package_TO_SOT_SMD:TSOT-23, symbol Transistor_BJT:Q_PNP_BEC
- added Q6: BC846, Package_TO_SOT_SMD:SOT-23, symbol Transistor_BJT:BC846
- added R22: R, Resistor_SMD:R_1206_3216Metric, symbol Device:R
- added R23, R24, R25, R26, R27, R28, R29: ~, Resistor_SMD:R_0603_1608Metric, symbol Device:R
- added TP36: TestPoint, TestPoint:TestPoint_Pad_D1.5mm, symbol Connector:TestPoint
- D10: footprint Package_TO_SOT_SMD:SOT-23 -> Package_TO_SOT_SMD:TSOT-23
- Q3: footprint Package_TO_SOT_SMD:SOT-23 -> Package_TO_SOT_SMD:SOT-23-3
Connections:
- net GND: now also Q6.2 (E), R29.2
- net PF4: now also RN8.3 (R3.1)
- net VDD: now also C38.1, R4.2, RN8.5 (R4.2), RN8.6 (R3.2), RN8.7 (R2.2), RN8.8 (R1.2)
- net cPQS3: now also J9.b1 (Pin_b1)
- net at C24.1, R11.1, U2.19 (ADC6): now also R29.1
- net PD5: now reaches Q2.1 (C), U2.9 (PD5)
- net at Q2.3 (E): now also Q6.1 (B), R28.2
- net PC2: now reaches R16.1, R17.1, TP35.1, U2.25 (PC2)
- net PD1: now reaches R10.1, R9.1, TP19.1, U2.31 (PD1)
- net at D4.3 (K), TP28.1: now also C27.1, Q4.7 (D), Q4.8 (D), Q5.3 (C)
- net PD3: now reaches TP17.1, U2.1 (PD3)
- net PD3: now also D12.1 (K), D12.2 (K), Q6.3 (C)
- net PD7: now reaches R19.1, TP24.1, U2.11 (PD7)
- net PD4: now reaches TP16.1, U2.2 (PD4)
- net PD4: now also R23.1
- net PC1: now reaches R18.1, TP18.1, U2.24 (PC1)
- net PC4: now reaches U2.27 (PC4)
- net PC5: now reaches TP27.1, U2.28 (PC5)
- net PC5: now also R26.2
- net RST: now reaches C26.1, TP26.1, U2.29 (~{RESET}/PC6)
- net RST: now also R27.2
- net PD0: now reaches TP14.1, U2.30 (PD0)
- net PD2: now reaches U2.32 (PD2)
- net PD2: now also R25.2
- net at R11.2: now also R24.1
- net at Q4.4 (G): now also C40.1, R22.1, R23.2, TP36.1
- new net: D13.1 (K), D13.2 (K)
- new net: Q5.1 (B), R26.1
- new net: C40.2, R22.2
- no-connect marks 20 -> 21
Other:
- moved on the sheet: D4, R4, TP26, TP28
