File: DB1MBRedesign/DB1MB.kicad_pcb (KiCad board)
At the start: 4 copper layers, 124.5 x 69.2 mm, 160 parts, among them J7 Conn_01x04_Socket, J8 DIN41612_03x10_ABC, J9 DIN41612_03x10_ABC, Q1 Q_Photo_NPN_CBE, Q2 Q_Photo_NPN_CBE, Q3 BSS84, Q4 IRF7313, Q5 BC807-40W, Q6 BC846, U1 MC68331, U11 74LS08, U2 ATmega48V-10A, U3 CY62157, U4 74LS573, U5 74LS245, U6 74LS573, U7 74LS573, U8 74LS245, U9 74LS20, Y1 32.768k

Commit message: komponenten werte
Parts:
- D9: value D_Zener -> SM6T6V8A; footprint Diode_SMD:D_SOD-123 -> Diode_SMD:D_SMB
- R10, R9: value ~ -> 1k
- R11: value ~ -> 0
- R22: value R -> 10M
- R4: value R -> 1k
- R5: value R -> 100k
- R6: value R -> 21.5k
- RN10: value R_Pack04 -> 750
- RN12: value R_Pack04 -> 330
- RN13: value R_Pack04 -> 822
- TP2: value TestPoint -> DSI
- TP4: value TestPoint -> DSCLK
- moved D9 0.76 mm to (210.4, 88.4)
- moved J7 0.20 mm to (141.7, 94.0)
Connections:
- C40 pad 2: Net-(C40-Pad2) -> GND
- R22 pad 2: Net-(C40-Pad2) -> GND
Routing:
- net /cPQS3: track 88.7 -> 122.0 mm
- net GND: track 686.7 -> 710.2 mm, vias 47 -> 55
- net FC1: track 23.0 -> 45.5 mm, vias 1 -> 2
- net Net-(C40-Pad2): track 18.9 -> 0.00 mm, vias 2 -> 0
- net FC0: track 18.6 -> 34.0 mm, vias 2 -> 3
- net /cPQS0: track 8.76 -> 24.1 mm
- net RESET: track 57.1 -> 62.4 mm, vias 1 -> 2
- added copper zone on In1.Cu, net GND
- added copper zone on In2.Cu, net VDD

Commit message: rtc
Routing:
- net A0: track 6.21 -> 56.2 mm, vias 1 -> 2
- net A1: track 8.37 -> 45.5 mm
- net A3: track 10.2 -> 46.6 mm
- net A2: track 8.06 -> 43.4 mm
- net GND: track 710.2 -> 726.3 mm
- net VDD: track 420.1 -> 427.2 mm
- net Net-(U1-EXTAL): track 7.98 -> 12.4 mm
- net PQS3: track 13.5 -> 14.9 mm
- net PD7: track 26.6 -> 28.0 mm
- net Net-(U2-ADC6): track 14.1 -> 15.2 mm
- net Net-(Q4B-G): track 12.3 -> 13.4 mm
- net Net-(U2-ADC7): track 8.21 -> 9.29 mm
- net Net-(Q3-G): track 20.1 -> 21.0 mm
- net PD1: track 37.4 -> 38.3 mm
- net PD3: track 12.0 -> 12.9 mm
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
Commit message: drc
Routing:
- net GND: track 726.3 -> 706.0 mm
- net Net-(D13-K-Pad1): track 14.2 -> 1.90 mm
- net VDD: track 427.2 -> 416.0 mm
- net RESET: track 62.4 -> 59.0 mm
- net Net-(Q4B-G): track 13.4 -> 10.7 mm
- net Net-(Q3-G): track 21.0 -> 18.6 mm
- net Net-(Q3-S): track 9.86 -> 7.41 mm
- net D9: track 32.3 -> 29.9 mm
- net D6: track 48.7 -> 46.7 mm
- net CS0: track 2.04 -> 0.00 mm
- net D13: track 37.8 -> 35.8 mm
- net D11: track 35.8 -> 33.8 mm
- net D3: track 53.1 -> 51.3 mm
- net D5: track 47.4 -> 45.6 mm
- net Net-(U2-ADC6): track 15.2 -> 13.5 mm
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
Commit message: led
Connections:
- net Net-(J8C-Pin_c2) renamed /cA23
- D6 pad 4: unconnected-(D6-A-Pad4) -> LED_R
- D7 pad 4: unconnected-(D7-A-Pad4) -> LED_L
- R10 pad 2: unconnected-(R10-Pad2) -> LED_L
- R9 pad 2: unconnected-(R9-Pad2) -> LED_R
- U11 pad 1: Net-(U11-Pad1) -> A23
- U11 pad 2: Net-(U11-Pad1) -> A23
- U8 pad 1: unconnected-(U8-A->B-Pad1) -> GND
- U9 pad 9: Net-(U11-Pad1) -> A23
Routing:
- net Net-(U11-Pad1): track 19.4 -> 0.00 mm, vias 1 -> 0
- net A23: track 1.88 -> 21.3 mm, vias 1 -> 2
- net LED_L: track 0.00 -> 17.5 mm, vias 0 -> 2
- net unconnected-(R10-Pad2): track 15.5 -> 0.00 mm, vias 1 -> 0
- net LED_R: track 0.00 -> 10.1 mm, vias 0 -> 2
- net unconnected-(R9-Pad2): track 7.96 -> 0.00 mm, vias 1 -> 0
- net unconnected-(D6-A-Pad4): track 2.15 -> 0.00 mm, vias 1 -> 0
- net unconnected-(D7-A-Pad4): track 1.98 -> 0.00 mm, vias 1 -> 0
- net unconnected-(U8-A->B-Pad1): track 1.27 -> 0.00 mm, vias 1 -> 0
- net GND: track 706.0 -> 707.3 mm, vias 55 -> 56
