File: Zulassungskarte/Zulassungskarte.kicad_sch (KiCad schematic)
At the start: 28 parts, among them J1 Conn_02x04_Counter_Clockwise, J2 Conn_02x04_Counter_Clockwise, U1 ATmega48-20A

Commit message: we
Parts:
- added D1: ~, Package_SO:SO-8_3.9x4.9mm_P1.27mm, symbol Protection:ESDA6V1U1
- added D2: D, Diode_SMD:D_SOD-123, symbol Device:D
- added FID1, FID2: Fiducial, Fiducial:Fiducial_1.5mm_Mask3mm, symbol Mechanical:Fiducial
- added R7: 1002, Resistor_SMD:R_0805_2012Metric, symbol Device:R
- R2, R3, R5: value R -> 4640
- TP1, TP10: value TestPoint -> MISO
- TP11, TP2: value TestPoint -> GND
- TP12: value TestPoint -> AREF
- TP13: value TestPoint -> ~{RESET}
- TP14: value TestPoint -> XTAL1
- TP15: value TestPoint -> XTAL2
- TP16: value TestPoint -> VCC
- TP3: value TestPoint -> RST
- TP4, TP5: value TestPoint -> MOSI
- TP6, TP9: value TestPoint -> SCK
- TP7: value TestPoint -> I/O6
- TP8: value TestPoint -> 12V
Connections:
- net GND: now also TP11.1, U1.19 (ADC6), D1.6 (GND), D1.7 (GND), D2.2 (A), R7.1
- net MISO: now also R2.1, D1.3 (I/O_3)
- net MOSI: now also R1.1, D1.4 (I/O_4)
- net RST: now also D1.1 (I/O_1)
- net SCK: now also R3.1, D1.2 (I/O_2)
- net VCC: now also C3.1, R6.2, U1.18 (AVCC), D1.5 (I/O_5), D2.1 (K); no longer J1.1 (Pin_1), J2.1 (Pin_1), R6.1, TP8.1
- net at R1.2: now also TP4.1, U1.15 (PB3), R7.2
- net at TP12.1: now also U1.20 (AREF)
- net at TP10.1: now also R2.2, U1.16 (PB4)
- net at R3.2: now also TP6.1, U1.17 (PB5)
- net at TP7.1: now also D1.8 (I/O_6)
- new net +12V: J1.1 (Pin_1), J2.1 (Pin_1), R6.1, TP8.1
- no-connect marks 4 -> 7
Other:
- moved on the sheet: C3, J1, J2, R1, R2, R3, TP10, TP11, TP12, TP4, TP6, TP7

Commit message: ordentlicher scan
Parts:
- removed FID1, FID2: Fiducial, Fiducial:Fiducial_1.5mm_Mask3mm, symbol Mechanical:Fiducial
- C1, C2, C3: footprint Capacitor_SMD:C_0805_2012Metric -> Capacitor_SMD:C_0805_2012Metric_Pad1.18x1.45mm_HandSolder
- D2: footprint Diode_SMD:D_SOD-123 -> Diode_SMD:D_1206_3216Metric
- R1, R2, R3: footprint Resistor_SMD:R_0805_2012Metric -> Resistor_SMD:R_0603_1608Metric_Pad0.98x0.95mm_HandSolder
- R4, R5, R6, R7: footprint Resistor_SMD:R_0805_2012Metric -> Resistor_SMD:R_0805_2012Metric_Pad1.20x1.40mm_HandSolder
- TP10, TP12: footprint TestPoint:TestPoint_Pad_D1.5mm -> TestPoint:TestPoint_Pad_D1.0mm
Connections:
- net GND: no longer R7.1
- net VCC: now also R7.1
- net at U1.12 (PB0): now also U1.13 (PB1), U1.14 (PB2)
- no-connect marks 7 -> 4
Changed lines of the file:
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@@
 	)
 	(junction
+		(at 87.63 59.69)
+		(diameter 0)
+		(color 0 0 0 0)
+	)
+	(junction
 		(at 74.93 49.53)
 		(diameter 0)
@@
 	)
 	(no_connect
-		(at 87.63 59.69)
-	)
-	(no_connect
 		(at 90.17 29.21)
 	)
@@
 	)
 	(no_connect
-		(at 87.63 62.23)
-	)
-	(no_connect
 		(at 45.72 29.21)
 	)
-	(no_connect
-		(at 87.63 57.15)
-	)
 	(wire
 		(pts
@@
 	(wire
 		(pts
+			(xy 87.63 57.15) (xy 87.63 59.69)
+		)
+		(stroke
+			(width 0)
+			(type default)
+		)
+	)
+	(wire
+		(pts
 			(xy 144.78 69.85) (xy 87.63 69.85)
 		)
@@
 	(wire
 		(pts
+			(xy 87.63 59.69) (xy 87.63 62.23)
+		)
+		(stroke
+			(width 0)
+			(type default)
+		)
+	)
+	(wire
+		(pts
 			(xy 153.67 110.49) (xy 144.78 110.49)
 		)
@@
 			)
 		)
-		(property "Footprint" "Resistor_SMD:R_0805_2012Metric"
+		(property "Footprint" "Resistor_SMD:R_0603_1608Metric_Pad0.98x0.95mm_HandSolder"
 			(at 157.48 117.348 90)
 			(effects
@@
 			)
 		)
-		(property "Footprint" "TestPoint:TestPoint_Pad_D1.5mm"
+		(property "Footprint" "TestPoint:TestPoint_Pad_D1.0mm"
 			(at 52.07 57.15 0)
 			(effects
@@
 			)
 		)
-		(property "Footprint" "TestPoint:TestPoint_Pad_D1.5mm"
+		(property "Footprint" "TestPoint:TestPoint_Pad_D1.0mm"
 			(at 104.14 67.31 0)
 			(effects
@@
 	(symbol
 		(lib_id "power:GND")
-		(at 157.48 97.79 90)
-		(unit 1)
-		(exclude_from_sim no)
-		(in_bom yes)
-		(on_board yes)
-		(dnp no)
-		(fields_autoplaced yes)
-		(property "Reference" "#PWR025"
-			(at 163.83 97.79 0)
-			(effects
-				(font
-					(size 1.27 1.27)
-				)
-				(hide yes)
-			)
-		)
-		(property "Value" "GND"
-			(at 161.29 97.7899 90)
-			(effects
-				(font
-					(size 1.27 1.27)
-				)
-				(justify right)
-			)
-		)
-		(property "Footprint" ""
-			(at 157.48 97.79 0)
-			(effects
-				(font
-					(size 1.27 1.27)
-				)
-				(hide yes)
-			)
-		)
-		(property "Datasheet" ""
-			(at 157.48 97.79 0)
-			(effects
-				(font
-					(size 1.27 1.27)
-				)
-				(hide yes)
-			)
-		)
-		(property "Description" "Power symbol creates a global label with name \"GND\" , ground"
-			(at 157.48 97.79 0)
-			(effects
-				(font
-					(size 1.27 1.27)
-				)
-				(hide yes)
-			)
-		)
-		(pin "1"
-		)
-		(instances
-			(project "Zulassungskarte"
-				(path "/f437cf05-d297-460e-8639-991b777c08ac"
-					(reference "#PWR025")
-					(unit 1)
-				)
-			)
-		)
-	)
-	(symbol
-		(lib_id "power:GND")
 		(at 87.63 86.36 90)
 		(unit 1)
@@
 			)
 		)
-		(property "Footprint" "Resistor_SMD:R_0805_2012Metric"
+		(property "Footprint" "Resistor_SMD:R_0603_1608Metric_Pad0.98x0.95mm_HandSolder"
 			(at 157.48 112.268 90)
 			(effects
@@
 			)
 		)
-		(property "Footprint" "Resistor_SMD:R_0805_2012Metric"
+		(property "Footprint" "Resistor_SMD:R_0805_2012Metric_Pad1.20x1.40mm_HandSolder"
 			(at 114.3 103.378 90)
 			(effects
@@
 			)
 		)
-		(property "Footprint" "Resistor_SMD:R_0805_2012Metric"
+		(property "Footprint" "Resistor_SMD:R_0805_2012Metric_Pad1.20x1.40mm_HandSolder"
 			(at 137.16 123.698 90)
 			(effects
@@
 			)
 		)
-		(property "Footprint" "Capacitor_SMD:C_0805_2012Metric"
+		(property "Footprint" "Capacitor_SMD:C_0805_2012Metric_Pad1.18x1.45mm_HandSolder"
 			(at 119.0752 109.22 0)
 			(effects
@@
 	)
 	(symbol
-		(lib_id "Mechanical:Fiducial")
-		(at 19.05 26.67 0)
-		(unit 1)
-		(exclude_from_sim yes)
-		(in_bom no)
-		(on_board yes)
-		(dnp no)
-		(fields_autoplaced yes)
-		(property "Reference" "FID1"
-			(at 21.59 25.3999 0)
-			(effects
-				(font
-					(size 1.27 1.27)
-				)
-				(justify left)
-			)
-		)
-		(property "Value" "Fiducial"
-			(at 21.59 27.9399 0)
-			(effects
-				(font
-					(size 1.27 1.27)
-				)
-				(justify left)
-			)
-		)
-		(property "Footprint" "Fiducial:Fiducial_1.5mm_Mask3mm"
-			(at 19.05 26.67 0)
-			(effects
-				(font
-					(size 1.27 1.27)
-				)
-				(hide yes)
-			)
-		)
-		(property "Datasheet" "~"
-			(at 19.05 26.67 0)
-			(effects
-				(font
-					(size 1.27 1.27)
-				)
-				(hide yes)
-			)
-		)
-		(property "Description" "Fiducial Marker"
-			(at 19.05 26.67 0)
-			(effects
-				(font
-					(size 1.27 1.27)
-				)
-				(hide yes)
-			)
-		)
-		(instances
-			(project ""
-				(path "/f437cf05-d297-460e-8639-991b777c08ac"
-					(reference "FID1")
-					(unit 1)
-				)
-			)
-		)
-	)
-	(symbol
 		(lib_id "power:GND")
 		(at 199.39 111.76 90)
@@
 			)
 		)
-		(property "Footprint" "Diode_SMD:D_SOD-123"
+		(property "Footprint" "Diode_SMD:D_1206_3216Metric"
 			(at 74.93 45.72 0)
 			(effects
@@
 			)
 		)
-		(property "Footprint" "Resistor_SMD:R_0805_2012Metric"
+		(property "Footprint" "Resistor_SMD:R_0805_2012Metric_Pad1.20x1.40mm_HandSolder"
 			(at 153.67 99.568 90)
 			(effects
@@
 	(symbol
 		(lib_id "power:VCC")
+		(at 157.48 97.79 270)
+		(unit 1)
+		(exclude_from_sim no)
+		(in_bom yes)
+		(on_board yes)
+		(dnp no)
+		(fields_autoplaced yes)
+		(property "Reference" "#PWR025"
+			(at 153.67 97.79 0)
+			(effects
+				(font
+					(size 1.27 1.27)
+				)
+				(hide yes)
+			)
+		)
+		(property "Value" "VCC"
+			(at 161.29 97.7899 90)
+			(effects
+				(font
+					(size 1.27 1.27)
+				)
+				(justify left)
+			)
+		)
+		(property "Footprint" ""
+			(at 157.48 97.79 0)
+			(effects
+				(font
+					(size 1.27 1.27)
+				)
+				(hide yes)
+			)
+		)
+		(property "Datasheet" ""
+			(at 157.48 97.79 0)
+			(effects
+				(font
+					(size 1.27 1.27)
+				)
+				(hide yes)
+			)
+		)
+		(property "Description" "Power symbol creates a global label with name \"VCC\""
+			(at 157.48 97.79 0)
+			(effects
+				(font
+					(size 1.27 1.27)
+				)
+				(hide yes)
+			)
+		)
+		(pin "1"
+		)
+		(instances
+			(project "Zulassungskarte"
+				(path "/f437cf05-d297-460e-8639-991b777c08ac"
+					(reference "#PWR025")
+					(unit 1)
+				)
+			)
+		)
+	)
+	(symbol
+		(lib_id "power:VCC")
 		(at 140.97 121.92 270)
 		(unit 1)
@@
 			)
 		)
-		(property "Footprint" "Capacitor_SMD:C_0805_2012Metric"
+		(property "Footprint" "Capacitor_SMD:C_0805_2012Metric_Pad1.18x1.45mm_HandSolder"
 			(at 96.52 48.5648 0)
 			(effects
@@
 			)
 		)
-		(property "Footprint" "Capacitor_SMD:C_0805_2012Metric"
+		(property "Footprint" "Capacitor_SMD:C_0805_2012Metric_Pad1.18x1.45mm_HandSolder"
 			(at 160.9852 62.23 0)
 			(effects
@@
 			)
 		)
-		(property "Footprint" "Resistor_SMD:R_0805_2012Metric"
+		(property "Footprint" "Resistor_SMD:R_0805_2012Metric_Pad1.20x1.40mm_HandSolder"
 			(at 121.92 103.378 90)
 			(effects
@@
 			)
 		)
-		(property "Footprint" "Resistor_SMD:R_0805_2012Metric"
+		(property "Footprint" "Resistor_SMD:R_0603_1608Metric_Pad0.98x0.95mm_HandSolder"
 			(at 157.48 114.808 90)
 			(effects
@@
 					(unit 1)
 				)
-			)
-		)
-	)
-	(symbol
-		(lib_id "Mechanical:Fiducial")
-		(at 19.05 33.02 0)
-		(unit 1)
-		(exclude_from_sim yes)
-		(in_bom no)
-		(on_board yes)
-		(dnp no)
-		(fields_autoplaced yes)
-		(property "Reference" "FID2"
-			(at 21.59 31.7499 0)
-			(effects
-				(font
-					(size 1.27 1.27)
-				)
-				(justify left)
-			)
-		)
-		(property "Value" "Fiducial"
-			(at 21.59 34.2899 0)
-			(effects
-				(font
-					(size 1.27 1.27)
-				)
-				(justify left)
-			)
-		)
-		(property "Footprint" "Fiducial:Fiducial_1.5mm_Mask3mm"
-			(at 19.05 33.02 0)
-			(effects
-				(font
-					(size 1.27 1.27)
-				)
-				(hide yes)
-			)
-		)
-		(property "Datasheet" "~"
-			(at 19.05 33.02 0)
-			(effects
-				(font
-					(size 1.27 1.27)
-				)
-				(hide yes)
-			)
-		)
-		(property "Description" "Fiducial Marker"
-			(at 19.05 33.02 0)
-			(effects
-				(font
-					(size 1.27 1.27)
-				)
-				(hide yes)
-			)
-		)
-		(instances
-			(project "Zulassungskarte"
-				(path "/f437cf05-d297-460e-8639-991b777c08ac"
-					(reference "FID2")
-					(unit 1)
-				)

Commit message: rueckseite maske
Parts:
- C1: value C -> 100nF
- C2: renamed from C3; value C -> 100nF
- C3: renamed from C2; value C -> 100nF
- D1: renamed from D2; value D -> 500mW 4.7V; footprint Diode_SMD:D_1206_3216Metric -> Diode_SMD:D_SOD-123
- D2: renamed from D1; value ~ -> ESDA6V1U1
- J1: renamed from J2; now left out of the parts list
- J2: renamed from J1; now left out of the parts list
- R1: renamed from R6; value R -> 270; footprint Resistor_SMD:R_0805_2012Metric_Pad1.20x1.40mm_HandSolder -> Resistor_SMD:R_0603_1608Metric_Pad0.98x0.95mm_HandSolder
- R2: value 4640 -> 470
- R3: renamed from R1; value R -> 470
- R4: value R -> 470; footprint Resistor_SMD:R_0805_2012Metric_Pad1.20x1.40mm_HandSolder -> Resistor_SMD:R_0603_1608Metric_Pad0.98x0.95mm_HandSolder
- R5: value 4640 -> 470; footprint Resistor_SMD:R_0805_2012Metric_Pad1.20x1.40mm_HandSolder -> Resistor_SMD:R_0603_1608Metric_Pad0.98x0.95mm_HandSolder
- R6: renamed from R3; value 4640 -> 470
- R7: value 1002 -> 10k; footprint Resistor_SMD:R_0805_2012Metric_Pad1.20x1.40mm_HandSolder -> Resistor_SMD:R_0603_1608Metric_Pad0.98x0.95mm_HandSolder
- U1: value ATmega48-20A -> ATmega48V-10AU
Other:
- moved on the sheet: R2, R3
Changed lines of the file:
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@@
 (kicad_sch
-	(version 20231120)
+	(version 20250114)
 	(generator "eeschema")
-	(generator_version "8.0")
+	(generator_version "9.0")
 	(paper "A4")
 	(junction
@@
 	(wire
 		(pts
-			(xy 153.67 113.03) (xy 147.32 113.03)
+			(xy 157.48 113.03) (xy 147.32 113.03)
 		)
 		(stroke
@@
 	(wire
 		(pts
+			(xy 160.02 115.57) (xy 153.67 115.57)
+		)
+		(stroke
+			(width 0)
+			(type default)
+		)
+	)
+	(wire
+		(pts
 			(xy 87.63 86.36) (xy 87.63 87.63)
 		)
@@
 	(wire
 		(pts
-			(xy 161.29 113.03) (xy 173.99 113.03)
+			(xy 165.1 113.03) (xy 173.99 113.03)
 		)
 		(stroke
@@
 	(wire
 		(pts
-			(xy 161.29 115.57) (xy 173.99 115.57)
+			(xy 167.64 115.57) (xy 173.99 115.57)
 		)
 		(stroke
@@
 	(symbol
 		(lib_id "Device:R")
-		(at 157.48 115.57 270)
-		(mirror x)
+		(at 163.83 115.57 270)
 		(unit 1)
 		(exclude_from_sim no)
@@
 		(on_board yes)
 		(dnp no)
-		(property "Reference" "R1"
-			(at 157.48 109.22 90)
+		(property "Reference" "R3"
+			(at 163.83 121.92 90)
 			(effects
 				(font
@@
 			)
 		)
-		(property "Value" "R"
-			(at 157.48 111.76 90)
+		(property "Value" "470"
+			(at 163.83 119.38 90)
 			(effects
 				(font
@@
 		)
 		(property "Footprint" "Resistor_SMD:R_0603_1608Metric_Pad0.98x0.95mm_HandSolder"
-			(at 157.48 117.348 90)
+			(at 163.83 113.792 90)
 			(effects
 				(font
@@
 		)
 		(property "Datasheet" "~"
-			(at 157.48 115.57 0)
+			(at 163.83 115.57 0)
 			(effects
 				(font
@@
 		)
 		(property "Description" "Resistor"
-			(at 157.48 115.57 0)
+			(at 163.83 115.57 0)
 			(effects
 				(font
@@
 			(project ""
 				(path "/f437cf05-d297-460e-8639-991b777c08ac"
-					(reference "R1")
+					(reference "R3")
 					(unit 1)
 				)
@@
 		(unit 1)
 		(exclude_from_sim no)
-		(in_bom yes)
+		(in_bom no)
 		(on_board yes)
 		(dnp no)
 		(fields_autoplaced yes)
-		(property "Reference" "J1"
+		(property "Reference" "J2"
 			(at 52.07 15.24 0)
 			(effects
@@
 			(project ""
 				(path "/f437cf05-d297-460e-8639-991b777c08ac"
-					(reference "J1")
+					(reference "J2")
 					(unit 1)
 				)
@@
 		(unit 1)
 		(exclude_from_sim no)
-		(in_bom yes)
+		(in_bom no)
 		(on_board yes)
 		(dnp no)
 		(fields_autoplaced yes)
-		(property "Reference" "J2"
+		(property "Reference" "J1"
 			(at 83.82 15.24 0)
 			(effects
@@
 			(project "Zulassungskarte"
 				(path "/f437cf05-d297-460e-8639-991b777c08ac"
-					(reference "J2")
+					(reference "J1")
 					(unit 1)
 				)
@@
 		(on_board yes)
 		(dnp no)
-		(property "Reference" "R3"
+		(property "Reference" "R6"
 			(at 157.48 104.14 90)
 			(effects
@@
 			)
 		)
-		(property "Value" "4640"
+		(property "Value" "470"
 			(at 157.48 106.68 90)
 			(effects
@@
 			(project "Zulassungskarte"
 				(path "/f437cf05-d297-460e-8639-991b777c08ac"
-					(reference "R3")
+					(reference "R6")
 					(unit 1)
 				)
@@
 			)
 		)
-		(property "Value" "R"
+		(property "Value" "470"
 			(at 114.3 97.79 90)
 			(effects
@@
 			)
 		)
-		(property "Footprint" "Resistor_SMD:R_0805_2012Metric_Pad1.20x1.40mm_HandSolder"
+		(property "Footprint" "Resistor_SMD:R_0603_1608Metric_Pad0.98x0.95mm_HandSolder"
 			(at 114.3 103.378 90)
 			(effects
@@
 		(dnp no)
 		(fields_autoplaced yes)
-		(property "Reference" "R6"
+		(property "Reference" "R1"
 			(at 137.16 115.57 90)
 			(effects
@@
 			)
 		)
-		(property "Value" "R"
+		(property "Value" "270"
 			(at 137.16 118.11 90)
 			(effects
@@
 			)
 		)
-		(property "Footprint" "Resistor_SMD:R_0805_2012Metric_Pad1.20x1.40mm_HandSolder"
+		(property "Footprint" "Resistor_SMD:R_0603_1608Metric_Pad0.98x0.95mm_HandSolder"
 			(at 137.16 123.698 90)
 			(effects
@@
 			(project "Zulassungskarte"
 				(path "/f437cf05-d297-460e-8639-991b777c08ac"
-					(reference "R6")
+					(reference "R1")
 					(unit 1)
 				)
@@
 		(dnp no)
 		(fields_autoplaced yes)
-		(property "Reference" "C2"
+		(property "Reference" "C3"
 			(at 121.92 104.1399 0)
 			(effects
@@
 			)
 		)
-		(property "Value" "C"
+		(property "Value" "100nF"
 			(at 121.92 106.6799 0)
 			(effects
@@
 			(project "Zulassungskarte"
 				(path "/f437cf05-d297-460e-8639-991b777c08ac"
-					(reference "C2")
+					(reference "C3")
 					(unit 1)
 				)
@@
 		(fields_autoplaced yes)
 		(property "Reference" "U1"
-			(at 74.5841 125.73 0)
+			(at 74.5333 125.73 0)
 			(effects
 				(font
@@
 			)
 		)
-		(property "Value" "ATmega48-20A"
-			(at 74.5841 128.27 0)
+		(property "Value" "ATmega48V-10AU"
+			(at 74.5333 128.27 0)
 			(effects
 				(font
@@
 		(dnp no)
 		(fields_autoplaced yes)
-		(property "Reference" "D2"
-			(at 81.28 45.72 0)
+		(property "Reference" "D1"
+			(at 77.47 44.4499 90)
 			(effects
 				(font
 					(size 1.27 1.27)
 				)
+				(justify left)
 			)
 		)
-		(property "Value" "D"
-			(at 78.74 45.72 0)
+		(property "Value" "500mW 4.7V"
+			(at 77.47 46.9899 90)
 			(effects
 				(font
 					(size 1.27 1.27)
 				)
+				(justify left)
 			)
 		)
-		(property "Footprint" "Diode_SMD:D_1206_3216Metric"
+		(property "Footprint" "Diode_SMD:D_SOD-123"
 			(at 74.93 45.72 0)
 			(effects
@@
 			(project ""
 				(path "/f437cf05-d297-460e-8639-991b777c08ac"
-					(reference "D2")
+					(reference "D1")
 					(unit 1)
 				)
@@
 			)
 		)
-		(property "Value" "1002"
+		(property "Value" "10k"
 			(at 153.67 93.98 90)
 			(effects
@@
 			)
 		)
-		(property "Footprint" "Resistor_SMD:R_0805_2012Metric_Pad1.20x1.40mm_HandSolder"
+		(property "Footprint" "Resistor_SMD:R_0603_1608Metric_Pad0.98x0.95mm_HandSolder"
 			(at 153.67 99.568 90)
 			(effects
@@
 		(dnp no)
 		(fields_autoplaced yes)
-		(property "Reference" "C3"
-			(at 91.4399 45.72 0)
+		(property "Reference" "C2"
+			(at 92.71 41.91 90)
 			(effects
 				(font
 					(size 1.27 1.27)
 				)
-				(justify left)
 			)
 		)
-		(property "Value" "C"
-			(at 93.9799 45.72 0)
+		(property "Value" "100nF"
+			(at 92.71 44.45 90)
 			(effects
 				(font
 					(size 1.27 1.27)
 				)
-				(justify left)
 			)
 		)
@@
 			(project "Zulassungskarte"
 				(path "/f437cf05-d297-460e-8639-991b777c08ac"
-					(reference "C3")
+					(reference "C2")
 					(unit 1)
 				)
@@
 			)
 		)
-		(property "Value" "C"
+		(property "Value" "100nF"
 			(at 163.83 59.6899 0)
 			(effects
@@
 			)
 		)
-		(property "Value" "4640"
+		(property "Value" "470"
 			(at 121.92 97.79 90)
 			(effects
@@
 			)
 		)
-		(property "Footprint" "Resistor_SMD:R_0805_2012Metric_Pad1.20x1.40mm_HandSolder"
+		(property "Footprint" "Resistor_SMD:R_0603_1608Metric_Pad0.98x0.95mm_HandSolder"
 			(at 121.92 103.378 90)
 			(effects
@@
 	(symbol
 		(lib_id "Device:R")
-		(at 157.48 113.03 270)
+		(at 161.29 113.03 270)
 		(mirror x)
 		(unit 1)
@@
 		(dnp no)
 		(property "Reference" "R2"
-			(at 157.48 106.68 90)
+			(at 161.29 106.68 90)
 			(effects
 				(font
@@
 			)
 		)
-		(property "Value" "4640"
-			(at 157.48 109.22 90)
+		(property "Value" "470"
+			(at 161.29 109.22 90)
 			(effects
 				(font
@@
 		)
 		(property "Footprint" "Resistor_SMD:R_0603_1608Metric_Pad0.98x0.95mm_HandSolder"
-			(at 157.48 114.808 90)
+			(at 161.29 114.808 90)
 			(effects
 				(font
@@
 		)
 		(property "Datasheet" "~"
-			(at 157.48 113.03 0)
+			(at 161.29 113.03 0)
 			(effects
 				(font
@@
 		)
 		(property "Description" "Resistor"
-			(at 157.48 113.03 0)
+			(at 161.29 113.03 0)
 			(effects
 				(font
@@
 		(dnp no)
 		(fields_autoplaced yes)
-		(property "Reference" "D1"
+		(property "Reference" "D2"
 			(at 186.69 101.6 0)
 			(effects
@@
 			)
 		)
-		(property "Value" "~"
+		(property "Value" "ESDA6V1U1"
 			(at 186.69 104.14 0)
 			(effects
@@
 			(project ""
 				(path "/f437cf05-d297-460e-8639-991b777c08ac"
-					(reference "D1")
+					(reference "D2")
 					(unit 1)
 				)
@@
 		)
 	)
+	(embedded_fonts no)
 )
