File: EMP/EMP.kicad_sch (KiCad schematic)
At the start: 31 parts, among them J1 Conn_01x03_MountingPin, J2 Conn_01x03_MountingPin, J3 Conn_01x03_MountingPin, J4 Conn_01x03_MountingPin, J5 Netzteil, J6 Conn_01x08, J7 EMP/MDB, J8 Li Rohr, J9 Li Auswurf, Q1 Q_NMOS_GDS, Q2 Q_NMOS_GDS, Q3 Q_NMOS_GDS, Q4 Q_NMOS_GDS, U1 74HC245, U12 L7805, U2 74HC123, U3 74HC165, U4 74HC157, U5 74HC165, U6 74HC123, U7 74HC123, U8 74HC595, U9 74HC238

Commit message: vnd10bsp
Parts:
- added D1, D18, D19, D2, D20, D21, D5, D6, D7, D8, D9: LED, LED_SMD:LED_Osram_Lx_P47F_D2mm_ReverseMount, symbol Device:LED
- added D10, D11, D12, D13, D14, D15, D16, D17, D22: D_Photo, LED_SMD:LED_Osram_Lx_P47F_D2mm_ReverseMount, symbol Device:D_Photo
- added FID1, FID2, FID3, FID4: Fiducial, Fiducial:Fiducial_0.75mm_Mask2.25mm, symbol Mechanical:Fiducial
- added H1, H2: MountingHole, MountingHole:MountingHole_3.2mm_M3, symbol Mechanical:MountingHole
- U13, U14: symbol ST_Power:VND10B -> ST_Power:VND10BSP
Connections:
- net GND: now reaches U12.2 (GND)
- net GND: now also C2.2, J5.4 (Pin_4), J5.5 (Pin_5), J5.6 (Pin_6), J5.7 (Pin_7), J8.10 (Pin_10), J8.3 (Pin_3), J8.8 (Pin_8), Q2.3 (S), U1.10 (GND), U10.14 (GND), U10.15 (GND), U10.16 (GND), U10.17 (GND), U10.4 (GND), U10.5 (GND), U10.6 (GND), U10.7 (GND), U11.14 (GND), U11.15 (GND), U11.16 (GND), U11.17 (GND), U11.4 (GND), U11.5 (GND), U11.6 (GND), U11.7 (GND), U13.6 (GROUND), U14.6 (GROUND), U2.8 (GND), U3.8 (GND), U4.8 (GND), U5.8 (GND), U6.8 (GND), D1.1 (K), D18.1 (K), D19.1 (K), D2.1 (K), D20.1 (K), D21.1 (K), D5.1 (K), D6.1 (K), D7.1 (K), D8.1 (K), D9.1 (K)
- net at U13.10 (NC): now also U13.3 (NC)
- net at J8.4 (Pin_4): now also U5.6 (D7)
- net at Q3.3 (S): now also Q4.3 (S)
- net at U10.18 (OUT2): now also D10.1 (K)
- net at U7.4 (~{Q}): now also U6.12 (~{Q})
- net at J9.10 (Pin_10): now also U5.14 (D3)
- net at J9.4 (Pin_4): now also U5.11 (D0)
- net at J9.6 (Pin_6): now also U5.12 (D1)
- net at J9.8 (Pin_8): now also U5.13 (D2)
- net at C2.1: now also C1.1, J5.3 (Pin_3)
- net at U8.10 (~{SRCLR}): now also U9.6 (E3)
- net at U14.10 (NC): now also U14.3 (NC)
- net at U14.7 (INPUT1): now also U9.12 (Y3)
- net at U14.9 (INPUT2): now also U9.11 (Y4)
- net at Q2.2 (D): now also J1.3 (Pin_3)
- net at J5.1 (Pin_1): now also J5.2 (Pin_2)
- new net: D10.2 (A), D14.1 (K)
- new net: D11.1 (K), D12.2 (A)
- new net: D15.2 (A), D22.1 (K)
Other:
- moved on the sheet: C1, C2, J5, J7, J8, J9, Q2, U5, U6B, U7A, U8, U9

Commit message: emp mit foto
Parts:
- added R1, R10, R11, R12, R13, R14, R15, R16, R17, R18, R19, R2, R20, R3, R4, R5, R6, R7, R8, R9: R, Resistor_SMD:R_0805_2012Metric, symbol Device:R
Connections:
- net +12V: now reaches U12.1 (IN)
- net +12V: now also C1.1, C2.1, D13.2 (A), J5.3 (Pin_3)
- net +5V: now reaches U12.3 (OUT)
- net +5V: now also U4.16 (VCC)
- net at U1.1 (A->B): now also R5.1
- net at U1.4 (A2): now also R3.2
- net at J6.5 (Pin_5): now also R16.2
Other:
- moved on the sheet: J6, U1, U12

Commit message: schalplan
Parts:
- added C10, C11, C12, C13, C14, C15, C16, C17, C18, C19, C20, C21, C22, C5, C6, C7, C8, C9: C, Capacitor_SMD:C_0805_2012Metric, symbol Device:C
- added R21, R22, R23, R24, R25, R26, R27: R, Resistor_SMD:R_0805_2012Metric, symbol Device:R
Connections:
- net +5V: now also U3.16 (VCC)
- net GND: now also C1.2, J7.1 (Pin_1), C10.2, C11.1
- net at R2.1: now also J7.3 (Pin_3), R3.1, C11.2
- net at R2.2: now also R1.2
- net at R8.2: now also R9.2
- net at R16.1: now also U1.15 (B3), C16.1
- net at U6.14 (Cext): now also C22.2
- net at U6.15 (RCext): now also C22.1
- net at D17.2 (A): now also D16.1 (K)
- net at U1.16 (B2): now also R12.1, C15.1
- net at J8.6 (Pin_6): now also U5.4 (D5)
- net at U3.3 (D4): now also R22.2
- net at U3.4 (D5): now also R23.2
- net at U3.5 (D6): now also R24.2
- net at R5.2: now also C20.2
- net at R14.2: now also R11.2
- net at U10.13 (OUT3): now also R21.1
- net at U11.10 (IN4): now also U9.13 (Y2)
- net at R11.1: now also R10.1
- net at J6.4 (Pin_4): now also R12.2
- net at R4.2: now also R7.2
- net at D13.1 (K): now also R21.2
- net at U6.6 (Cext): now also C21.2
- net at U6.7 (RCext): now also C21.1
- net at R18.1: now also J7.5 (Pin_5), C12.1
- new net: C15.2, C16.2
- new net: R22.1, R23.1, R24.1, R25.2, R26.2
Other:
- moved on the sheet: D13, D16, J1, J2, J6, J7, Q2, R1, R12, R14, R16, R18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

Commit message: em
Parts:
- added TP1, TP2, TP3, TP4, TP5, TP6, TP7, TP8, TP9: TestPoint, TestPoint:TestPoint_Pad_D1.5mm, symbol Connector:TestPoint
Connections:
- net at J8.1 (Pin_1): now also U10.12 (OUT4), TP4.1
- net at U3.11 (D0): now also U4.7 (Zb), TP8.1
- net at U3.14 (D3): now also U4.4 (Za), TP7.1
- net at U3.7 (~{Q7}): now also TP6.1
- net at R21.1, U10.13 (OUT3): now also TP5.1
- net at U2.5 (Q): now also TP1.1
- net at U2.6 (Cext): now also TP2.1
- net at U2.7 (RCext): now also R25.1, R26.1, TP3.1
- net at U4.12 (Zd): now also TP9.1
Other:
- moved on the sheet: C3, C4, D10, D13, D14, D18, D19, D20, D21, D5, D6, D7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

Commit message: kondensatoren
Parts:
- added C23, C24, C25: C, Capacitor_SMD:C_1812_4532Metric, symbol Device:C
- added D3: 1N4148W, Diode_SMD:D_SOD-123, symbol Diode:1N4148W
- added R28, R29, R30, R31, R32, R33, R34: R, Resistor_SMD:R_0805_2012Metric, symbol Device:R
Connections:
- net +12V: now also C24.1, R28.1, R29.1, R30.1, R31.2, R32.2, R33.1, R34.1
- net GND: now also C24.2
- new net: R33.2, R34.2
- new net: R28.2, R29.2, R30.2
- new net: R31.1, R32.1

Commit message: led
Parts:
- added C26: C, Capacitor_SMD:C_0805_2012Metric, symbol Device:C
- added R35, R36, R37, R38, R39, R40, R41, R42, R43, R44, R45, R46, R47, R48, R49, R50, R51, R52, R53, R54, R55: R, Resistor_SMD:R_0805_2012Metric, symbol Device:R
- added TP10, TP11, TP12, TP13, TP14, TP15, TP16, TP52, TP53, TP54, TP55, TP56, TP57, TP58, TP59, TP60, TP61: TestPoint, TestPoint:TestPoint_Pad_D1.5mm, symbol Connector:TestPoint
- added TP17, TP18, TP19, TP20, TP21, TP22, TP23, TP24, TP25, TP26, TP27, TP28, TP29, TP30, TP31, TP32, TP33, TP34, TP35, TP36, TP37, TP38, TP39, TP40, TP41, TP42, TP43, TP44, TP45, TP46, TP47, TP48, TP49, TP50, TP51: ~, TestPoint:TestPoint_Pad_D1.5mm, symbol Connector:TestPoint
- D1, D10, D11, D12, D13, D14, D15, D16, D17, D18, D19, D2, D20, D21, D22, D5, D6, D7, D8, D9: footprint LED_SMD:LED_Osram_Lx_P47F_D2mm_ReverseMount -> EMP:LED_ReverseMount
Connections:
- net +12V: now also J9.1 (Pin_1)
- net GND: now also C17.2, C18.2, C19.1, C3.2, C4.2, J9.3 (Pin_3), Q1.3 (S), R40.2, R43.2, R44.2, TP21.1; no longer U1.10 (GND)
- net at U6.1 (A): now also R43.1
- net at U6.3 (Clr): now also R39.2, TP25.1
- net at D17.1 (K): now also TP18.1
- net at D16.1 (K), D17.2 (A): now also TP17.1
- net at R5.1, U1.1 (A->B): now also TP60.1
- net at U1.3 (A1): now also TP59.1
- net at R3.2, U1.4 (A2): now also TP61.1
- net at U1.8 (A6): now also TP58.1
- net at U1.9 (A7): now also R20.1
- net at U13.7 (INPUT1): now also U9.10 (Y5)
- net at U13.8 (DIAG.): now also R35.1, TP19.1
- net at U13.9 (INPUT2): now also U9.9 (Y6), TP20.1
- net at U13.TAB (Vcc): now also C3.1
- net at J8.4 (Pin_4), U5.6 (D7): now also TP51.1
- net at D7.2 (A): now also TP55.1
- net at U7.16 (VCC): now also R50.1, R51.1
- net at Q3.1 (G): now also R37.2
- net at Q1.1 (G): now also R40.1, TP22.1
- net at Q1.2 (D): now also TP37.1
- net at D10.2 (A), D14.1 (K): now also TP36.1
- net at U7.7 (RCext): now also TP52.1
- net at U7.2 (B): now also TP27.1
- net at U7.3 (Clr): now also TP26.1
- net at Q4.1 (G): now also R38.2, TP10.1
- net at J9.2 (Pin_2): now also R47.2, TP43.1
- net at U11.10 (IN4), U9.13 (Y2): now also TP49.1
- net at U11.12 (OUT4): now also R49.1, TP46.1
- net at U11.13 (OUT3): now also R48.1, TP45.1
- net at U11.18 (OUT2): now also R47.1, TP42.1
- net at U11.19 (OUT1): now also R46.1, TP41.1
- net at U11.3 (DIAG): now also TP31.1
- net at U8.9 (QH'): now also TP16.1
- net at D9.2 (A): now also TP57.1
- net at U14.7 (INPUT1), U9.12 (Y3): now also TP14.1
- net at U14.9 (INPUT2), U9.11 (Y4): now also TP13.1
- net at Q2.1 (G): now also R44.1, R45.1, TP33.1
- net at J1.3 (Pin_3), Q2.2 (D): now also TP32.1
- net at D13.1 (K), R21.2: now also TP53.1
- net at U6.5 (Q): now also TP24.1
- net at C21.2, U6.6 (Cext): now also TP23.1
- net at C21.1, U6.7 (RCext): now also R41.1, R42.1, TP38.1
- net at D15.1 (K): now also TP34.1
- net at D15.2 (A), D22.1 (K): now also TP35.1
- net at D8.2 (A): now also TP56.1
- net at D22.2 (A): now also TP40.1
- net at U5.5 (D6): now also TP50.1
- net at U9.1 (A0): now also TP30.1
- net at U9.2 (A1): now also TP29.1
- net at U9.3 (A2): now also TP28.1
- net at U9.7 (Y7): now also TP15.1
- new net: R46.2, TP44.1
- new net: R39.1, R41.2, R42.2
- new net: R45.2, TP39.1
- new net: R48.2, TP47.1
- new net: R49.2, TP48.1
- new net: R35.2, R36.2, TP11.1
- new net: R36.1, TP12.1
- new net: R53.1, TP54.1
Other:
- moved on the sheet: C17, C18, C19, C21, C22, C3, C4, D10, D11, D12, D13, D14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
