File: Lampentreiber/Lampentreiber.kicad_sch (KiCad schematic)
At the start: 10 parts, among them J8 Zentrale, U2 74HC245, U3 74HC165

Commit message: seite 1
Parts:
- added C1, C18, C26: 1nF63V, symbol Device:C
- added C14, C25, C3, C4: VC100nF63V, symbol Device:C
- added C20: MKT10nF63V, symbol Device:C
- added C27: MKT100nF63V, symbol Device:C
- added D10, D11, D12: SD103C, symbol Device:D_Schottky
- added R49, R51, R53, R55, R56: 470, symbol Device:R
- added R57: 270, symbol Device:R
- added R58: 18K, symbol Device:R
- added R61, R86, R90, R91, R92, R93, R97: 2.7K, symbol Device:R
- added R70, R95: 1K, symbol Device:R
- added R71: 10K, symbol Device:R
- added R87, R96: 47K, symbol Device:R
- added R88: 100, symbol Device:R
- added R89: 68K, symbol Device:R
- added U1: L7805, symbol Regulator_Linear:L7805
- added U10, U5, U9: 74HC4094, symbol 4xxx:HEF4094B
- added U11, U8: ULN2803A, symbol Transistor_Array:ULN2803A
- added U12: 74HC107, symbol 74xx:74LS107
- added U4: 4051, symbol 4xxx:4051
- added U6: 74HC123, symbol 74xx:74HC123
- added U7: TC1428, symbol Driver_FET:MIC4428
Connections:
- net +5V: now also C14.1, C4.1, R49.1, R51.1, R53.1, R55.1, R56.1, R58.2, R71.2, R87.2, R88.2, R89.2, U1.3 (OUT), U12.1 (J), U12.14 (VCC), U12.8 (J), U6.16 (VCC), U7.6 (V+)
- net DataAnz: now also R49.2
- net DataAnzp: now also U5.2 (D)
- net DataLp: now also U10.2 (D)
- net DataMux: now also R56.2
- net EL: now also R57.1
- net EnAnz: now also R51.2
- net EnAnzp: now also C1.1, R70.2, U6.1 (A)
- net EnMUX: now also R53.2
- net GND: now also C14.2, C18.2, C25.2, C3.2, C4.2, D10.2 (A), D12.2 (A), R61.1, R86.1, R96.1, R97.1, U1.2 (GND), U10.8 (V_{SS}), U11.9 (GND), U12.11 (K), U12.4 (K), U12.7 (GND), U4.7 (VEE), U4.8 (VSS), U5.8 (V_{SS}), U6.8 (GND), U7.3 (GND), U8.9 (GND), U9.8 (V_{SS})
- net Shift: now also U12.6 (~{Q})
- net nTakt: now also R55.2
- net nTaktp: now also U10.3 (CP), U12.10 (~{R}), U5.3 (CP), U9.3 (CP)
- new net: D11.1 (K), R95.1, U7.4 (IN_B)
- new net: D11.2 (A), U6.13 (Q)
- new net: C18.1, R70.1, U7.2 (IN_A)
- new net: C25.1, R87.1, U12.13 (~{R})
- new net: U12.12 (C), U12.5 (Q)
- new net: C20.1, R58.1, U6.15 (RCext)
- new net: R57.2, U12.9 (C)
- new net: C26.2, D12.1 (K), R97.2, U10.1 (STR), U9.1 (STR)
- new net: C27.1, R89.1, U6.7 (RCext)
- new net: C1.2, D10.1 (K), R86.2, U5.1 (STR)
- new net: U8.4 (I4), U9.12 (QP6)
- new net: U8.3 (I3), U9.13 (QP5)
- new net: U6.9 (A), U8.2 (I2), U9.14 (QP4)
- new net: R93.1, U9.4 (QP0)
- new net: R92.1, U9.5 (QP1)
- new net: R91.1, U9.6 (QP2)
- new net: R90.1, U9.7 (QP3)
- new net: U10.6 (QP2), U11.1 (I1)
- new net: U10.4 (QP0), U11.2 (I2)
- new net: U10.14 (QP4), U11.3 (I3)
- new net: U10.7 (QP3), U11.4 (I4)
- new net: U10.13 (QP5), U11.5 (I5)
- new net: U10.12 (QP6), U11.6 (I6)
- new net: U10.5 (QP1), U11.7 (I7)
- new net: U10.11 (QP7), U11.8 (I8)
- new net: U6.5 (Q), U8.1 (I1)
- new net: U4.9 (C), U8.15 (O4)
- new net: U4.10 (B), U8.16 (O3)
- new net: U4.11 (A), U8.17 (O2)
- new net: U4.6 (Inh), U8.18 (O1)
- new net: R91.2, U8.5 (I5)
- new net: R92.2, U8.6 (I6)
- new net: R90.2, U8.7 (I7)
- new net: R93.2, U8.8 (I8)
- new net: R88.1, U6.10 (B), U6.11 (Clr)
- new net: C27.2, U6.6 (Cext)
- new net: C20.2, U6.14 (Cext)
- new net: R61.2, U4.3 (X)
- new net: R71.1, U6.2 (B), U6.3 (Clr)
- new net +12V: C3.1, U1.1 (IN)
- new net Anzout0: U5.4 (QP0)
- new net Anzout1: U5.5 (QP1)
- new net Anzout2: U5.6 (QP2)
- new net Anzout3: U5.7 (QP3)
- new net Anzout4: U5.14 (QP4)
- new net Anzout5: U5.13 (QP5)
- new net Anzout6: U5.12 (QP6)
- new net Anzout7: U5.11 (QP7)
- new net EnLSp: U6.4 (~{Q})
- new net EnLSpr: U12.3 (Q), U5.15 (OE), U9.15 (OE)
- new net EnLp: C26.1
- new net EnSDAp: R95.2, R96.2, U9.11 (QP7)
- new net EnSDa: U7.5 (OUT_B)
- new net IDp: U10.9 (QS1), U9.2 (D)
- new net LSTr0: U11.17 (O2)
- new net LSTr1: U11.12 (O7)
- new net LSTr10: U8.14 (O5)
- new net LSTr11: U8.12 (O7)
- new net LSTr2: U11.18 (O1)
- new net LSTr3: U11.15 (O4)
- new net LSTr4: U11.16 (O3)
- new net LSTr5: U11.14 (O5)
- new net LSTr6: U11.13 (O6)
- new net LSTr7: U11.11 (O8)
- new net LSTr8: U8.11 (O8)
- new net LSTr9: U8.13 (O6)
- new net LZTr0: U4.13 (X0)
- new net LZTr1: U4.14 (X1)
- new net LZTr2: U4.15 (X2)
- new net LZTr3: U4.12 (X3)
- new net LZTr4: U4.1 (X4)
- new net LZTr5: U4.5 (X5)
- new net LZTr6: U4.2 (X6)
- new net LZTr7: U4.4 (X7)
- new net TaktSDA: U7.7 (~{OUT_A})
- no-connect marks 2 -> 11
Other:
- moved on the sheet: J8, R47, R48, R50, R52, R54, R59, R72, U2, U3

Commit message: lampen
Parts:
- C1, C14, C18, C20, C25, C26, C27, C3, C4: footprint (none) -> Capacitor_SMD:C_0805_2012Metric
- D10, D11, D12: footprint (none) -> Diode_SMD:D_SOD-123
- J8: footprint (none) -> Connector_PinHeader_2.54mm:PinHeader_1x08_P2.54mm_Horizontal
- R47, R48, R49, R50, R51, R52, R53, R54, R55, R56, R57, R58, R59, R61, R70, R71, R72, R86, R87, R88, R89, R90, R91, R92, R93, R95, R96, R97: footprint (none) -> Resistor_SMD:R_0805_2012Metric
- U1: footprint (none) -> Package_TO_SOT_SMD:TO-252-3_TabPin2
- U10, U3, U4, U5, U6, U9: footprint (none) -> Package_SO:SO-16_3.9x9.9mm_P1.27mm
- U11: footprint (none) -> Package_SO:SOP-18_7x12.5mm_P1.27mm
- U12: footprint (none) -> Package_SO:SOIC-14_3.9x8.7mm_P1.27mm
- U2: footprint (none) -> Package_SO:SOIC-20W_7.5x12.8mm_P1.27mm
- U7: footprint (none) -> Package_SO:SO-8_3.9x4.9mm_P1.27mm
- U8: footprint (none) -> Package_SO:SOP-18_7.495x11.515mm_P1.27mm
Changed lines of the file:
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@@
 			)
 		)
-		(property "Footprint" ""
+		(property "Footprint" "Diode_SMD:D_SOD-123"
 			(at 200.66 182.88 0)
 			(effects
@@
 			)
 		)
-		(property "Footprint" ""
+		(property "Footprint" "Capacitor_SMD:C_0805_2012Metric"
 			(at 199.0852 242.57 0)
 			(effects
@@
 			)
 		)
-		(property "Footprint" ""
+		(property "Footprint" "Capacitor_SMD:C_0805_2012Metric"
 			(at 143.2052 227.33 0)
 			(effects
@@
 			)
 		)
-		(property "Footprint" ""
+		(property "Footprint" "Resistor_SMD:R_0805_2012Metric"
 			(at 31.242 162.56 90)
 			(effects
@@
 			)
 		)
-		(property "Footprint" ""
+		(property "Footprint" "Package_SO:SOIC-14_3.9x8.7mm_P1.27mm"
 			(at 177.8 212.09 0)
 			(effects
@@
 			)
 		)
-		(property "Footprint" ""
+		(property "Footprint" "Resistor_SMD:R_0805_2012Metric"
 			(at 81.28 221.488 90)
 			(effects
@@
 			)
 		)
-		(property "Footprint" ""
+		(property "Footprint" "Resistor_SMD:R_0805_2012Metric"
 			(at 159.258 170.18 90)
 			(effects
@@
 			)
 		)
-		(property "Footprint" ""
+		(property "Footprint" "Capacitor_SMD:C_0805_2012Metric"
 			(at 140.6652 158.75 0)
 			(effects
@@
 			)
 		)
-		(property "Footprint" ""
+		(property "Footprint" "Resistor_SMD:R_0805_2012Metric"
 			(at 115.57 178.308 90)
 			(effects
@@
 			)
 		)
-		(property "Footprint" ""
+		(property "Footprint" "Resistor_SMD:R_0805_2012Metric"
 			(at 133.35 236.728 90)
 			(effects
@@
 			)
 		)
-		(property "Footprint" ""
+		(property "Footprint" "Package_SO:SO-16_3.9x9.9mm_P1.27mm"
 			(at 327.66 231.14 0)
 			(effects
@@
 			)
 		)
-		(property "Footprint" ""
+		(property "Footprint" "Resistor_SMD:R_0805_2012Metric"
 			(at 268.732 121.92 90)
 			(effects
@@
 			)
 		)
-		(property "Footprint" ""
+		(property "Footprint" "Resistor_SMD:R_0805_2012Metric"
 			(at 115.57 188.468 90)
 			(effects
@@
 			)
 		)
-		(property "Footprint" ""
+		(property "Footprint" "Package_SO:SO-16_3.9x9.9mm_P1.27mm"
 			(at 81.28 251.46 0)
 			(effects
@@
 			)
 		)
-		(property "Footprint" ""
+		(property "Footprint" "Resistor_SMD:R_0805_2012Metric"
 			(at 307.848 25.4 90)
 			(effects
@@
 			)
 		)
-		(property "Footprint" ""
+		(property "Footprint" "Resistor_SMD:R_0805_2012Metric"
 			(at 207.518 236.22 90)
 			(effects
@@
 			)
 		)
-		(property "Footprint" ""
+		(property "Footprint" "Resistor_SMD:R_0805_2012Metric"
 			(at 196.342 223.52 90)
 			(effects
@@
 			)
 		)
-		(property "Footprint" ""
+		(property "Footprint" "Resistor_SMD:R_0805_2012Metric"
 			(at 214.122 193.04 90)
 			(effects
@@
 			)
 		)
-		(property "Footprint" ""
+		(property "Footprint" "Resistor_SMD:R_0805_2012Metric"
 			(at 109.22 191.008 90)
 			(effects
@@
 			)
 		)
-		(property "Footprint" ""
+		(property "Footprint" "Package_SO:SO-16_3.9x9.9mm_P1.27mm"
 			(at 290.83 121.92 0)
 			(effects
@@
 			)
 		)
-		(property "Footprint" ""
+		(property "Footprint" "Package_SO:SOP-18_7x12.5mm_P1.27mm"
 			(at 327.66 88.9 0)
 			(effects
@@
 			)
 		)
-		(property "Footprint" ""
+		(property "Footprint" "Resistor_SMD:R_0805_2012Metric"
 			(at 109.22 173.228 90)
 			(effects
@@
 			)
 		)
-		(property "Footprint" ""
+		(property "Footprint" "Package_SO:SOP-18_7.495x11.515mm_P1.27mm"
 			(at 332.74 114.3 0)
 			(effects
@@
 			)
 		)
-		(property "Footprint" ""
+		(property "Footprint" "Package_SO:SOIC-20W_7.5x12.8mm_P1.27mm"
 			(at 81.28 184.15 0)
 			(effects
@@
 			)
 		)
-		(property "Footprint" ""
+		(property "Footprint" "Resistor_SMD:R_0805_2012Metric"
 			(at 309.88 123.952 90)
 			(effects
@@
 			)
 		)
-		(property "Footprint" ""
+		(property "Footprint" "Capacitor_SMD:C_0805_2012Metric"
 			(at 269.5448 59.69 0)
 			(effects
@@
 			)
 		)
-		(property "Footprint" ""
+		(property "Footprint" "Resistor_SMD:R_0805_2012Metric"
 			(at 302.768 142.24 90)
 			(effects
@@
 			)
 		)
-		(property "Footprint" ""
+		(property "Footprint" "Capacitor_SMD:C_0805_2012Metric"
 			(at 123.4948 158.75 0)
 			(effects
@@
 			)
 		)
-		(property "Footprint" ""
+		(property "Footprint" "Package_SO:SO-16_3.9x9.9mm_P1.27mm"
 			(at 326.39 39.37 0)
 			(effects
@@
 			)
 		)
-		(property "Footprint" ""
+		(property "Footprint" "Package_TO_SOT_SMD:TO-252-3_TabPin2"
 			(at 132.715 154.94 0)
 			(effects
@@
 			)
 		)
-		(property "Footprint" ""
+		(property "Footprint" "Package_SO:SO-16_3.9x9.9mm_P1.27mm"
 			(at 238.76 187.96 0)
 			(effects
@@
 			)
 		)
-		(property "Footprint" ""
+		(property "Footprint" "Resistor_SMD:R_0805_2012Metric"
 			(at 49.022 147.32 90)
 			(effects
@@
 			)
 		)
-		(property "Footprint" ""
+		(property "Footprint" "Resistor_SMD:R_0805_2012Metric"
 			(at 309.88 126.492 90)
 			(effects
@@
 			)
 		)
-		(property "Footprint" ""
+		(property "Footprint" "Connector_PinHeader_2.54mm:PinHeader_1x08_P2.54mm_Horizontal"
 			(at 16.51 181.61 0)
 			(effects
@@
 			)
 		)
-		(property "Footprint" ""
+		(property "Footprint" "Capacitor_SMD:C_0805_2012Metric"
 			(at 165.1 180.6448 0)
 			(effects
@@
 			)
 		)
-		(property "Footprint" ""
+		(property "Footprint" "Resistor_SMD:R_0805_2012Metric"
 			(at 401.828 162.56 90)
 			(effects
@@
 			)
 		)
-		(property "Footprint" ""
+		(property "Footprint" "Resistor_SMD:R_0805_2012Metric"
 			(at 54.102 162.56 90)
 			(effects
@@
 			)
 		)
-		(property "Footprint" ""
+		(property "Footprint" "Capacitor_SMD:C_0805_2012Metric"
 			(at 313.69 35.8648 0)
 			(effects
@@
 			)
 		)
-		(property "Footprint" ""
+		(property "Footprint" "Resistor_SMD:R_0805_2012Metric"
 			(at 150.622 170.18 90)
 			(effects
@@
 			)
 		)
-		(property "Footprint" ""
+		(property "Footprint" "Diode_SMD:D_SOD-123"
 			(at 275.59 121.92 0)
 			(effects
@@
 			)
 		)
-		(property "Footprint" ""
+		(property "Footprint" "Resistor_SMD:R_0805_2012Metric"
 			(at 46.482 162.56 90)
 			(effects
@@
 			)
 		)
-		(property "Footprint" ""
+		(property "Footprint" "Resistor_SMD:R_0805_2012Metric"
 			(at 299.212 25.4 90)
 			(effects
@@
 			)
 		)
-		(property "Footprint" ""
+		(property "Footprint" "Package_SO:SOIC-14_3.9x8.7mm_P1.27mm"
 			(at 177.8 234.95 0)
 			(effects
@@
 			)
 		)
-		(property "Footprint" ""
+		(property "Footprint" "Capacitor_SMD:C_0805_2012Metric"
 			(at 215.9 185.1152 0)
 			(effects
@@
 			)
 		)
-		(property "Footprint" ""
+		(property "Footprint" "Resistor_SMD:R_0805_2012Metric"
 			(at 36.83 185.928 90)
 			(effects
@@
 			)
 		)
-		(property "Footprint" ""
+		(property "Footprint" "Package_SO:SOIC-14_3.9x8.7mm_P1.27mm"
 			(at 355.6 231.14 0)
 			(effects
@@
 			)
 		)
-		(property "Footprint" ""
+		(property "Footprint" "Package_SO:SO-8_3.9x4.9mm_P1.27mm"
 			(at 231.14 245.11 0)
 			(effects
@@
 			)
 		)
-		(property "Footprint" ""
+		(property "Footprint" "Resistor_SMD:R_0805_2012Metric"
 			(at 144.018 215.9 90)
 			(effects
@@
 			)
 		)
-		(property "Footprint" ""
+		(property "Footprint" "Capacitor_SMD:C_0805_2012Metric"
 			(at 72.0852 151.13 0)
 			(effects
@@
 			)
 		)
-		(property "Footprint" ""
+		(property "Footprint" "Resistor_SMD:R_0805_2012Metric"
 			(at 309.88 122.428 90)
 			(effects
@@
 			)
 		)
-		(property "Footprint" ""
+		(property "Footprint" "Package_SO:SO-16_3.9x9.9mm_P1.27mm"
 			(at 387.35 143.51 0)
 			(effects
@@
 			)
 		)
-		(property "Footprint" ""
+		(property "Footprint" "Diode_SMD:D_SOD-123"
 			(at 220.98 193.04 0)
 			(effects
@@
 			)
 		)
-		(property "Footprint" ""
+		(property "Footprint" "Package_SO:SO-16_3.9x9.9mm_P1.27mm"
 			(at 177.8 184.15 0)
 			(effects
@@
 			)
 		)
-		(property "Footprint" ""
+		(property "Footprint" "Package_SO:SO-16_3.9x9.9mm_P1.27mm"
 			(at 290.83 71.12 0)
 			(effects
@@
 			)
 		)
-		(property "Footprint" ""
+		(property "Footprint" "Resistor_SMD:R_0805_2012Metric"
 			(at 64.77 196.088 90)
 			(effects
@@
 			)
 		)
-		(property "Footprint" ""
+		(property "Footprint" "Resistor_SMD:R_0805_2012Metric"
 			(at 38.862 162.56 90)
 			(effects
@@
 			)
 		)
-		(property "Footprint" ""
+		(property "Footprint" "Resistor_SMD:R_0805_2012Metric"
 			(at 309.88 124.968 90)
 			(effects
