File: SuS/SuS.kicad_sch (KiCad schematic)
At the start: 83 parts, among them P1 DIN41612_03x10_ABC, P2 DIN41612_03x10_ABC, Q1 BC556, U1 74HC245, U10 74HC32, U11 74HC245, U12 MAX691CPE, U13 74HC138, U14 74HC573, U15 74HC32, U16 74HC573, U17 74HC08, U18 74HC10, U19 74HC32, U2 27C040, U20 74HC21, U21 MC68EC000FN, U22 RTC62421, U3 V62C5181024LL-70P, U4 74HC573, U5 M48Tx2, U6 27C040, U7 V62C5181024LL-70P, U8 M48Tx2, U9 SG-531

Commit message: vcc
Connections:
- net GND: now also C15.2, D2.2 (A)
- net VCC: now reaches C15.1
- net VCC: now also C1.1, C11.1, C14.1, C17.1, C2.1, C20.1, C21.1, C22.1, C4.1, C5.1, C6.1, C7.1, C9.1, D2.1 (K), Q1.3 (E), R16.2, R19.2, R20.2, U1.20 (VCC), U10.14 (VCC), U11.20 (VCC), U12.3 (VCC), U13.16 (VCC), U14.20 (VCC), U15.14 (VCC), U16.20 (VCC), U17.14 (VCC), U18.14 (VCC), U19.14 (VCC), U2.32 (VCC), U20.14 (VCC), U21.15 (V_{CC}), U21.19 (MODE), U21.53 (V_{CC}), U22.18 (VDD), U3.32 (VCC), U4.20 (VCC), U5.24 (VCC), U6.1 (VPP), U6.32 (VCC), U7.32 (VCC), U8.24 (VCC), U9.8 (Vcc)
- net at U18.12: now also U14.1 (OE)
- net at R24.2: now also R19.1
- net at C16.1: now also C14.2
Other:
- moved on the sheet: C1, C14, C16, C2, R19, R21, R24, U14, U17C, U17E, U18A, U18C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

Commit message: neues bild
Parts:
- added D4: SD103C, Diode_THT:D_DO-34_SOD68_P7.62mm_Horizontal, symbol Device:D_Schottky
Connections:
- net A1: now also U2.12 (A0), U3.12 (A0), U6.12 (A0), U7.12 (A0)
- net A10: now also U2.26 (A9), U3.26 (A9), U6.26 (A9), U7.26 (A9)
- net A11: now also U2.23 (A10), U3.23 (A10), U6.23 (A10), U7.23 (A10)
- net A12: now also U2.25 (A11), U3.25 (A11), U6.25 (A11), U7.25 (A11)
- net A13: now also U2.4 (A12), U3.4 (A12), U6.4 (A12), U7.4 (A12)
- net A14: now also U2.28 (A13), U3.28 (A13), U6.28 (A13), U7.28 (A13)
- net A15: now also U2.29 (A14), U3.3 (A14), U6.29 (A14)
- net A16: now also U2.3 (A15), U3.31 (A15), U6.3 (A15)
- net A17: now also U2.2 (A16), U3.2 (A16), U6.2 (A16)
- net A18: now also U2.30 (A17), U6.30 (A17)
- net A19: now also U2.31 (A18), U6.31 (A18)
- net A2: now also U2.11 (A1), U3.11 (A1), U6.11 (A1), U7.11 (A1)
- net A3: now also U2.10 (A2), U3.10 (A2), U6.10 (A2), U7.10 (A2)
- net A4: now also U2.9 (A3), U3.9 (A3), U6.9 (A3), U7.9 (A3)
- net A5: now also U2.8 (A4), U3.8 (A4), U6.8 (A4), U7.8 (A4)
- net A6: now also U2.7 (A5), U3.7 (A5), U6.7 (A5), U7.7 (A5)
- net A7: now also U2.6 (A6), U3.6 (A6), U6.6 (A6), U7.6 (A6)
- net A8: now also U2.5 (A7), U3.5 (A7), U6.5 (A7), U7.5 (A7)
- net A9: now also U2.27 (A8), U3.27 (A8), U6.27 (A8), U7.27 (A8)
- net D0: now also U1.6 (A4), U22.14 (D0), U4.6 (D4), U6.13 (D0), U7.13 (I/O0), U8.9 (DQ0)
- net D1: now also U1.7 (A5), U22.13 (D1), U4.7 (D5), U6.14 (D1), U7.14 (I/O1), U8.10 (DQ1)
- net D10: now also U2.15 (D2), U3.15 (I/O2), U5.11 (DQ2)
- net D11: now also U2.17 (D3), U3.17 (I/O3), U5.13 (DQ3)
- net D12: now also U2.18 (D4), U3.18 (I/O4), U5.14 (DQ4)
- net D13: now also U2.19 (D5), U3.19 (I/O5), U5.15 (DQ5)
- net D14: now also U2.20 (D6), U3.20 (I/O6), U5.16 (DQ6)
- net D15: now also U2.21 (D7), U3.21 (I/O7), U5.17 (DQ7)
- net D2: now also U1.5 (A3), U22.12 (D2), U4.5 (D3), U6.15 (D2), U7.15 (I/O2), U8.11 (DQ2)
- net D3: now also U1.9 (A7), U22.11 (D3), U4.9 (D7), U6.17 (D3), U7.17 (I/O3), U8.13 (DQ3)
- net D4: now also U1.4 (A2), U4.4 (D2), U6.18 (D4), U7.18 (I/O4), U8.14 (DQ4)
- net D5: now also U1.3 (A1), U4.3 (D1), U6.19 (D5), U7.19 (I/O5), U8.15 (DQ5)
- net D6: now also U1.8 (A6), U4.8 (D6), U6.20 (D6), U7.20 (I/O6), U8.16 (DQ6)
- net D7: now also U1.2 (A0), U4.2 (D0), U6.21 (D7), U7.21 (I/O7), U8.17 (DQ7)
- net D8: now also U2.13 (D0), U3.13 (I/O0), U5.9 (DQ0)
- net D9: now also U2.14 (D1), U3.14 (I/O1), U5.10 (DQ1)
- net GND: now also P1.a7 (Pin_a7)
- net VCC: now also C13.1
- net at R4.2: now also D1.2 (A), R3.2, R5.2
- net CLK: now reaches R15.1
- net CLK: now also U21.16 (CLK), U9.5 (OUT)
- net at U13.13 (~{Y2}), U19.12, U20.10: now also U20.9
- net DTACK: now reaches U21.11 (~{DTACK})
- net BG: now reaches U21.12 (~{BG})
- net BGACK: now reaches U21.13 (~{BGACK})
- net BR: now reaches U21.14 (~{BR})
- net BR: now also C10.1, P1.a4 (Pin_a4)
- net HALT: now reaches U21.20 (~{HALT})
- net HALT: now also U13.6 (E2)
- net RESET: now reaches U21.21 (~{RESET})
- net AVEC: now reaches U21.23 (~{AVEC})
- net BERR: now reaches U21.24 (~{BERR})
- net IPL2: now reaches U21.25 (~{IPL2})
- net IPL1: now reaches U21.26 (~{IPL1})
- net IPL0: now reaches U21.27 (~{IPL0})
- net FC2: now reaches U21.28 (FC2)
- net FC1: now reaches U21.29 (FC1)
- net FC0: now reaches U21.30 (FC0)
- net AS: now reaches U21.7 (~{AS})
- net UDS: now reaches U21.8 (~{UDS})
- net LDS: now reaches U21.9 (~{LDS})
- net LDS: now also U10.5
- net p1_c10: now reaches P1.c10 (Pin_c10)
- net p1_c5: now reaches P1.c5 (Pin_c5)
- net p1_c5: now also R13.2
- net p1_c6: now reaches P1.c6 (Pin_c6)
- net p1_c6: now also D6.2 (A)
- net EXT_D7: now reaches P1.c7 (Pin_c7)
- net EXT_D7: now also U1.18 (B0), U4.19 (Q0)
- net EXT_D5: now reaches P1.c8 (Pin_c8)
- net EXT_D5: now also U1.17 (B1), U4.18 (Q1)
- net EXT_D2: now reaches P1.c9 (Pin_c9)
- net EXT_D2: now also U1.15 (B3), U4.16 (Q3)
- net p1_a10: now reaches P1.a10 (Pin_a10)
- net EXT_D3: now reaches P1.a8 (Pin_a8)
- net EXT_D3: now also U1.11 (B7), U4.12 (Q7)
- net EXT_D0: now reaches P1.a9 (Pin_a9)
- net EXT_D0: now also U1.14 (B4), U4.15 (Q4)
- net at U13.12 (~{Y3}): now also U10.2, U10.4
- net Y1: now reaches U13.14 (~{Y1})
- net Y1: now also U15.10
- net at U13.5 (~{E1}): now also U16.11 (Load)
- net EXT_D15: now reaches U11.18 (B0)
- net p1_b10: now reaches P1.b10 (Pin_b10)
- net p1_b5: now reaches P1.b5 (Pin_b5)
- net p1_b6: now reaches P1.b6 (Pin_b6)
- net EXT_D6: now reaches P1.b7 (Pin_b7)
- net EXT_D6: now also U1.12 (B6), U4.13 (Q6)
- net EXT_D4: now reaches P1.b8 (Pin_b8)
- net EXT_D4: now also U1.16 (B2), U4.17 (Q2)
- net EXT_D1: now reaches P1.b9 (Pin_b9)
- net EXT_D1: now also U1.13 (B5), U4.14 (Q5)
- net at C16.2: now also D4.2 (A)
- net at U15.4: now also U15.5
- net at U7.3 (A14): now also R21.2
Other:
- moved on the sheet: C14, C16, R11, R21, R4, U10A, U10B

Commit message: greeeen
Parts:
- removed U5, U8: M48Tx2, Package_DIP:DIP-24_18.0mmx34.29mm_W15.24mm_Socket, symbol Memory_RAM:M48Tx2
- U2, U6: value 27C040 -> 27C4001
Connections:
- net IPL1 is gone; now on net IPL0: U21.26 (~{IPL1})
- net p1_a10 is gone; now on net VCC: P1.a10 (Pin_a10)
- net p1_b10 is gone; now on net VCC: P1.b10 (Pin_b10)
- net p1_c10 is gone; now on net VCC: P1.c10 (Pin_c10)
- net A1: now also U22.4 (A0)
- net A16: now also U7.31 (A15)
- net A17: now also U7.2 (A16)
- net A2: now also U17.5, U22.5 (A1)
- net A3: now also U22.6 (A2)
- net A4: now also U22.7 (A3)
- net D10: now also U11.8 (A6), U14.8 (D6)
- net D11: now also U11.9 (A7), U14.9 (D7)
- net D12: now also U11.7 (A5), U14.7 (D5)
- net D13: now also U11.6 (A4), U14.6 (D4)
- net D14: now also U11.5 (A3), U14.5 (D3)
- net D15: now also U14.2 (D0)
- net D8: now also U11.3 (A1), U14.3 (D1)
- net D9: now also U11.4 (A2), U14.4 (D2)
- net EXT_D10: now also P2.c9 (Pin_c9), U11.12 (B6), U14.13 (Q6)
- net EXT_D11: now also P2.a8 (Pin_a8), U11.11 (B7), U14.12 (Q7)
- net EXT_D12: now also P2.b8 (Pin_b8), U11.13 (B5), U14.14 (Q5)
- net EXT_D13: now also P2.c8 (Pin_c8), U11.14 (B4), U14.15 (Q4)
- net EXT_D14: now also P2.b7 (Pin_b7), U11.15 (B3), U14.16 (Q3)
- net EXT_D15: now also P2.c7 (Pin_c7), U14.19 (Q0)
- net EXT_D8: now also P2.a9 (Pin_a9), U11.17 (B1), U14.18 (Q1)
- net EXT_D9: now also P2.b9 (Pin_b9), U11.16 (B2), U14.17 (Q2)
- net FC1: now also U17.1
- net GND: now also R5.1
- net VCC: now also C19.1, R2.1, R8.2, U2.1 (VPP), U22.3 (ALE), U3.30 (CS2/CE2), U7.30 (CS2/CE2); no longer C2.1, U22.18 (VDD), U3.32 (VCC), U7.32 (VCC)
- net at R11.2, R4.1: now also U12.9 (PFI)
- net at D4.1 (K): now also U19.6
- net at C16.2, D4.2 (A): now also R13.1
- net at U22.15 (CS1): now also R8.1
- net at U3.24 (~{OE}): now also U10.8, U7.24 (~{OE})
- net at U20.1: now also D7.2 (A)
- net at U11.19 (CE): now also U1.19 (CE)
- net at U15.1, U15.2, U15.9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: now also U15.13, U15.4, U15.5
- net at U7.22 (~{CS1}/~{CE1}): now also R18.2
- net at U9.1 (OE): now also R12.1
- new net VCCQ: C2.1, U22.18 (VDD), U3.32 (VCC), U7.32 (VCC)
Other:
- moved on the sheet: C14, C16, D1, D4, D7, P2A, P2B, R11, R12, R13, R18, R3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

Commit message: a14
Parts:
- R21: now not fitted
Connections:
- net A14: now also R7.1; no longer U3.28 (A13), U7.28 (A13)
- net A15: now also R21.1
- net VCC: now also R12.2, R14.2
- net at S1.1 (A): now also D1.2 (A), R3.2, R4.2, R5.2
- net at R7.2: now also R1.1, U3.28 (A13)
- net at R16.1: now also D5.2 (A)
Other:
- moved on the sheet: R1, R12, R16, R7, S1

Commit message: oben
Parts:
- D7, D8, U15, U22: now not fitted
Connections:
- net A15: no longer U3.3 (A14)
- net A18: no longer U2.30 (A17), U6.30 (A17)
- net A22: now also U13.1 (A0)
- net A23: now also U13.2 (A1)
- net GND: now also C18.1, D3.2 (A), R18.1, R9.1; no longer C18.2
- net RW: now also U13.3 (A2)
- net VCC: now also C8.1, D3.1 (K), P2.a10 (Pin_a10), P2.b10 (Pin_b10), P2.c10 (Pin_c10), R10.2, R17.1, R2.2, R6.1; no longer C5.1, C9.1, R2.1, R8.2, U22.3 (ALE), U3.30 (CS2/CE2), U7.30 (CS2/CE2)
- net VCCQ: now also R2.1, R8.2, U3.30 (CS2/CE2), U7.30 (CS2/CE2); no longer C2.1, U22.18 (VDD), U3.32 (VCC), U7.32 (VCC)
- net Y1: now also D7.1 (K)
- net at R11.2, R4.1, U12.9 (PFI): now also R6.2
- net at R1.1, R7.2, U3.28 (A13): now also U7.28 (A13)
- net Y2: now reaches U13.13 (~{Y2}), U19.12, U20.10, U20.9
- net CE: now reaches U2.22 (~{CE})
- net CE: now also R18.2, U1.1 (A->B), U11.1 (A->B), U16.1 (OE), U3.22 (~{CS1}/~{CE1}), U6.22 (~{CE}), U7.22 (~{CS1}/~{CE1})
- net at U2.24 (~{OE}): now also U6.24 (~{OE})
- net at U12.13 (~{CE_IN}): now also R10.1, R9.2
- net VDD: now reaches U12.2 (VOUT)
- net VDD: now also C18.2, C2.1, C5.1, C9.1, Q1.1 (C), U22.18 (VDD), U22.3 (ALE), U3.32 (VCC), U7.32 (VCC)
- net at R8.1, U22.15 (CS1): now also R1.2, R17.2
- net at D7.2 (A), U20.1: now also D8.2 (A)
- net Y4: now reaches U20.2
- net Y4: now also U13.11 (~{Y4})
- net Y3: now reaches U20.5
- net Y3: now also U10.2, U10.4, U13.12 (~{Y3})
- net at U18.1: now also U18.2
- net at U17.10, U18.13, U18.9: now also U19.8
- net Y5: now reaches U13.10 (~{Y5})
- net Y7: now reaches U13.7 (~{Y7})
- net Y6: now reaches U13.9 (~{Y6})
- net at U1.19 (CE), U11.19 (CE): now also U17.8
- net at R25.2: now also R20.1, U2.30 (A17), U6.30 (A17)
- net at U7.29 (~{WE}): now also U10.6
- net at R21.2, U7.3 (A14): now also U3.3 (A14)
- net at D8.1 (K): now also U15.12
- no-connect marks 0 -> 5
Other:
- moved on the sheet: C1, C11, C18, C2, C20, C21, C22, C8, C9, Q1, R10, R17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

Commit message: untenrum fertig
Parts:
- added H3, H4: MountingHole, MountingHole:MountingHole_2.1mm, symbol Mechanical:MountingHole
Connections:
- net at U12.10 (~{PFO}): now also P2.a5 (Pin_a5)
- net at R22.1: now also U19.5
Other:
- moved on the sheet: R22
Changed lines of the file:
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@@
 	(wire
 		(pts
+			(xy 218.44 208.28) (xy 218.44 138.43)
+		)
+		(stroke
+			(width 0)
+			(type default)
+		)
+	)
+	(wire
+		(pts
 			(xy 309.88 111.76) (xy 309.88 121.92)
 		)
@@
 	(wire
 		(pts
+			(xy 149.86 208.28) (xy 218.44 208.28)
+		)
+		(stroke
+			(width 0)
+			(type default)
+		)
+	)
+	(wire
+		(pts
 			(xy 106.68 119.38) (xy 106.68 85.09)
 		)
@@
 	(wire
 		(pts
+			(xy 149.86 182.88) (xy 149.86 208.28)
+		)
+		(stroke
+			(width 0)
+			(type default)
+		)
+	)
+	(wire
+		(pts
 			(xy 510.54 0) (xy 513.08 0)
 		)
@@
 	(wire
 		(pts
+			(xy 463.55 2.54) (xy 467.36 2.54)
+		)
+		(stroke
+			(width 0)
+			(type default)
+		)
+	)
+	(wire
+		(pts
 			(xy 355.6 -93.98) (xy 375.92 -93.98)
 		)
@@
 	(wire
 		(pts
+			(xy 119.38 182.88) (xy 149.86 182.88)
+		)
+		(stroke
+			(width 0)
+			(type default)
+		)
+	)
+	(wire
+		(pts
 			(xy 96.52 -17.78) (xy 111.76 -17.78)
 		)
@@
 	(wire
 		(pts
+			(xy 218.44 138.43) (xy 210.82 138.43)
+		)
+		(stroke
+			(width 0)
+			(type default)
+		)
+	)
+	(wire
+		(pts
 			(xy 195.58 -2.54) (xy 195.58 15.24)
 		)
@@
 	)
 	(symbol
+		(lib_id "Mechanical:MountingHole")
+		(at 403.86 185.42 0)
+		(unit 1)
+		(exclude_from_sim no)
+		(in_bom no)
+		(on_board yes)
+		(dnp no)
+		(fields_autoplaced yes)
+		(property "Reference" "H4"
+			(at 406.4 184.1499 0)
+			(effects
+				(font
+					(size 1.27 1.27)
+				)
+				(justify left)
+			)
+		)
+		(property "Value" "MountingHole"
+			(at 406.4 186.6899 0)
+			(effects
+				(font
+					(size 1.27 1.27)
+				)
+				(justify left)
+			)
+		)
+		(property "Footprint" "MountingHole:MountingHole_2.1mm"
+			(at 403.86 185.42 0)
+			(effects
+				(font
+					(size 1.27 1.27)
+				)
+				(hide yes)
+			)
+		)
+		(property "Datasheet" "~"
+			(at 403.86 185.42 0)
+			(effects
+				(font
+					(size 1.27 1.27)
+				)
+				(hide yes)
+			)
+		)
+		(property "Description" "Mounting Hole without connection"
+			(at 403.86 185.42 0)
+			(effects
+				(font
+					(size 1.27 1.27)
+				)
+				(hide yes)
+			)
+		)
+		(instances
+			(project "SuS"
+				(path "/842e655d-6d5c-434c-9eb4-fefb155e89e7"
+					(reference "H4")
+					(unit 1)
+				)
+			)
+		)
+	)
+	(symbol
 		(lib_id "power:GND")
 		(at 220.98 116.84 0)
@@
 	)
 	(symbol
+		(lib_id "Mechanical:MountingHole")
+		(at 403.86 170.18 0)
+		(unit 1)
+		(exclude_from_sim no)
+		(in_bom no)
+		(on_board yes)
+		(dnp no)
+		(fields_autoplaced yes)
+		(property "Reference" "H3"
+			(at 406.4 168.9099 0)
+			(effects
+				(font
+					(size 1.27 1.27)
+				)
+				(justify left)
+			)
+		)
+		(property "Value" "MountingHole"
+			(at 406.4 171.4499 0)
+			(effects
+				(font
+					(size 1.27 1.27)
+				)
+				(justify left)
+			)
+		)
+		(property "Footprint" "MountingHole:MountingHole_2.1mm"
+			(at 403.86 170.18 0)
+			(effects
+				(font
+					(size 1.27 1.27)
+				)
+				(hide yes)
+			)
+		)
+		(property "Datasheet" "~"
+			(at 403.86 170.18 0)
+			(effects
+				(font
+					(size 1.27 1.27)
+				)
+				(hide yes)
+			)
+		)
+		(property "Description" "Mounting Hole without connection"
+			(at 403.86 170.18 0)
+			(effects
+				(font
+					(size 1.27 1.27)
+				)
+				(hide yes)
+			)
+		)
+		(instances
+			(project ""
+				(path "/842e655d-6d5c-434c-9eb4-fefb155e89e7"
+					(reference "H3")
+					(unit 1)
+				)
+			)
+		)
+	)
+	(symbol
 		(lib_id "74xx:74LS32")
 		(at 363.22 -101.6 0)
@@
 	(symbol
 		(lib_id "Device:R")
-		(at 344.17 204.47 90)
+		(at 459.74 2.54 270)
 		(unit 1)
 		(exclude_from_sim no)
@@
 		(fields_autoplaced yes)
 		(property "Reference" "R22"
-			(at 344.17 198.12 90)
+			(at 459.74 8.89 90)
 			(effects
 				(font
@@
 		)
 		(property "Value" "22k"
-			(at 344.17 200.66 90)
+			(at 459.74 6.35 90)
 			(effects
 				(font
@@
 		)
 		(property "Footprint" "Resistor_THT:R_Axial_DIN0207_L6.3mm_D2.5mm_P10.16mm_Horizontal"
-			(at 344.17 206.248 90)
+			(at 459.74 0.762 90)
 			(effects
 				(font
@@
 		)
 		(property "Datasheet" "~"
-			(at 344.17 204.47 0)
+			(at 459.74 2.54 0)
 			(effects
 				(font
@@
 		)
 		(property "Description" "Resistor"
-			(at 344.17 204.47 0)
+			(at 459.74 2.54 0)
 			(effects
 				(font
@@
 	(symbol
 		(lib_id "power:GND")
-		(at 347.98 204.47 90)
+		(at 455.93 2.54 270)
 		(unit 1)
 		(exclude_from_sim no)
@@
 		(fields_autoplaced yes)
 		(property "Reference" "#PWR08"
-			(at 354.33 204.47 0)
+			(at 449.58 2.54 0)
 			(effects
 				(font
@@
 		)
 		(property "Value" "GND"
-			(at 351.79 204.4699 90)
+			(at 452.12 2.5401 90)
 			(effects
 				(font
@@
 		)
 		(property "Footprint" ""
-			(at 347.98 204.47 0)
+			(at 455.93 2.54 0)
 			(effects
 				(font
@@
 		)
 		(property "Datasheet" ""
-			(at 347.98 204.47 0)
+			(at 455.93 2.54 0)
 			(effects
 				(font
@@
 		)
 		(property "Description" "Power symbol creates a global label with name \"GND\" , ground"
-			(at 347.98 204.47 0)
+			(at 455.93 2.54 0)
 			(effects
 				(font

Commit message: alles verbunden
Parts:
- removed D4: SD103C, Diode_THT:D_DO-34_SOD68_P7.62mm_Horizontal, symbol Device:D_Schottky
- added D4: 1N4148, Diode_THT:D_DO-35_SOD27_P7.62mm_Horizontal, symbol Diode:1N4148
- R1, R2: now fitted
- R20, R24, R25, R7, R8, R9: now not fitted
- U9: value SG-531 -> 8_0000Mhz
Connections:
- net AVEC is gone; now on net VCC: U21.23 (~{AVEC})
- net BGACK is gone; now on net VCC: U21.13 (~{BGACK})
- net BR is gone; now on net VCC: C10.1, P1.a4 (Pin_a4), U21.14 (~{BR})
- net IPL2 is gone; now on net VCC: U21.25 (~{IPL2})
- net p1_c6 is gone; now on net RESET: D6.2 (A), P1.c6 (Pin_c6)
- net A1: now also U17.4
- net A19: no longer U2.31 (A18), U6.31 (A18)
- net AS: now also U13.5 (~{E1}), U16.11 (Load), U19.2, U19.4
- net BERR: now also U19.6, D4.1 (K)
- net DTACK: now also U12.11 (WDI), U20.6
- net EXT_A4: now also P1.b3 (Pin_b3)
- net EXT_A6: now also P1.a2 (Pin_a2)
- net FC0: now also U17.2
- net GND: now also BT1.2 (-), C14.2, C16.1
- net HALT: now also D5.2 (A), R16.1
- net IPL0: now also P2.a3 (Pin_a3)
- net LDS: now also U17.12
- net RESET: now also R14.1
- net UDS: now also U10.1, U17.13
- net VCC: now also C3.1, P2.a4 (Pin_a4)
- net Y4: now also U10.12
- net Y5: now also D8.1 (K), U15.12
- net Y6: now also U19.9, U20.12, U20.13
- net Y7: now also U10.9, U20.4
- net p1_b6: now also D7.2 (A), D8.2 (A), U20.1
- net at S1.2 (B): now also BT1.1 (+)
- net at C16.2, R13.1: now also R22.1, U19.5, D4.2 (A)
- net p1_a5: now reaches R15.2
- net p1_a5: now also P1.a5 (Pin_a5)
- net at U17.3, U18.3, U18.4: now also U13.4 (~{E0})
- net at U18.6: now also U19.1
- net p2_b2: now reaches U20.8
- net p2_b2: now also P2.b2 (Pin_b2)
- net at U2.24 (~{OE}), U6.24 (~{OE}): now also U10.11
- net at U12.1 (VBATT): now also D1.1 (K), R3.1
- net at U12.15 (~{RESET}): now also D5.1 (K), D6.1 (K)
- net at U12.5 (BATT_ON): now also Q1.2 (B)
- net at U12.6 (~{LOW_LINE}): now also R1.2, R17.2, R8.1, U22.15 (CS1)
- net at U12.8 (OSC_SEL): now also R23.2
- net p2_c3: now reaches U19.3
- net p2_c3: now also P2.c3 (Pin_c3), U17.9, U18.1, U18.10, U18.2
- net at U22.8 (~{RD}): now also U15.11
- net at U3.29 (~{WE}): now also U10.3
- net at U14.1 (OE), U18.12: now also U4.1 (OE)
- net p2_a2: now reaches U17.10, U18.13, U18.9, U19.8
- net p2_a2: now also P2.a2 (Pin_a2)
- net at U10.10, U10.13: now also U15.1, U15.13, U15.2, U15.4, U15.5, U15.9, U17.11, U19.10, U19.13
- net at R19.1, R24.2: now also U2.31 (A18), U6.31 (A18)
- net at U14.11 (Load): now also U18.8, U4.11 (Load)
- net p2_c2: now reaches U18.11
- net p2_c2: now also P2.c2 (Pin_c2), U19.11
- net A0: no longer names the net of U21.31 (A0)
- net A20: no longer names the net of U21.52 (A20)
- net A21: no longer names the net of U21.54 (A21)
- net BG: no longer names the net of U21.12 (~{BG})
- net FC2: no longer names the net of U21.28 (FC2)
- net p1_b5: no longer names the net of P1.b5 (Pin_b5)
- no-connect marks 5 -> 23
Other:
- moved on the sheet: BT1, C14, C16, C18, D3, D5, D6, D7, D8, Q1, R13, R14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

Commit message: battok
Parts:
- S1: value Jumper_2_Open -> Batterie
Connections:
- net ~{SPACE_VALID}: now reaches U13.4 (~{E0}), U17.3, U18.3, U18.4
- net BATT_OK: now reaches P2.a5 (Pin_a5), U12.10 (~{PFO})
- net ~{DATA_VALID}: now reaches U10.10, U10.13, U15.1, U15.13, U15.2, U15.4, U15.5, U15.9, U17.11, U19.10, U19.13
- net LDS renamed ~{LDS}
- net UDS renamed ~{UDS}
Other:
- moved on the sheet: BT1, C1, C10, C11, C12, C13, C14, C15, C16, C17, C18, C19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
