File: STE25/STE25.kicad_sch (KiCad schematic)
At the start: 43 parts, among them Q201 16.0, Q202 3.686, SW201 RESET, T201 BC547, T204 BC547, T205 BC547, T206 BC547, T207 BD679, T208 BD679, T209 BC556, T210 BC547, T211 BC547, T212 BC547

Commit message: oki du ar
Parts:
- added H201, H202, H203: MountingHole, MountingHole:MountingHole_4.3mm_M4, symbol Mechanical:MountingHole
- added ICC2: D70322L, Package_LCC:PLCC-84_THT-Socket, symbol FPGA_Microsemi:ACT1225PL84
- added ICC3: 74HC138, Package_DIP:DIP-16_W7.62mm, symbol 74xx:74HC138
- added ICC4: 74AS138, Package_DIP:DIP-16_W7.62mm, symbol 74xx:74LS138
- added ICC5: 74HC4050, Package_DIP:DIP-16_W7.62mm, symbol 4xxx:4050
- added ICD3, ICD5: 74HC04, Package_DIP:DIP-14_W7.62mm, symbol 74xx:74HC04
- added ICD4: 74HCT21, Package_DIP:DIP-14_W7.62mm, symbol 74xx:74LS21
- added ICE2: IS62C256AL, Package_DIP:DIP-28_W15.24mm, symbol Memory_RAM:IS62C256AL
- added ICE7: MSM6376, Package_LQFP:QFP-64_14x20_Pitch1mm, symbol OKI:MSM6376
- added ICF4: SCC2692AC1N28, Package_DIP:DIP-28_W15.24mm, symbol DUART:SCC2692AC
- added ICF5: 27C020, Package_DIP:DIP-32_W15.24mm, symbol Memory_EPROM:27C020
- added R201, R202, R203, R204, R205, R206, R207, R208, R209, R210, R211, R212, R213, R214, R215, R216, R217, R218, R219, R220, R221, R222, R223, R224, R225, R226, R227, R228, R229, R230, R231, R232, R233, R234, R235, R236, R237, R238, R241, R243, R245, R247, R248, R249, R250, R251, R252, R253, R254, R255, R256, R258, R259, R260, R261, R262, R263, R264, R265, R266, R267, R268, R269, R270, R271, R272, R273, R274, R275, R276, R277, R278, R279, R281, R282, R283, R284, R285, R286, R287, R288, R289, R290, R291, R292, R293, R294, R295, R296: R, Resistor_THT:R_Axial_DIN0207_L6.3mm_D2.5mm_P10.16mm_Horizontal, symbol Device:R
- added R239: 9A472G, Resistor_THT:R_Array_SIP9, symbol Device:R_Network08
- added R240, R244: 330, Resistor_THT:R_Axial_DIN0207_L6.3mm_D2.5mm_P10.16mm_Horizontal, symbol Device:R
- added R242, R246: 4.7k, Resistor_THT:R_Axial_DIN0207_L6.3mm_D2.5mm_P10.16mm_Horizontal, symbol Device:R
- added R257: 1.2k, Resistor_THT:R_Axial_DIN0207_L6.3mm_D2.5mm_P10.16mm_Horizontal, symbol Device:R
- added R280: 1, Resistor_THT:R_Axial_DIN0411_L9.9mm_D3.6mm_P25.40mm_Horizontal, symbol Device:R
- added R304: 180, Resistor_THT:R_Axial_Power_L20.0mm_W6.4mm_P25.40mm, symbol Device:R
- added RV202: LAUTSTAERKE, Potentiometer_THT:Potentiometer_ACP_CA14V-15_Vertical, symbol Device:R_Potentiometer
- added RV203: R_Potentiometer, Potentiometer_THT:Potentiometer_ACP_CA9-V10_Vertical, symbol Device:R_Potentiometer
- added STA2: Versorgungseinheit, Connector_Stocko:Stocko_MKS_1660-6-0-1010_1x10_P2.50mm_Vertical, symbol Connector_Generic:Conn_01x10
- added STB2: IOS, Connector_Stocko:Stocko_MKS_1658-6-0-808_1x8_P2.50mm_Vertical, symbol Connector_Generic:Conn_01x08
- added STC2, STD2, STE2: Conn_01x06, Connector_Stocko:Stocko_MKS_1656-6-0-606_1x6_P2.50mm_Vertical, symbol Connector_Generic:Conn_01x06
- added STG2: Service, Connector_PinSocket_2.54mm:PinSocket_1x13_P2.54mm_Vertical, symbol Connector_Generic:Conn_02x13_Counter_Clockwise
- added STH2: Lautsprecher, Connector_Stocko:Stocko_MKS_1651-6-0-202_1x2_P2.50mm_Vertical, symbol Connector_Generic:Conn_01x02
- added STK2: Alarm, Connector_Stocko:Stocko_MKS_1651-6-0-202_1x2_P2.50mm_Vertical, symbol Connector_Generic:Conn_01x02
- added STL2: Spielezähler, Connector_Stocko:Stocko_MKS_1651-6-0-202_1x2_P2.50mm_Vertical, symbol Connector_Generic:Conn_01x02
- added STM2: Tür, Connector_Stocko:Stocko_MKS_1656-6-0-606_1x6_P2.50mm_Vertical, symbol Connector_Generic:Conn_01x06
- added STP2: Tresorständer, Connector_Stocko:Stocko_MKS_1654-6-0-404_1x4_P2.50mm_Vertical, symbol Connector_Generic:Conn_01x04
- added STT2: Kartenleser, Connector_Stocko:Stocko_MKS_1656-6-0-606_1x6_P2.50mm_Vertical, symbol Connector_Generic:Conn_01x06
- added STU2: Duobetrieb, Connector_Stocko:Stocko_MKS_1656-6-0-606_1x6_P2.50mm_Vertical, symbol Connector_Generic:Conn_01x06
- added STV2, STW2: Conn_01x04, Connector_Stocko:Stocko_MKS_1654-6-0-404_1x4_P2.50mm_Vertical, symbol Connector_Generic:Conn_01x04
- added ZD201: D_Zener, Diode_THT:D_T-1_P12.70mm_Horizontal, symbol Device:D_Zener
- STR2: renamed from ST18; value DE9_Socket -> DATAprint
Connections:
- net at D201.2 (A): now also R257.2
- net at T204.1 (C): now also ICA3.2, SW201.1
- net GND: now reaches T204.3 (E)
- net GND: now also R304.2, STA2.1 (Pin_1), STC2.6 (Pin_6), STD2.6 (Pin_6), STE2.6 (Pin_6), STM2.2 (Pin_2), STP2.1 (Pin_1), STT2.6 (Pin_6)
- net at ICA4.1: now also SW201.2
- net at ICA3.12: now also ICA3.10
- net at Q202.1: now also ICF4.24 (X2)
- net at Q202.2: now also ICF4.23 (X1/CLK)
- net at ICA6.5: now also ICA6.2
- net at D211.1 (K): now also D210.2 (A)
- net at D211.2 (A): now also D212.1 (K)
- net +5V: now reaches C216.1
- net +5V: now also STA2.4 (Pin_4), ZD201.1 (K)
- net GND2: now reaches C216.2
- net GND2: now also STA2.10 (Pin_10), STU2.6 (Pin_6), ZD201.2 (A)
- net at D212.2 (A): now also D213.1 (K)
- net at R310.2 (R1): now also STW2.1 (Pin_1)
- net at R310.3 (R2): now also STW2.2 (Pin_2)
- net at R310.4 (R3): now also STW2.3 (Pin_3)
- net at R310.5 (R4): now also STW2.4 (Pin_4)
- net at R310.8 (R7): now also R246.2
- net at R310.9 (R8): now also R242.2
- net +12V: now reaches D210.1 (K)
- net +12V: now also STP2.4 (Pin_4)
- net +15V: now reaches D213.2 (A)
- net +15V: now also C202.1, STA2.2 (Pin_2), STA2.3 (Pin_3), STC2.1 (Pin_1), STD2.1 (Pin_1), STE2.1 (Pin_1), STL2.2 (Pin_2), STM2.4 (Pin_4), STT2.1 (Pin_1), STU2.1 (Pin_1)
- net at C203.1: now also R280.1
- net at ICB4.12 (I5): now also ICB4.14 (I6)
- new net: R276.1, R283.1
- new net: ICD4.4, ICD4.5
- new net: R244.1, STT2.4 (Pin_4)
- new net: R246.1, STT2.5 (Pin_5)
- new net ALARM: STK2.1 (Pin_1)
- new net DB_RTS2: STU2.4 (Pin_4)
- new net DB_RXD2: STU2.3 (Pin_3)
- new net DB_TXD2: STU2.2 (Pin_2)
- new net IOS_CLOCK_IN: STB2.3 (Pin_3)
- new net IOS_CLOCK_OUT: STB2.7 (Pin_7)
- new net IOS_DATA_IN: STB2.5 (Pin_5)
- new net IOS_DATA_OUT: STB2.1 (Pin_1)
- new net IOS_LOAD_IN: STB2.2 (Pin_2)
- new net IOS_LOAD_MOT: STB2.4 (Pin_4)
- new net IOS_LOAD_OUT: STB2.6 (Pin_6)
- new net KL_RX: R242.1, STT2.3 (Pin_3)
- new net KL_TX: R240.1, STT2.2 (Pin_2)
- new net LSP1: STH2.1 (Pin_1)
- new net LSP2: STH2.2 (Pin_2)
- new net MONEY_RXD: STC2.3 (Pin_3), STD2.3 (Pin_3), STE2.3 (Pin_3)
- new net MONEY_TXD: R273.1, STC2.2 (Pin_2), STD2.2 (Pin_2), STE2.2 (Pin_2)
- new net P0.4: STL2.1 (Pin_1)
- new net READY: R210.2, STC2.5 (Pin_5), STD2.5 (Pin_5), STE2.5 (Pin_5)
- new net RESET: STB2.8 (Pin_8), STC2.4 (Pin_4), STD2.4 (Pin_4), STE2.4 (Pin_4), STM2.1 (Pin_1)
- new net RESET_ASY: STU2.5 (Pin_5)
- new net TRESOR_DATA_IN: STP2.2 (Pin_2)
- new net TRESOR_DATA_OUT: STP2.3 (Pin_3)
- new net TUER_MELDUNG: STM2.3 (Pin_3)
- new net TUER_TASTE: STM2.5 (Pin_5)
- no-connect marks 0 -> 14
Other:
- moved on the sheet: C203, D210, D212, D213, ICA3A, ICA4A, ICA6B, ICF1, ICF2, Q202, R310, SW201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

Commit message: ste
Parts:
- removed ICC2: D70322L, Package_LCC:PLCC-84_THT-Socket, symbol FPGA_Microsemi:ACT1225PL84
- added C210: 33uF 35V, Capacitor_THT:CP_Radial_D8.0mm_P5.00mm, symbol Device:C_Polarized
- added C220, C221: 15p, Capacitor_THT:C_Disc_D4.3mm_W1.9mm_P5.00mm, symbol Device:C
- added C222, C223: 47, Capacitor_THT:C_Disc_D4.3mm_W1.9mm_P5.00mm, symbol Device:C
- added ICC2: uPD70322L-8-232, Package_LCC:PLCC-84_THT-Socket, symbol NEC:uPD70325
- added LB1, LB2, LB3: Jumper_2_Open, TestPoint:TestPoint_2Pads_Pitch2.54mm_Drill0.8mm, symbol Jumper:Jumper_2_Open
- added R301, R325: R, Resistor_THT:R_Axial_DIN0207_L6.3mm_D2.5mm_P10.16mm_Horizontal, symbol Device:R
- added STS2: ~, Connector_Stocko:Stocko_MKS_1651-6-0-202_1x2_P2.50mm_Vertical, symbol Connector_Generic:Conn_01x02
Connections:
- net GND: now also ICD5.7 (GND), T207.3 (E), T208.3 (E), C220.2, C221.2, ICC2.42 (GND), ICC2.46 (~{CTS1}), ICC2.77 (GND)
- net TRESOR_DATA_OUT: now also T207.2 (C)
- net at T210.1 (C): now also T211.2 (B)
- net at T212.2 (B): now also ICB2.5 (~{RESET})
- net D0: now reaches ICF1.2 (D0)
- net D0: now also ICC2.13 (D0)
- net D1: now reaches ICF1.3 (D1)
- net D1: now also ICC2.14 (D1)
- net D2: now reaches ICF1.4 (D2)
- net D2: now also ICC2.15 (D2)
- net D3: now reaches ICF1.5 (D3)
- net D3: now also ICC2.16 (D3)
- net D4: now reaches ICF1.6 (D4)
- net D4: now also ICC2.17 (D4)
- net D5: now reaches ICF1.7 (D5)
- net D5: now also ICC2.18 (D5)
- net D6: now reaches ICF1.8 (D6)
- net D6: now also ICC2.19 (D6)
- net D7: now reaches ICF1.9 (D7)
- net D7: now also ICC2.20 (D7)
- net at Q201.1: now also R287.2, C220.1, ICC2.78 (X1)
- net at Q201.2: now also C221.1, ICC2.79 (X2)
- net at R206.2: now also ICC2.49 (IC)
- new net A0: ICC2.21 (A0)
- new net A1: ICC2.22 (A1)
- new net A10: ICC2.31 (A10)
- new net A11: ICC2.32 (A11)
- new net A12: ICC2.33 (A12)
- new net A13: ICC2.34 (A13)
- new net A14: ICC2.35 (A14)
- new net A15: ICC2.36 (A15)
- new net A16: ICC2.37 (A16)
- new net A17: ICC2.38 (A17)
- new net A18: ICC2.39 (A18)
- new net A19: ICC2.40 (A19)
- new net A2: ICC2.23 (A2)
- new net A3: ICC2.24 (A3)
- new net A4: ICC2.25 (A4)
- new net A5: ICC2.26 (A5)
- new net A6: ICC2.27 (A6)
- new net A7: ICC2.28 (A7)
- new net A8: ICC2.29 (A8)
- new net A9: ICC2.30 (A9)
Other:
- moved on the sheet: ICB2, Q201, R206, R266, R287, T207, T208, T211, T212

Commit message: ste25
Parts:
- added C224: 1uF 100V, Capacitor_THT:CP_Radial_D8.0mm_P5.00mm, symbol Device:C_Polarized
- added C233, C242: 4.7uF 100V, Capacitor_THT:CP_Radial_D8.0mm_P5.00mm, symbol Device:C_Polarized
- added C253, C276: 100nF, Capacitor_THT:C_Disc_D4.3mm_W1.9mm_P5.00mm, symbol Device:C
- added C265: C, Capacitor_THT:C_Disc_D4.3mm_W1.9mm_P5.00mm, symbol Device:C
- added C268, C269: 27, Capacitor_THT:C_Disc_D4.3mm_W1.9mm_P5.00mm, symbol Device:C
- added C280, C281, C282, C283, C284, C285: 271, Capacitor_THT:C_Disc_D4.3mm_W1.9mm_P5.00mm, symbol Device:C
- added D209: BAT85, Diode_THT:D_DO-35_SOD27_P10.16mm_Horizontal, symbol Diode:BAT48RL
- added D238, D240, D246: BAT85, Diode_THT:D_DO-35_SOD27_P10.16mm_Horizontal, symbol Diode:BAT85
- added H204, H205: MountingHole, MountingHole:MountingHole_2.5mm, symbol Mechanical:MountingHole
- added LB12: Jumper_2_Open, TestPoint:TestPoint_2Pads_Pitch2.54mm_Drill0.8mm, symbol Jumper:Jumper_2_Bridged
- added LB14, LB4, LB5: Jumper_2_Open, TestPoint:TestPoint_2Pads_Pitch2.54mm_Drill0.8mm, symbol Jumper:Jumper_2_Open
- added R327: R, Resistor_THT:R_Axial_DIN0207_L6.3mm_D2.5mm_P10.16mm_Horizontal, symbol Device:R
- added R332, R340, R341, R342, R343: 4.7k, Resistor_THT:R_Axial_DIN0207_L6.3mm_D2.5mm_P10.16mm_Horizontal, symbol Device:R
- added R333, R334, R335, R336: 330, Resistor_THT:R_Axial_DIN0207_L6.3mm_D2.5mm_P10.16mm_Horizontal, symbol Device:R
- R241, R245: value R -> 330
- R243: value R -> 4.7k
- R260: value R -> 1.2k
- ZD201: footprint Diode_THT:D_T-1_P12.70mm_Horizontal -> Resistor_THT:R_Axial_DIN0309_L9.0mm_D3.2mm_P20.32mm_Horizontal
- renumbered ST2 to BU1, ST1 to BU2, D201 to LED201, D202 to LED202, RV202 to P202, RV203 to P203
Connections:
- net A0: now also BU2.b12 (Pin_b12), ICE2.10 (A0), ICF4.1 (A0)
- net A1: now also BU2.b11 (Pin_b11), ICE2.9 (A1), ICF4.2 (A1)
- net A10: now also BU2.a10 (Pin_a10)
- net A11: now also BU2.a8 (Pin_a8)
- net A12: now also BU2.b4 (Pin_b4)
- net A13: now also BU2.a5 (Pin_a5), ICC3.1 (A0)
- net A14: now also BU2.b3 (Pin_b3), ICC3.2 (A1)
- net A15: now also BU2.a3 (Pin_a3), ICC3.3 (A2)
- net A16: now also BU2.b1 (Pin_b1)
- net A17: now also BU2.a2 (Pin_a2), ICC4.1 (A0)
- net A18: now also BU1.b1 (Pin_b1), ICC4.2 (A1)
- net A19: now also ICC4.3 (A2)
- net A2: now also BU2.b10 (Pin_b10), ICE2.8 (A2), ICF4.3 (A2)
- net A3: now also BU2.b9 (Pin_b9), ICE2.7 (A3), ICF4.4 (A3)
- net A4: now also BU2.b8 (Pin_b8), ICE2.6 (A4)
- net A5: now also BU2.b7 (Pin_b7), ICE2.5 (A5)
- net A6: now also BU2.b6 (Pin_b6), ICE2.4 (A6)
- net A7: now also BU2.b5 (Pin_b5), ICE2.3 (A7)
- net A8: now also BU2.a6 (Pin_a6)
- net A9: now also BU2.a7 (Pin_a7)
- net D0: now also BU2.b13 (Pin_b13), ICE2.11 (I/O0), ICF2.2 (A0), ICF4.19 (D0), R239.2 (R1)
- net D1: now also BU2.b14 (Pin_b14), ICE2.12 (I/O1), ICF2.3 (A1), ICF4.10 (D1), R239.3 (R2)
- net D2: now also BU2.b16 (Pin_b16), ICE2.13 (I/O2), ICF2.4 (A2), ICF4.18 (D2), R239.4 (R3)
- net D3: now also BU2.a16 (Pin_a16), ICE2.15 (I/O3), ICF2.5 (A3), ICF4.11 (D3)
- net D4: now also BU2.a15 (Pin_a15), ICE2.16 (I/O4), ICF2.6 (A4), ICF4.17 (D4)
- net D5: now also BU2.a14 (Pin_a14), ICE2.17 (I/O5), ICF2.7 (A5), ICF4.12 (D5)
- net D6: now also BU2.a13 (Pin_a13), ICE2.18 (I/O6), ICF2.8 (A6), ICF4.16 (D6)
- net D7: now also BU2.a12 (Pin_a12), ICE2.19 (I/O7), ICF2.9 (A7), ICF4.13 (D7)
- net DB_RTS2: now also R245.2; no longer STU2.4 (Pin_4)
- net DB_RXD2: now also R243.2, R310.7 (R6), D246.1 (K); no longer STU2.3 (Pin_3)
- net DB_TXD2: now also R241.2; no longer STU2.2 (Pin_2)
- net GND: now also BU2.a1 (Pin_a1), C222.2, ICA4.7 (GND), ICA5.7 (GND), ICA6.7 (GND), ICC3.8 (GND), ICC4.8 (GND), ICD3.7 (GND), ICD4.7 (GND), ICE2.14 (GND), ICF1.10 (GND), ICF2.1 (A->B), ICF2.10 (GND), ICF5.16 (GND), STG2.1 (Pin_1), STG2.13 (Pin_13), T201.3 (E), T211.3 (E), T212.3 (E), C233.2, C268.1, C269.1, C280.1, C283.1, C284.2, C285.1
- net IOS_LOAD_IN: now also ICD3.8, C285.2
- net IOS_LOAD_MOT: now also ICD3.6, C284.1
- net IOS_LOAD_OUT: now also ICA5.2, ICD3.4
- net KL_RX: now also R242.2, R310.9 (R8), D240.1 (K); no longer R242.1, STT2.3 (Pin_3)
- net KL_TX: now also R240.2; no longer R240.1, STT2.2 (Pin_2)
- net RESET: no longer STB2.8 (Pin_8)
- net VCC: now reaches ICA5.14 (VCC)
- net VCC: now also ICA3.14 (VCC), ICA4.14 (VCC), ICA6.14 (VCC), ICB1.16 (VCC), ICB2.8 (VCC), ICB4.16 (VCC), ICC2.50 (VDD), ICC2.76 (VTH), ICC2.80 (VDD), ICC3.16 (VCC), ICC4.16 (VCC), ICC5.1 (VCC), ICD3.14 (VCC), ICD4.14 (VCC), ICD5.14 (VCC), ICE2.28 (VDD), ICF1.20 (VCC), ICF5.32 (VCC), R206.1, R207.1, R239.1 (common), R257.1, R260.1, R266.1, R308.1 (common), R325.2, STG2.7 (Pin_7)
- net at LED201.1 (K): now also T212.1 (C)
- net ~{SERVICE_DATA}: now reaches ICD5.3
- net ~{SERVICE_DATA}: now also ICC2.44 (TxD0)
- net SERVICE_DATA: now reaches ICD5.4
- net SERVICE_DATA: now also STG2.5 (Pin_5)
- net at R301.2: now also ICE7.12 (OSC1)
- net at ICF4.24 (X2), Q202.1: now also C268.2
- net at ICF4.23 (X1/CLK), Q202.2: now also C269.2
- net at R260.2: now also LED202.2 (A)
- net at ICF2.15 (B3): now also R343.1
- net at ICF2.16 (B2): now also R342.1
- net at ICF2.17 (B1): now also R341.1
- net at ICF2.18 (B0): now also R340.1
- net at ICD3.9: now also ICC3.12 (~{Y3})
- net SOUND_I0: now reaches R308.2 (R1)
- net SOUND_I0: now also ICC2.48 (P20/DMARQ0), ICE7.22 (I0)
- net SOUND_I1: now reaches R308.3 (R2)
- net SOUND_I1: now also ICC2.51 (P21/~{DMAAK0}), ICE7.23 (I1)
- net SOUND_I2: now reaches R308.4 (R3)
- net SOUND_I2: now also ICC2.52 (P22/~{TC0}), ICE7.24 (I2)
- net SOUND_I3: now reaches R308.5 (R4)
- net SOUND_I3: now also ICC2.54 (P23/DMARQ1), ICE7.25 (I3)
- net SOUND_I4: now reaches R308.6 (R5)
- net SOUND_I4: now also ICC2.55 (P24/~{DMAAK1}), ICE7.26 (I4)
- net SOUND_I5: now reaches R308.7 (R6)
- net SOUND_I5: now also ICC2.56 (P25/~{TC1}), ICE7.27 (I5)
- net SOUND_I6: now reaches R308.8 (R7)
- net SOUND_I6: now also ICC2.57 (P26/~{HLDAK}), ICE7.28 (I6)
- net at ICD5.1: now also ICA5.1
- net NVRAM_E1: now reaches ICC4.10 (O5)
- net NVRAM_E1: now also BU2.a9 (Pin_a9)
- net at ICC4.11 (O4): now also ICD4.13
- net at ICC4.12 (O3): now also ICD4.12
- net at ICC4.13 (O2): now also ICD4.10
- net at ICC4.14 (O1): now also ICD4.9, LB12.1 (A)
- net RAM_CE: now reaches ICC4.15 (O0)
- net RAM_CE: now also ICE2.20 (~{CE})
- net at STV2.1 (Pin_1): now also R333.1
- net at STV2.2 (Pin_2): now also R334.1
- net at STV2.3 (Pin_3): now also R335.1
- net at STV2.4 (Pin_4): now also R336.1
- net IO5: now reaches ICC3.10 (~{Y5})
- net IO5: now also D209.1 (K)
- net IO4: now reaches ICC3.11 (~{Y4})
- net IO4: now also ICB1.9 (A)
- net at ICC3.13 (~{Y2}): now also ICD3.5
- net at ICC3.14 (~{Y1}): now also ICD3.3
- net at ICC3.15 (~{Y0}): now also ICD3.11
- net UART_CE: now reaches ICC3.4 (~{E0})
- net UART_CE: now also ICF4.26 (CEN)
- net IO7: now reaches ICC3.7 (~{Y7})
- net IO6: now reaches ICC3.9 (~{Y6})
- net at ICB1.5 (Q): now also LED202.1 (K)
- net at R288.1: now also P203.3
- net C_DB_TXD2: now reaches R241.1
- net C_DB_TXD2: now also STU2.2 (Pin_2)
- net C_DB_RTS2: now reaches R245.1
- net C_DB_RTS2: now also STU2.4 (Pin_4)
- net SERVICE_STROBE: now reaches STG2.3 (Pin_3)
- net SERVICE_STROBE: now also ICD3.10
- net SERVICE_CLK: now reaches STG2.9 (Pin_9)
- net SERVICE_CLK: now also ICC5.15, C282.1
- net NVRAM_W: now reaches ICA3.8
- net NVRAM_W: now also BU2.a4 (Pin_a4)
- net at ICF1.1 (OE): now also ICD5.6
- net at ICF1.16 (Q3): now also R336.2
- net at ICF1.17 (Q2): now also R335.2
- net at ICF1.18 (Q1): now also R334.2
- net at ICF1.19 (Q0): now also R333.2
- net at C223.1: now also C265.1
- net at C223.2: now also ICE7.15 (OSC3), C265.2
- net at R310.2 (R1), STW2.1 (Pin_1): now also R340.2
- net at R310.3 (R2), STW2.2 (Pin_2): now also R341.2
- net at R310.4 (R3), STW2.3 (Pin_3): now also R342.2
- net at R310.5 (R4), STW2.4 (Pin_4): now also R343.2
- net SND_A2: now reaches ICF5.10 (A2)
- net SND_A2: now also BU1.b11 (Pin_b11), ICE7.43 (A2)
- net SND_A1: now reaches ICF5.11 (A1)
- net SND_A1: now also BU1.a12 (Pin_a12), ICE7.42 (A1)
- net SND_A0: now reaches ICF5.12 (A0)
- net SND_A0: now also BU1.b12 (Pin_b12), ICE7.41 (A0)
- net SND_D0: now reaches ICF5.13 (D0)
- net SND_D0: now also BU1.b16 (Pin_b16), ICE7.31 (D0)
- net SND_D1: now reaches ICF5.14 (D1)
- net SND_D1: now also BU1.a16 (Pin_a16), ICE7.32 (D1)
- net SND_D2: now reaches ICF5.15 (D2)
- net SND_D2: now also BU1.a2 (Pin_a2), ICE7.35 (D2)
- net SND_D3: now reaches ICF5.17 (D3)
- net SND_D3: now also BU1.a15 (Pin_a15), ICE7.36 (D3)
- net SND_D4: now reaches ICF5.18 (D4)
- net SND_D4: now also BU1.b14 (Pin_b14), ICE7.37 (D4)
- net SND_D5: now reaches ICF5.19 (D5)
- net SND_D5: now also BU1.a14 (Pin_a14), ICE7.38 (D5)
- net SND_D6: now reaches ICF5.20 (D6)
- net SND_D6: now also BU1.b13 (Pin_b13), ICE7.39 (D6)
- net SND_D7: now reaches ICF5.21 (D7)
- net SND_D7: now also BU1.a13 (Pin_a13), ICE7.40 (D7)
- net SND_ROM_CE: now reaches ICF5.22 (~{CE})
- net SND_A10: now reaches ICF5.23 (A10)
- net SND_A10: now also BU1.b7 (Pin_b7), ICE7.52 (A10)
- net SND_ROM_OE: now reaches ICF5.24 (~{OE})
- net SND_A9: now reaches ICF5.26 (A9)
- net SND_A9: now also BU1.a8 (Pin_a8), ICE7.50 (A9)
- net SND_A8: now reaches ICF5.27 (A8)
- net SND_A8: now also BU1.b8 (Pin_b8), ICE7.49 (A8)
- net SND_A7: now reaches ICF5.5 (A7)
- net SND_A7: now also BU1.a9 (Pin_a9), ICE7.48 (A7)
- net SND_A6: now reaches ICF5.6 (A6)
- net SND_A6: now also BU1.b9 (Pin_b9), ICE7.47 (A6)
- net SND_A5: now reaches ICF5.7 (A5)
- net SND_A5: now also BU1.a10 (Pin_a10), ICE7.46 (A5)
- net SND_A4: now reaches ICF5.8 (A4)
- net SND_A4: now also BU1.b10 (Pin_b10), ICE7.45 (A4)
- net SND_A3: now reaches ICF5.9 (A3)
- net SND_A3: now also BU1.a11 (Pin_a11), ICE7.44 (A3)
- net at C222.1: now also ICE7.17 (~{ST}), R266.2, D209.2 (A)
- net ~{SERVICE_CLK}: now reaches ICC5.14
- net ~{SERVICE_CLK}: now also ICC2.65 (P16/~{SCK0})
- net at ICC5.2: now also ICC5.7, ICD5.5
- net at T209.3 (E): now also ICB2.2 (~{RESIN})
- net UART_WE: now reaches ICF4.5 (WRN)
- net UART_RE: now reaches ICF4.6 (RDN)
- net at R246.2, R310.8 (R7): now also D238.1 (K)
- net at P203.1: now also ICE7.13 (OSC2)
- net PRG_CE: now reaches BU2.a11 (Pin_a11)
- net PRG_CE: now also ICD4.8
- net PRG_OE: now reaches BU1.a1 (Pin_a1)
- net SND_OE: now reaches BU1.a3 (Pin_a3)
- net SND_A17: now reaches BU1.a4 (Pin_a4)
- net SND_A17: now also ICE7.59 (A17)
- net SND_A15: now reaches BU1.a5 (Pin_a5)
- net SND_A15: now also ICE7.57 (A15)
- net SND_A13: now reaches BU1.a6 (Pin_a6)
- net SND_A13: now also ICE7.55 (A13)
- net SND_A11: now reaches BU1.a7 (Pin_a7)
- net SND_A11: now also ICE7.53 (A11)
- net SND_CE: now reaches BU1.b2 (Pin_b2)
- net SND_A18: now reaches BU1.b3 (Pin_b3)
- net SND_A18: now also ICE7.60 (A18)
- net SND_A16: now reaches BU1.b4 (Pin_b4)
- net SND_A16: now also ICE7.58 (A16)
- net SND_A14: now reaches BU1.b5 (Pin_b5)
- net SND_A14: now also ICE7.56 (A14)
- net SND_A12: now reaches BU1.b6 (Pin_b6)
- net SND_A12: now also ICE7.54 (A12)
- net P13: now reaches ICE7.1 (~{BUSY})
- net P13: now also ICC2.62 (P13/~{INTP2}/~{INTAK})
- net C_DB_RXD2: now reaches R243.1
- net C_DB_RXD2: now also STU2.3 (Pin_3)
- net at ICB4.11 (O5b): now also ICB4.13 (O6b)
- net RAM_OE: now reaches ICE2.22 (~{OE})
- net RAM_WE: now reaches ICE2.27 (~{WE})
- new net: LB12.2 (B), LB14.1 (A)
- new net C_KL_RX: R242.1, STT2.3 (Pin_3)
- new net C_KL_TX: R240.1, STT2.2 (Pin_2)
- new net OE_PERIPH: STB2.8 (Pin_8)
- no-connect marks 14 -> 15
Other:
- moved on the sheet: BU1, C222, C223, ICA3E, ICA6E, ICB1B, ICC3, ICC4, ICC5A, ICC5C, ICC5G, ICD3B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

Commit message: io
Parts:
- removed R231: R, Resistor_THT:R_Axial_DIN0207_L6.3mm_D2.5mm_P10.16mm_Horizontal, symbol Device:R
- added C228, C244, C246, C248, C249, C250, C251, C252, C254, C256, C257, C258, C259, C260, C261, C263, C274, C275: 104, Capacitor_THT:C_Disc_D6.0mm_W2.5mm_P5.00mm, symbol Device:C
- added D215, D216, D217, D218, D219, D220, D221, D222, D223, D224, D225, D226: BAT85, Diode_THT:D_DO-35_SOD27_P10.16mm_Horizontal, symbol Diode:BAT48RL
- added LB7: Spielmodul Sound A19, NSM:NSM_Jumper, symbol Jumper:Jumper_2_Bridged
- added LB8: Spielmodul Sound A20, NSM:NSM_Jumper, symbol Jumper:Jumper_2_Open
- added R328, R329: 10k, Resistor_THT:R_Axial_DIN0207_L6.3mm_D2.5mm_P10.16mm_Horizontal, symbol Device:R
- C253, C276: value 100nF -> 104; footprint Capacitor_THT:C_Disc_D4.3mm_W1.9mm_P5.00mm -> Capacitor_THT:C_Disc_D6.0mm_W2.5mm_P5.00mm
- ICF5: value 27C020 -> 27C4001; symbol Memory_EPROM:27C020 -> Memory_EPROM:27C040
- LB1, LB12, LB14, LB2, LB3, LB5: footprint TestPoint:TestPoint_2Pads_Pitch2.54mm_Drill0.8mm -> NSM:NSM_Jumper
- LB4: footprint TestPoint:TestPoint_2Pads_Pitch2.54mm_Drill0.8mm -> NSM:NSM_Jumper; symbol Jumper:Jumper_2_Open -> Jumper:Jumper_2_Bridged
- R223: value R -> 1k
- R228, R229: value R -> 10k
- R231: renamed from R251; value R -> 4.7K
- R237: value R -> 4.7K
- R279: value R -> 820
Connections:
- net SND_ROM_OE is gone; now on net SND_OE: ICF5.24 (~{OE})
- net UART_CE is gone; now on net ~{IOSTB}: ICC3.4 (~{E0}), ICF4.26 (CEN)
- net UART_RE is gone; now on net UART_RD: ICF4.6 (RDN)
- net UART_WE is gone; now on net UART_WR: ICF4.5 (WRN)
- net +5V: now also C261.1
- net GND: now also C204.2, ICA3.7 (GND), C228.2, C244.2, C246.2, C248.2, C249.2, C250.2, C251.2, C252.2, C254.2, C256.2, C257.2, C258.2, C259.2, C260.2, C263.2, C274.2, C275.2
- net IO6: now also ICA6.2, ICA6.5
- net IOS_DATA_OUT: now also C281.2, ICA4.6
- net SND_A11: now also ICF5.25 (A11)
- net SND_A12: now also ICF5.4 (A12)
- net SND_A13: now also ICF5.28 (A13)
- net SND_A14: now also ICF5.29 (A14)
- net SND_A15: now also ICF5.3 (A15)
- net SND_A16: now also ICF5.2 (A16)
- net SND_A17: now also ICF5.30 (A17)
- net SND_A18: now also ICF5.31 (A18)
- net SND_CE: now also R308.9 (R8), LB7.1 (A), LB8.1 (A)
- net SND_OE: now also ICE7.29 (~{OE})
- net SND_ROM_CE: now also BU1.b15 (Pin_b15)
- net VCC: now also ICF2.20 (VCC), LB4.1 (A), C244.1, C249.1, C250.1, C251.1, C252.1, C254.1, C256.1, C257.1, C258.1, C259.1, C260.1, C263.1, C274.1, C275.1
- net SND_A19: now reaches LB5.1 (A)
- net SND_A19: now also ICE7.61 (A19), STS2.2 (Pin_2), LB7.2 (B)
- net at LB5.2 (B): now also ICF5.1 (VPP), LB4.2 (B)
- net at R332.1: now also BU2.b15 (Pin_b15)
- net UART_RD: now reaches ICA6.6
- net RW: now reaches ICA6.1
- net RW: now also ICC2.83 (R/~{W})
- net UART_WR: now reaches ICA6.3
- net at R231.1: now also ICC2.11 (P06)
- net at R231.2: now also R229.2
- net SND_A20: now reaches STS2.1 (Pin_1)
- net SND_A20: now also ICE7.62 (A20), LB8.2 (B)
- net at ICA4.4: now also ICA5.11
- net KB5: now reaches STG2.10 (Pin_10)
- net KB6: now reaches STG2.12 (Pin_12)
- net KB1: now reaches STG2.2 (Pin_2)
- net KB2: now reaches STG2.4 (Pin_4)
- net KB3: now reaches STG2.6 (Pin_6)
- net KB4: now reaches STG2.8 (Pin_8)
- net at C204.1: now also ICC7.9 (V+), C228.1
- net at ICB2.2 (~{RESIN}), T209.3 (E): now also C246.1
- net UART_INT: now reaches ICF4.15 (INTRN)
- net UART_INT: now also ICC2.61 (P12/~{INTP1})
- net TXDA: now reaches ICF4.21 (TxDA)
- net RXDA: now reaches ICF4.22 (RxDA)
- net RXDB: now reaches ICF4.7 (RxDB)
- net TXDB: now reaches ICF4.8 (TxDB)
- net at R223.2: now also D221.1 (K)
- net ~{IOSTB}: now reaches ICC2.1 (~{IOSTB})
- net P13 renamed ~{SOUND_BUSY}
Other:
- moved on the sheet: BU1, C204, C222, C223, C265, C281, D209, ICA3B, ICA3C, ICA3D, ICA4B, ICA5D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
