File: STE25/STE25.kicad_sch (KiCad schematic)
At the start: 251 parts, among them P202 LAUTSTAERKE, P203 R_Potentiometer, Q201 16.0, Q202 3.686, SW201 RESET, T201 BC547, T204 BC547, T205 BC547, T206 BC547, T207 BD679, T208 BD679, T209 BC556, T210 BC547, T211 BC547, T212 BC547

Commit message: ste25 serial
Parts:
- added D208: BAT85, Diode_THT:D_DO-35_SOD27_P10.16mm_Horizontal, symbol Diode:BAT48RL
- STS2: value ~ -> (none)
Connections:
- net DB_TXD2 is gone; now on net TXDB: R241.2
- net KL_RX is gone; now on net RXDA: D240.1 (K), R242.2, R310.9 (R8)
- net KL_TX is gone; now on net TXDA: R240.2
- net DB_RXD2: no longer D246.1 (K), R243.2
- net GND: now also C203.2, STR2.5
- net MONEY_RXD: now also D208.1 (K)
- net RXDB: now also D246.1 (K), R243.2
- net MONEY_TXD_L: now reaches R273.2
- net MONEY_TXD_L: now also ICB4.11 (O5b), ICB4.13 (O6b)
- net PRINTER_RX: now reaches R327.1
- net PRINTER_RX: now also STR2.2
- net PRINTER_RX_L: now reaches R327.2
- net PRINTER_RX_L: now also ICD5.12
- net PRINTER_DSR: now reaches STR2.6
- net ~{PRINTER_RX_L}: now reaches ICD5.13
- net ~{PRINTER_RX_L}: now also ICA5.8
- net RX1: now reaches ICC2.45 (RxD1)
- net TX1: now reaches ICC2.47 (TxD1)
- net TX1: now also ICB4.12 (I5), ICB4.14 (I6)
