File: Adapter68000/Adapter68000.kicad_pcb (KiCad board)
At the start: 2 copper layers, 131.5 x 55 mm, 34 parts, among them P22 Service-Tast.

Commit message: dicke fertig
Parts:
- added C1: 100nF, Capacitor_THT:C_Axial_L3.8mm_D2.6mm_P7.50mm_Horizontal, F.Cu at (171.8, 116.5)
- added C10: 100nF, Capacitor_THT:C_Axial_L3.8mm_D2.6mm_P7.50mm_Horizontal, F.Cu at (184.5, 81.8)
- added C2: 100nF, Capacitor_THT:C_Axial_L3.8mm_D2.6mm_P7.50mm_Horizontal, F.Cu at (159.0, 116.5)
- added C3: 4.7uF 63V, Capacitor_THT:CP_Axial_L11.0mm_D5.0mm_P18.00mm_Horizontal, F.Cu at (136.5, 115.5)
- added C4: 100nF, Capacitor_THT:C_Axial_L3.8mm_D2.6mm_P7.50mm_Horizontal, F.Cu at (192.2, 106.2)
- added C5: 100nF, Capacitor_THT:C_Axial_L3.8mm_D2.6mm_P7.50mm_Horizontal, F.Cu at (184.5, 91.5)
- added C6: 100nF, Capacitor_THT:C_Axial_L3.8mm_D2.6mm_P7.50mm_Horizontal, F.Cu at (171.5, 91.5)
- added C7: 100nF, Capacitor_THT:C_Axial_L3.8mm_D2.6mm_P7.50mm_Horizontal, F.Cu at (159.0, 91.5)
- added C8: 100nF, Capacitor_THT:C_Axial_L3.8mm_D2.6mm_P7.50mm_Horizontal, F.Cu at (184.5, 86.5)
- added C9: 100nF, Capacitor_THT:C_Axial_L3.8mm_D2.6mm_P7.50mm_Horizontal, F.Cu at (184.5, 84.0)
- added D1: 1N4148, Diode_THT:D_DO-35_SOD27_P7.62mm_Horizontal, F.Cu at (123.5, 113.5)
- added D2: 1N4148, Diode_THT:D_DO-35_SOD27_P7.62mm_Horizontal, F.Cu at (123.5, 116.0)
- added P21: Conn_01x20_Male, Connector_Stocko:Stocko_MKS_1670-6-0-2020_1x20_P2.50mm_Vertical, F.Cu at (98.2, 69.5)
- added U1: 74HC107, Package_DIP:DIP-14_W7.62mm, F.Cu at (171.8, 96.3)
- added U2: 74HC165, Package_DIP:DIP-16_W7.62mm, F.Cu at (159.0, 96.2)
- added U3: 74HC4094, Package_DIP:DIP-16_W7.62mm, F.Cu at (171.5, 71.5)
- added U4: 74HC4094, Package_DIP:DIP-16_W7.62mm, F.Cu at (159.0, 71.5)
- P22: footprint Connector_PinHeader_2.54mm:PinHeader_1x06_P2.54mm_Vertical -> Connector_Lumberg:Lumberg_MSF_B6B-MSF-A_1x06_P2.50mm_Vertical
- R12, R15, R18, R20, R23, R25, R27, R9: value 1k -> 100k
- moved P22 12.5 mm to (208.5, 105.0), turned to 90 degrees
Connections:
- P22 pad 2: /DataST -> DataST
- R10 pad 2: unconnected-(R10-Pad2) -> Net-(R10-Pad2)
- R11 pad 2: unconnected-(R11-Pad2) -> GND
- R12 pad 1: unconnected-(R12-Pad1) -> Net-(R12-Pad1)
- R12 pad 2: unconnected-(R12-Pad2) -> GND
- R13 pad 2: unconnected-(R13-Pad2) -> Net-(R12-Pad1)
- R14 pad 1: unconnected-(R14-Pad1) -> +5V
- R15 pad 1: unconnected-(R15-Pad1) -> Net-(R15-Pad1)
- R15 pad 2: unconnected-(R15-Pad2) -> GND
- R16 pad 2: unconnected-(R16-Pad2) -> Net-(R15-Pad1)
- R17 pad 2: unconnected-(R17-Pad2) -> +5V
- R18 pad 1: unconnected-(R18-Pad1) -> Net-(R18-Pad1)
- R18 pad 2: unconnected-(R18-Pad2) -> GND
- R19 pad 2: unconnected-(R19-Pad2) -> Net-(R18-Pad1)
- R20 pad 1: unconnected-(R20-Pad1) -> Net-(R20-Pad1)
- R20 pad 2: unconnected-(R20-Pad2) -> GND
- R21 pad 2: unconnected-(R21-Pad2) -> Net-(R20-Pad1)
- R22 pad 1: unconnected-(R22-Pad1) -> +5V
- R22 pad 2: unconnected-(R22-Pad2) -> DataST
- R23 pad 1: unconnected-(R23-Pad1) -> Net-(R23-Pad1)
- R23 pad 2: unconnected-(R23-Pad2) -> GND
- R24 pad 2: unconnected-(R24-Pad2) -> Net-(R23-Pad1)
- R25 pad 1: unconnected-(R25-Pad1) -> Net-(R25-Pad1)
- R25 pad 2: unconnected-(R25-Pad2) -> GND
- R26 pad 2: unconnected-(R26-Pad2) -> Net-(R25-Pad1)
- R27 pad 1: unconnected-(R27-Pad1) -> Net-(R27-Pad1)
- R27 pad 2: unconnected-(R27-Pad2) -> GND
- R28 pad 2: unconnected-(R28-Pad2) -> Net-(R27-Pad1)
- R3 pad 2: unconnected-(R3-Pad2) -> Net-(U4-QP3)
- R4 pad 1: unconnected-(R4-Pad1) -> +5V
- R5 pad 2: unconnected-(R5-Pad2) -> Net-(U4-QP2)
- R6 pad 2: unconnected-(R6-Pad2) -> Net-(U4-QP1)
- R7 pad 2: unconnected-(R7-Pad2) -> GND
- R8 pad 2: unconnected-(R8-Pad2) -> Net-(U4-QP0)
- R9 pad 1: unconnected-(R9-Pad1) -> Net-(R10-Pad2)
- R9 pad 2: unconnected-(R9-Pad2) -> GND
Routing:
- net GND: track 0.00 -> 305.3 mm
- net +5V: track 0.00 -> 258.0 mm
- net Net-(U4-QP0): track 0.00 -> 45.0 mm
- net Net-(U4-QP1): track 0.00 -> 44.7 mm
- net Net-(U4-QP2): track 0.00 -> 44.0 mm
- net Net-(U4-QP3): track 0.00 -> 43.6 mm
- net DataST: track 0.00 -> 21.2 mm
- net Net-(R27-Pad1): track 0.00 -> 3.34 mm
- net Net-(R25-Pad1): track 0.00 -> 3.34 mm
- net Net-(R23-Pad1): track 0.00 -> 3.34 mm
- net Net-(R20-Pad1): track 0.00 -> 3.34 mm
- net Net-(R18-Pad1): track 0.00 -> 3.34 mm
- net Net-(R15-Pad1): track 0.00 -> 3.34 mm
- net Net-(R12-Pad1): track 0.00 -> 3.34 mm
- net Net-(R10-Pad2): track 0.00 -> 3.34 mm

Commit message: gl label und q
Parts:
- added Q1: BC327, Package_TO_SOT_THT:TO-92, F.Cu at (200.5, 116.2)
- moved D1 2.75 mm to (123.5, 116.2)
- moved D2 2.25 mm to (123.5, 113.8)
Connections:
- C10 pad 2: unconnected-(C10-Pad2) -> DataST
- C5 pad 2: unconnected-(C5-Pad2) -> EnST
- P22 pad 3: /nTaktST -> nTaktST
- P22 pad 4: /EnST -> EnST
- P22 pad 5: /OutST -> OutST
- R1 pad 2: unconnected-(R1-Pad2) -> OutST
- R14 pad 2: unconnected-(R14-Pad2) -> nTaktST
- U1 pad 11: unconnected-(U1B-K-Pad11) -> Net-(U1A-K)
- U1 pad 3: unconnected-(U1A-Q-Pad3) -> Net-(U1A-Q)
- U1 pad 4: unconnected-(U1A-K-Pad4) -> Net-(U1A-K)
- U1 pad 9: unconnected-(U1B-C-Pad9) -> Net-(U1A-Q)
- U3 pad 1: unconnected-(U3-STR-Pad1) -> Net-(U3-STR)
- U3 pad 2: unconnected-(U3-D-Pad2) -> DataST
- U3 pad 3: unconnected-(U3-CP-Pad3) -> Net-(U3-CP)
- U3 pad 9: unconnected-(U3-QS1-Pad9) -> Net-(U3-QS1)
- U4 pad 1: unconnected-(U4-STR-Pad1) -> Net-(U3-STR)
- U4 pad 2: unconnected-(U4-D-Pad2) -> Net-(U3-QS1)
- U4 pad 3: unconnected-(U4-CP-Pad3) -> Net-(U3-CP)
Routing:
- net OutST: track 0.00 -> 33.9 mm
- net DataST: track 21.2 -> 54.4 mm
- net Net-(U3-QS1): track 0.00 -> 31.7 mm
- net EnST: track 0.00 -> 19.1 mm
- net GND: track 305.3 -> 322.8 mm
- net unconnected-(U2-CP-Pad2): track 0.00 -> 16.9 mm
- net Net-(U1A-Q): track 0.00 -> 16.2 mm
- net nTaktST: track 0.00 -> 15.3 mm
- net Net-(U3-STR): track 0.00 -> 13.7 mm
- net Net-(U3-CP): track 0.00 -> 13.7 mm
- net Net-(U1A-K): track 0.00 -> 7.62 mm
Other:
- board text added: "4520/002001/C"
- board text added: "B - SEITE"

Commit message: diode
Parts:
- added D3: SD103C, Diode_THT:D_DO-35_SOD27_P7.62mm_Horizontal, F.Cu at (184.5, 101.5)
Connections:
- C4 pad 2: unconnected-(C4-Pad2) -> Net-(U1B-~{R})
- C5 pad 1: unconnected-(C5-Pad1) -> Net-(C5-Pad1)
- C9 pad 2: unconnected-(C9-Pad2) -> nTaktST
- D1 pad 1: unconnected-(D1-K-Pad1) -> TZ7
- D2 pad 1: unconnected-(D2-K-Pad1) -> TZ6
- R10 pad 1: unconnected-(R10-Pad1) -> /cTS7
- R11 pad 1: unconnected-(R11-Pad1) -> Net-(C5-Pad1)
- R13 pad 1: unconnected-(R13-Pad1) -> /cTS6
- R16 pad 1: unconnected-(R16-Pad1) -> /cTS5
- R19 pad 1: unconnected-(R19-Pad1) -> /cTS4
- R2 pad 1: unconnected-(R2-Pad1) -> Net-(U1B-J)
- R21 pad 1: unconnected-(R21-Pad1) -> /cTS3
- R24 pad 1: unconnected-(R24-Pad1) -> /cTS2
- R26 pad 1: unconnected-(R26-Pad1) -> /cTS1
- R28 pad 1: unconnected-(R28-Pad1) -> /cTS0
- R29 pad 1: unconnected-(R29-Pad1) -> S3
- R29 pad 2: unconnected-(R29-Pad2) -> Net-(U4-QP7)
- R3 pad 1: unconnected-(R3-Pad1) -> SVA3
- R30 pad 1: unconnected-(R30-Pad1) -> S2
- R30 pad 2: unconnected-(R30-Pad2) -> Net-(U4-QP6)
- R31 pad 1: unconnected-(R31-Pad1) -> S1
- R31 pad 2: unconnected-(R31-Pad2) -> Net-(U4-QP5)
- R32 pad 1: unconnected-(R32-Pad1) -> S0
- R32 pad 2: unconnected-(R32-Pad2) -> Net-(U4-QP4)
- R33 pad 1: unconnected-(R33-Pad1) -> Net-(U1B-~{Q})
- R5 pad 1: unconnected-(R5-Pad1) -> SVA2
- R6 pad 1: unconnected-(R6-Pad1) -> SVA1
- R7 pad 1: unconnected-(R7-Pad1) -> Net-(U1A-K)
- R8 pad 1: unconnected-(R8-Pad1) -> SVA0
- U1 pad 10: unconnected-(U1B-~{R}-Pad10) -> Net-(U1B-~{R})
- U1 pad 12: unconnected-(U1A-C-Pad12) -> Net-(D3-K)
- U1 pad 13: unconnected-(U1A-~{R}-Pad13) -> Net-(U1A-~{R})
- U1 pad 2: unconnected-(U1A-~{Q}-Pad2) -> Net-(U1A-~{Q})
- U1 pad 5: unconnected-(U1B-Q-Pad5) -> Net-(U1B-Q)
- U1 pad 6: unconnected-(U1B-~{Q}-Pad6) -> Net-(U1B-~{Q})
- U1 pad 8: unconnected-(U1B-J-Pad8) -> Net-(U1B-J)
- U2 pad 1: unconnected-(U2-~{PL}-Pad1) -> Net-(U1A-~{Q})
- U2 pad 2: unconnected-(U2-CP-Pad2) -> Net-(U1A-~{R})
- U3 pad 15: unconnected-(U3-OE-Pad15) -> Net-(U1B-Q)
- U3 pad 3: Net-(U3-CP) -> Net-(U1A-~{R})
- U4 pad 11: unconnected-(U4-QP7-Pad11) -> Net-(U4-QP7)
- U4 pad 12: unconnected-(U4-QP6-Pad12) -> Net-(U4-QP6)
- U4 pad 13: unconnected-(U4-QP5-Pad13) -> Net-(U4-QP5)
- U4 pad 14: unconnected-(U4-QP4-Pad14) -> Net-(U4-QP4)
- U4 pad 15: unconnected-(U4-OE-Pad15) -> Net-(U1B-Q)
- U4 pad 3: Net-(U3-CP) -> Net-(U1A-~{R})
Routing:
- net Net-(U1A-~{R}): track 0.00 -> 67.6 mm
- net Net-(U1B-Q): track 0.00 -> 53.3 mm
- net unconnected-(U3-QP1-Pad5): track 0.00 -> 43.1 mm
- net unconnected-(U3-QP0-Pad4): track 0.00 -> 41.5 mm
- net unconnected-(U2-Q7-Pad9): track 0.00 -> 39.9 mm
- net Net-(U4-QP7): track 0.00 -> 37.4 mm
- net Net-(U4-QP6): track 0.00 -> 35.2 mm
- net Net-(U4-QP5): track 0.00 -> 34.0 mm
- net Net-(U4-QP4): track 0.00 -> 34.0 mm
- net Net-(U3-STR): track 13.7 -> 44.5 mm
- net unconnected-(U2-D7-Pad6): track 0.00 -> 29.9 mm
- net Net-(U1B-J): track 0.00 -> 29.1 mm
- net unconnected-(U2-D0-Pad11): track 0.00 -> 28.5 mm
- net unconnected-(U2-D1-Pad12): track 0.00 -> 24.5 mm
- net unconnected-(U2-D3-Pad14): track 0.00 -> 22.1 mm
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
Commit message: kompletti
Parts:
- added H1: MountingHole, MountingHole:MountingHole_3.2mm_M3, F.Cu at (212.8, 72.2)
- added H2: MountingHole, MountingHole:MountingHole_3.2mm_M3, F.Cu at (212.8, 114.0)
- added H3: MountingHole, MountingHole:MountingHole_3.2mm_M3, F.Cu at (104.5, 117.2)
- R1: value 1k -> 47
- R14, R17, R22: value 1k -> 470
Connections:
- C5 pad 1: Net-(C5-Pad1) -> Net-(D3-K)
- C8 pad 2: unconnected-(C8-Pad2) -> EnST
- D1 pad 2: unconnected-(D1-A-Pad2) -> Net-(D1-A)
- D2 pad 2: unconnected-(D2-A-Pad2) -> Net-(D2-A)
- D3 pad 2: unconnected-(D3-A-Pad2) -> GND
- Q1 pad 1: unconnected-(Q1-C-Pad1) -> Net-(Q1-C)
- Q1 pad 2: unconnected-(Q1-B-Pad2) -> Net-(Q1-B)
- Q1 pad 3: unconnected-(Q1-E-Pad3) -> Net-(Q1-E)
- R1 pad 1: unconnected-(R1-Pad1) -> Net-(Q1-C)
- R10 pad 2: Net-(R10-Pad2) -> Net-(U2-D0)
- R11 pad 1: Net-(C5-Pad1) -> Net-(D3-K)
- R12 pad 1: Net-(R12-Pad1) -> Net-(U2-D1)
- R13 pad 2: Net-(R12-Pad1) -> Net-(U2-D1)
- R15 pad 1: Net-(R15-Pad1) -> Net-(U2-D2)
- R16 pad 2: Net-(R15-Pad1) -> Net-(U2-D2)
- R17 pad 1: unconnected-(R17-Pad1) -> EnST
- R18 pad 1: Net-(R18-Pad1) -> Net-(U2-D3)
- R19 pad 2: Net-(R18-Pad1) -> Net-(U2-D3)
- R2 pad 1: Net-(U1B-J) -> Net-(U1A-J)
- R20 pad 1: Net-(R20-Pad1) -> Net-(U2-D4)
- R21 pad 2: Net-(R20-Pad1) -> Net-(U2-D4)
- R23 pad 1: Net-(R23-Pad1) -> Net-(U2-D5)
- R24 pad 2: Net-(R23-Pad1) -> Net-(U2-D5)
- R25 pad 1: Net-(R25-Pad1) -> Net-(U2-D6)
- R26 pad 2: Net-(R25-Pad1) -> Net-(U2-D6)
- R27 pad 1: Net-(R27-Pad1) -> Net-(U2-D7)
- R28 pad 2: Net-(R27-Pad1) -> Net-(U2-D7)
- R33 pad 2: unconnected-(R33-Pad2) -> Net-(Q1-B)
- R4 pad 2: unconnected-(R4-Pad2) -> Net-(U1B-~{R})
- R9 pad 1: Net-(R10-Pad2) -> Net-(U2-D0)
- U1 pad 1: unconnected-(U1A-J-Pad1) -> Net-(U1A-J)
- U1 pad 13: Net-(U1A-~{R}) -> nTaktST
- U1 pad 8: Net-(U1B-J) -> Net-(U1A-J)
- U2 pad 11: unconnected-(U2-D0-Pad11) -> Net-(U2-D0)
- U2 pad 12: unconnected-(U2-D1-Pad12) -> Net-(U2-D1)
- U2 pad 13: unconnected-(U2-D2-Pad13) -> Net-(U2-D2)
- U2 pad 14: unconnected-(U2-D3-Pad14) -> Net-(U2-D3)
- U2 pad 2: Net-(U1A-~{R}) -> nTaktST
- U2 pad 3: unconnected-(U2-D4-Pad3) -> Net-(U2-D4)
- U2 pad 4: unconnected-(U2-D5-Pad4) -> Net-(U2-D5)
- U2 pad 5: unconnected-(U2-D6-Pad5) -> Net-(U2-D6)
- U2 pad 6: unconnected-(U2-D7-Pad6) -> Net-(U2-D7)
- U2 pad 9: unconnected-(U2-Q7-Pad9) -> Net-(Q1-E)
- U3 pad 1: Net-(U3-STR) -> Net-(D3-K)
- U3 pad 3: Net-(U1A-~{R}) -> nTaktST
- U3 pad 4: unconnected-(U3-QP0-Pad4) -> Net-(D1-A)
- U3 pad 5: unconnected-(U3-QP1-Pad5) -> Net-(D2-A)
- U4 pad 1: Net-(U3-STR) -> Net-(D3-K)
- U4 pad 3: Net-(U1A-~{R}) -> nTaktST
Routing:
- net Net-(D1-A): track 0.00 -> 81.6 mm
- net Net-(D2-A): track 0.00 -> 78.3 mm
- net nTaktST: track 34.5 -> 111.8 mm
- net Net-(U1A-~{R}): track 67.6 -> 0.00 mm
- net Net-(D3-K): track 5.16 -> 64.3 mm
- net Net-(U2-D7): track 0.00 -> 54.5 mm
- net Net-(U2-D6): track 0.00 -> 48.8 mm
- net Net-(Q1-E): track 0.00 -> 46.5 mm
- net Net-(U3-STR): track 44.5 -> 0.00 mm
- net Net-(U2-D5): track 0.00 -> 43.5 mm
- net unconnected-(U3-QP1-Pad5): track 43.1 -> 0.00 mm
- net unconnected-(U3-QP0-Pad4): track 41.5 -> 0.00 mm
- net unconnected-(U2-Q7-Pad9): track 39.9 -> 0.00 mm
- net Net-(U2-D4): track 0.00 -> 37.5 mm
- net Net-(U2-D0): track 0.00 -> 36.0 mm
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
Commit message: ercdrc
Connections:
- R2 pad 2: unconnected-(R2-Pad2) -> +5V
Routing:
- net +5V: track 297.5 -> 308.6 mm
- net EnST: track 27.5 -> 32.5 mm
- net Net-(D3-K): track 64.3 -> 66.8 mm
