File: E60/E60.kicad_pcb (KiCad board)
At the start: 2 copper layers, 73.2 x 17.8 mm, 24 parts, among them J1 VDAI, J2 Bally/Bergmann, J3 ADP alt, J4 ESP-01, Q1 Q_NPN_BEC, Q2 Q_NPN_BEC, Q3 Q_NPN_BEC, U1 PC817, U2 PC817, U3 PC817, U4 SPX2920M3-3.3_SOT223, U5 PC817

Commit message: ercdrc
Parts:
- moved REF** 1.78 mm to (127.8, 99.1)
