File: E60/E60.kicad_sch (KiCad schematic)
At the start: 21 parts, among them J1 VDAI, J2 Bally/Bergmann, J3 ADP alt, J4 ESP-01, Q1 Q_NPN_BEC, Q2 Q_NPN_BEC, Q3 Q_NPN_BEC, U1 PC817, U2 PC817, U3 PC817, U4 SPX2920M3-3.3_SOT223, U5 PC817

Commit message: glaube hab irgendeinen scheiss verschoben
Parts:
- removed Q1: Q_NPN_BEC, Package_TO_SOT_SMD:SOT-23, symbol Device:Q_NPN_BEC
- added R6, R8, R9: 3k3, Resistor_SMD:R_0603_1608Metric_Pad0.98x0.95mm_HandSolder, symbol Device:R
- R1: value 3,3k -> 1000
- R3: value 330 -> 1000
- R4: value 10k -> 3k3
Connections:
- net +3.3V: now also R6.2, R8.2, R9.2; no longer J4.4 (Pin_4), R5.1
- net ESP_BUSY: now also R8.1
- net GND: now also U3.2, U5.2
- net TX: now also R5.1
- net at J4.3 (Pin_3), Q3.1 (B): now also R9.1
- new net: J4.4 (Pin_4), R6.1

Commit message: ercdrc
Parts:
- J1: footprint Connector_Dsub:DSUB-9_Male_EdgeMount_P2.77mm -> Connector_Dsub:DSUB-9_Pins_EdgeMount_P2.77mm; symbol Connector:DE9_Plug -> Connector:DE9_Pins
- Q2, Q3: symbol Device:Q_NPN_BEC -> Transistor_BJT:Q_NPN_BEC
Other:
- moved on the sheet: C1, C2, U4
