File: EBA410/EBA410.kicad_sch (KiCad schematic)
At the start: 3 parts, among them P1 rt, P2 auf L-SEITE

Commit message: ercdrc
Connections:
- no-connect marks 0 -> 21
Changed lines of the file:
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@@
 		(color 0 0 0 0)
+	)
+	(junction
+		(at 73.66 101.6)
+		(diameter 0)
+		(color 0 0 0 0)
+	)
+	(junction
+		(at 68.58 101.6)
+		(diameter 0)
+		(color 0 0 0 0)
+	)
+	(no_connect
+		(at 78.74 76.2)
+	)
+	(no_connect
+		(at 76.2 76.2)
+	)
+	(no_connect
+		(at 66.04 63.5)
+	)
+	(no_connect
+		(at 86.36 63.5)
+	)
+	(no_connect
+		(at 101.6 76.2)
+	)
+	(no_connect
+		(at 71.12 76.2)
+	)
+	(no_connect
+		(at 83.82 76.2)
+	)
+	(no_connect
+		(at 78.74 63.5)
+	)
+	(no_connect
+		(at 66.04 76.2)
+	)
+	(no_connect
+		(at 88.9 63.5)
+	)
+	(no_connect
+		(at 99.06 76.2)
+	)
+	(no_connect
+		(at 86.36 76.2)
+	)
+	(no_connect
+		(at 68.58 63.5)
+	)
+	(no_connect
+		(at 76.2 63.5)
+	)
+	(no_connect
+		(at 88.9 76.2)
+	)
+	(no_connect
+		(at 71.12 63.5)
+	)
+	(no_connect
+		(at 73.66 76.2)
+	)
+	(no_connect
+		(at 73.66 63.5)
+	)
+	(no_connect
+		(at 68.58 76.2)
+	)
+	(no_connect
+		(at 83.82 63.5)
+	)
+	(no_connect
+		(at 91.44 63.5)
 	)
 	(wire
@@
 		)
 		(instances
-			(project ""
+			(project "EBA410"
 				(path "/77f91d4d-a9c8-4f55-a847-0cd52f8aa927"
 					(reference "P2")
@@
 		)
 		(instances
-			(project ""
+			(project "EBA410"
 				(path "/77f91d4d-a9c8-4f55-a847-0cd52f8aa927"
 					(reference "H1")
+					(unit 1)
+				)
+			)
+		)
+	)
+	(symbol
+		(lib_id "power:PWR_FLAG")
+		(at 68.58 101.6 90)
+		(unit 1)
+		(exclude_from_sim no)
+		(in_bom yes)
+		(on_board yes)
+		(dnp no)
+		(fields_autoplaced yes)
+		(property "Reference" "#FLG01"
+			(at 66.675 101.6 0)
+			(effects
+				(font
+					(size 1.27 1.27)
+				)
+				(hide yes)
+			)
+		)
+		(property "Value" "PWR_FLAG"
+			(at 64.77 101.5999 90)
+			(effects
+				(font
+					(size 1.27 1.27)
+				)
+				(justify left)
+			)
+		)
+		(property "Footprint" ""
+			(at 68.58 101.6 0)
+			(effects
+				(font
+					(size 1.27 1.27)
+				)
+				(hide yes)
+			)
+		)
+		(property "Datasheet" "~"
+			(at 68.58 101.6 0)
+			(effects
+				(font
+					(size 1.27 1.27)
+				)
+				(hide yes)
+			)
+		)
+		(property "Description" "Special symbol for telling ERC where power comes from"
+			(at 68.58 101.6 0)
+			(effects
+				(font
+					(size 1.27 1.27)
+				)
+				(hide yes)
+			)
+		)
+		(pin "1"
+		)
+		(instances
+			(project "EBA410"
+				(path "/77f91d4d-a9c8-4f55-a847-0cd52f8aa927"
+					(reference "#FLG01")
 					(unit 1)
 				)
@@
 		)
 		(instances
-			(project ""
+			(project "EBA410"
 				(path "/77f91d4d-a9c8-4f55-a847-0cd52f8aa927"
 					(reference "#PWR01")
@@
 		)
 		(instances
-			(project ""
+			(project "EBA410"
 				(path "/77f91d4d-a9c8-4f55-a847-0cd52f8aa927"
 					(reference "P1")
@@
 		)
 		(instances
-			(project ""
+			(project "EBA410"
 				(path "/77f91d4d-a9c8-4f55-a847-0cd52f8aa927"
 					(reference "#PWR02")
 					(unit 1)
 				)
+			)
+		)
+	)
+	(symbol
+		(lib_id "power:PWR_FLAG")
+		(at 73.66 101.6 270)
+		(unit 1)
+		(exclude_from_sim no)
+		(in_bom yes)
+		(on_board yes)
+		(dnp no)
+		(fields_autoplaced yes)
+		(property "Reference" "#FLG02"
+			(at 75.565 101.6 0)
+			(effects
+				(font
+					(size 1.27 1.27)
+				)
+				(hide yes)
+			)
+		)
+		(property "Value" "PWR_FLAG"
+			(at 77.47 101.5999 90)
+			(effects
+				(font
+					(size 1.27 1.27)
+				)
+				(justify left)
+			)
+		)
+		(property "Footprint" ""
+			(at 73.66 101.6 0)
+			(effects
+				(font
+					(size 1.27 1.27)
+				)
+				(hide yes)
+			)
+		)
+		(property "Datasheet" "~"
+			(at 73.66 101.6 0)
+			(effects
+				(font
+					(size 1.27 1.27)
+				)
+				(hide yes)
+			)
+		)
+		(property "Description" "Special symbol for telling ERC where power comes from"
+			(at 73.66 101.6 0)
+			(effects
+				(font
+					(size 1.27 1.27)
+				)
+				(hide yes)
+			)
+		)
+		(pin "1"
+		)
+		(instances
+			(project "EBA410"
+				(path "/77f91d4d-a9c8-4f55-a847-0cd52f8aa927"
+					(reference "#FLG02")
+					(unit 1)
+				)
