File: ZLKalt/ZLKalt.kicad_pcb (KiCad board)
At the start: 2 copper layers, 88.8 x 45.5 mm, 30 parts, among them J1 Conn_02x04_Counter_Clockwise, J2 Conn_02x04_Counter_Clockwise, U1 AT90S1200A

Commit message: silkscreen, parts
Parts:
- C1, C2, C3: value C -> 100nF
- D1: value D -> 0,5W 4,7V
- D2: value ~ -> ESDA6V1U1
- R1: value R -> 270; footprint Resistor_SMD:R_0805_2012Metric_Pad1.20x1.40mm_HandSolder -> Resistor_SMD:R_0603_1608Metric
- R2, R6: value 4640 -> 4700; footprint Resistor_SMD:R_0603_1608Metric_Pad0.98x0.95mm_HandSolder -> Resistor_SMD:R_0603_1608Metric
- R3: value R -> 4700; footprint Resistor_SMD:R_0603_1608Metric_Pad0.98x0.95mm_HandSolder -> Resistor_SMD:R_0603_1608Metric
- R5, R7: footprint Resistor_SMD:R_0805_2012Metric_Pad1.20x1.40mm_HandSolder -> Resistor_SMD:R_0603_1608Metric
- TP10: renamed from MISO; footprint TestPoint:TestPoint_Pad_D1.0mm -> TestPoint:TestPoint_Pad_D1.5mm
- renumbered SCK to TP12, RESET to TP13, XTAL1 to TP14, XTAL2 to TP15, MOSI to TP4, SCK to TP6

Commit message: aussparung
Changed lines of the file:
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@@
 	)
 	(gr_text "Oben"
-		(at 101.092 39.497 -0)
+		(at 100.584 39.497 0)
 		(layer "B.Cu")
 		(effects
 			(font
-				(size 5 4.2)
+				(size 5 4)
 				(thickness 0.3)
 				(bold yes)
@@
 	)
 	(zone
+		(net 0)
+		(net_name "")
+		(layer "B.Cu")
+		(hatch edge 0.5)
+		(connect_pads
+			(clearance 0)
+		)
+		(min_thickness 0.25)
+		(filled_areas_thickness no)
+		(keepout
+			(tracks allowed)
+			(vias allowed)
+			(pads allowed)
+			(copperpour not_allowed)
+			(footprints allowed)
+		)
+		(placement
+			(enabled no)
+			(sheetname "/")
+		)
+		(fill
+			(thermal_gap 0.5)
+			(thermal_bridge_width 0.5)
+		)
+		(polygon
+			(pts
+				(xy 84.328 40.64) (xy 101.854 40.64) (xy 101.854 31.496) (xy 84.328 31.496)
+			)
+		)
+	)
+	(zone

Commit message: net namen
Parts:
- R5: value 4640 -> 4700
Connections:
- net Net-(U1-PB5) renamed /ISP_MOSI
- net Net-(U1-PB6) renamed /ISP_MISO
- net Net-(U1-PB7) renamed /ISP_SCK
- net Net-(U1-~{RESET}) renamed /ISP_RESET
Changed lines of the file:
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@@
 			(psa4output no)
 			(plot_black_and_white yes)
-			(plotinvisibletext no)
 			(sketchpadsonfab no)
 			(plotpadnumbers no)
@@
 	(net 13 "Net-(U1-XTAL1)")
 	(net 14 "Net-(U1-XTAL2)")
-	(net 15 "Net-(U1-~{RESET})")
-	(net 16 "Net-(U1-PB6)")
-	(net 17 "Net-(U1-PB7)")
-	(net 18 "Net-(U1-PB5)")
+	(net 15 "/ISP_RESET")
+	(net 16 "/ISP_MISO")
+	(net 17 "/ISP_MOSI")
+	(net 18 "/ISP_SCK")
 	(footprint "Diode_SMD:D_1206_3216Metric"
 		(layer "F.Cu")
@@
 			)
 		)
-		(property "Datasheet" ""
+		(property "Datasheet" "~"
 			(at 0 0 0)
 			(unlocked yes)
@@
 			)
 		)
-		(property "Datasheet" ""
+		(property "Datasheet" "~"
 			(at 0 0 0)
 			(unlocked yes)
@@
 			)
 		)
-		(property "Datasheet" ""
+		(property "Datasheet" "~"
 			(at 0 0 0)
 			(unlocked yes)
@@
 			)
 		)
-		(property "Datasheet" ""
+		(property "Datasheet" "~"
 			(at 0 0 0)
 			(unlocked yes)
@@
 			(layers "F.Cu" "F.Mask" "F.Paste")
 			(roundrect_rratio 0.25)
-			(net 16 "Net-(U1-PB6)")
+			(net 16 "/ISP_MISO")
 			(pintype "passive")
 		)
@@
 			)
 		)
-		(property "Datasheet" ""
+		(property "Datasheet" "~"
 			(at 0 0 180)
 			(unlocked yes)
@@
 			(layers "F.Cu" "F.Mask" "F.Paste")
 			(roundrect_rratio 0.212766)
-			(net 15 "Net-(U1-~{RESET})")
+			(net 15 "/ISP_RESET")
 			(pintype "passive")
 		)
@@
 			)
 		)
-		(property "Datasheet" ""
+		(property "Datasheet" "~"
 			(at 0 0 0)
 			(unlocked yes)
@@
 			(size 1.5 1.5)
 			(layers "F.Cu" "F.Mask")
-			(net 16 "Net-(U1-PB6)")
+			(net 16 "/ISP_MISO")
 			(pinfunction "1")
 			(pintype "passive")
@@
 			)
 		)
-		(property "Datasheet" ""
+		(property "Datasheet" "~"
 			(at 0 0 0)
 			(unlocked yes)
@@
 			)
 		)
-		(property "Datasheet" ""
+		(property "Datasheet" "~"
 			(at 0 0 0)
 			(unlocked yes)
@@
 			)
 		)
-		(property "Datasheet" ""
+		(property "Datasheet" "~"
 			(at 0 0 0)
 			(unlocked yes)
@@
 			)
 		)
-		(property "Datasheet" ""
+		(property "Datasheet" "~"
 			(at 0 0 0)
 			(unlocked yes)
@@
 			(size 1.5 1.5)
 			(layers "F.Cu" "F.Mask")
-			(net 17 "Net-(U1-PB7)")
+			(net 18 "/ISP_SCK")
 			(pinfunction "1")
 			(pintype "passive")
@@
 			(layers "F.Cu" "F.Mask" "F.Paste")
 			(roundrect_rratio 0.25)
-			(net 15 "Net-(U1-~{RESET})")
+			(net 15 "/ISP_RESET")
 			(pinfunction "~{RESET}")
 			(pintype "input")
@@
 			(layers "F.Cu" "F.Mask" "F.Paste")
 			(roundrect_rratio 0.25)
-			(net 18 "Net-(U1-PB5)")
+			(net 17 "/ISP_MOSI")
 			(pinfunction "PB5")
 			(pintype "bidirectional")
@@
 			(layers "F.Cu" "F.Mask" "F.Paste")
 			(roundrect_rratio 0.25)
-			(net 16 "Net-(U1-PB6)")
+			(net 16 "/ISP_MISO")
 			(pinfunction "PB6")
 			(pintype "bidirectional")
@@
 			(layers "F.Cu" "F.Mask" "F.Paste")
 			(roundrect_rratio 0.25)
-			(net 17 "Net-(U1-PB7)")
+			(net 18 "/ISP_SCK")
 			(pinfunction "PB7")
 			(pintype "bidirectional")
@@
 			)
 		)
-		(property "Datasheet" ""
+		(property "Datasheet" "~"
 			(at 0 0 0)
 			(unlocked yes)
@@
 			(layers "F.Cu" "F.Mask" "F.Paste")
 			(roundrect_rratio 0.25)
-			(net 17 "Net-(U1-PB7)")
+			(net 18 "/ISP_SCK")
 			(pintype "passive")
 		)
@@
 			)
 		)
-		(property "Datasheet" ""
+		(property "Datasheet" "~"
 			(at 0 0 0)
 			(unlocked yes)
@@
 			)
 		)
-		(property "Datasheet" ""
+		(property "Datasheet" "~"
 			(at 0 0 0)
 			(unlocked yes)
@@
 			)
 		)
-		(property "Datasheet" ""
+		(property "Datasheet" "~"
 			(at 0 0 0)
 			(unlocked yes)
@@
 			)
 		)
-		(property "Datasheet" ""
+		(property "Datasheet" "~"
 			(at 0 0 90)
 			(unlocked yes)
@@
 			(layers "F.Cu" "F.Mask" "F.Paste")
 			(roundrect_rratio 0.25)
-			(net 18 "Net-(U1-PB5)")
+			(net 17 "/ISP_MOSI")
 			(pintype "passive")
 		)
@@
 			)
 		)
-		(property "Datasheet" ""
+		(property "Datasheet" "~"
 			(at 0 0 0)
 			(unlocked yes)
@@
 			)
 		)
-		(property "Datasheet" ""
+		(property "Datasheet" "~"
 			(at 0 0 0)
 			(unlocked yes)
@@
 			)
 		)
-		(property "Datasheet" ""
+		(property "Datasheet" "~"
 			(at 0 0 0)
 			(unlocked yes)
@@
 			(size 1.5 1.5)
 			(layers "F.Cu" "F.Mask")
-			(net 15 "Net-(U1-~{RESET})")
+			(net 15 "/ISP_RESET")
 			(pinfunction "1")
 			(pintype "passive")
@@
 			)
 		)
-		(property "Datasheet" ""
+		(property "Datasheet" "~"
 			(at 0 0 0)
 			(unlocked yes)
@@
 			)
 		)
-		(property "Datasheet" ""
+		(property "Datasheet" "~"
 			(at 0 0 0)
 			(unlocked yes)
@@
 			)
 		)
-		(property "Datasheet" ""
+		(property "Datasheet" "~"
 			(at 0 0 270)
 			(unlocked yes)
@@
 			(layers "F.Cu" "F.Mask" "F.Paste")
 			(roundrect_rratio 0.25)
-			(net 18 "Net-(U1-PB5)")
+			(net 17 "/ISP_MOSI")
 			(pintype "passive")
 		)
@@
 			)
 		)
-		(property "Datasheet" ""
+		(property "Datasheet" "~"
 			(at 0 0 180)
 			(unlocked yes)
@@
 			)
 		)
-		(property "Value" "4640"
+		(property "Value" "4700"
 			(at 0 1.43 180)
 			(layer "F.Fab")
@@
 			)
 		)
-		(property "Datasheet" ""
+		(property "Datasheet" "~"
 			(at 0 0 180)
 			(unlocked yes)
@@
 			(layers "F.Cu" "F.Mask" "F.Paste")
 			(roundrect_rratio 0.25)
-			(net 15 "Net-(U1-~{RESET})")
+			(net 15 "/ISP_RESET")
 			(pintype "passive")
 		)
@@
 			)
 		)
-		(property "Datasheet" ""
+		(property "Datasheet" "~"
 			(at 0 0 0)
 			(unlocked yes)
@@
 			)
 		)
-		(property "Datasheet" ""
+		(property "Datasheet" "~"
 			(at 0 0 0)
 			(unlocked yes)
@@
 			)
 		)
-		(property "Datasheet" ""
+		(property "Datasheet" "~"
 			(at 0 0 0)
 			(unlocked yes)
@@
 			)
 		)
-		(property "Datasheet" ""
+		(property "Datasheet" "~"
 			(at 0 0 0)
 			(unlocked yes)
@@
 			(size 1.5 1.5)
 			(layers "F.Cu" "F.Mask")
-			(net 18 "Net-(U1-PB5)")
+			(net 17 "/ISP_MOSI")
 			(pinfunction "1")
 			(pintype "passive")
@@
 			)
 		)
-		(property "Datasheet" ""
+		(property "Datasheet" "~"
 			(at 0 0 0)
 			(unlocked yes)
@@
 	)
 	(segment
-		(start 117.094 67.564)
-		(end 117.602 67.564)
+		(start 116.84 58.642)
+		(end 116.84 60.405)
 		(width 0.2)
 		(layer "F.Cu")
@@
 	)
 	(segment
-		(start 117.602 67.564)
-		(end 118.745 66.421)
+		(start 118.491 63.881)
+		(end 118.11 63.5)
 		(width 0.2)
 		(layer "F.Cu")
@@
 	)
 	(segment
-		(start 117.094 67.564)
-		(end 117.094 68.58)
+		(start 124.968 67.564)
+		(end 124.968 68.834)
 		(width 0.2)
 		(layer "F.Cu")
@@
 	)
 	(segment
-		(start 117.094 68.58)
-		(end 118.11 69.596)
+		(start 121.285 63.881)
+		(end 124.968 67.564)
 		(width 0.2)
 		(layer "F.Cu")
@@
 	)
 	(segment
-		(start 118.745 66.421)
-		(end 119.86 66.421)
+		(start 118.11 63.5)
+		(end 118.11 61.214)
 		(width 0.2)
 		(layer "F.Cu")
@@
 	)
 	(segment
-		(start 116.84 58.642)
-		(end 116.84 60.405)
+		(start 119.86 63.881)
+		(end 121.285 63.881)
 		(width 0.2)
 		(layer "F.Cu")
-		(net 18)
+		(net 17)
 	)
 	(segment
-		(start 118.491 63.881)
-		(end 118.11 63.5)
+		(start 119.86 63.881)
+		(end 118.491 63.881)
 		(width 0.2)
 		(layer "F.Cu")
-		(net 18)
+		(net 17)
 	)
 	(segment
-		(start 124.968 67.564)
-		(end 124.968 68.834)
+		(start 117.301 60.405)
+		(end 116.84 60.405)
 		(width 0.2)
 		(layer "F.Cu")
-		(net 18)
+		(net 17)
 	)
 	(segment
-		(start 121.285 63.881)
-		(end 124.968 67.564)
+		(start 118.11 61.214)
+		(end 117.301 60.405)
 		(width 0.2)
 		(layer "F.Cu")
-		(net 18)
+		(net 17)
 	)
 	(segment
-		(start 118.11 63.5)
-		(end 118.11 61.214)
+		(start 117.094 67.564)
+		(end 117.602 67.564)
 		(width 0.2)
 		(layer "F.Cu")
@@
 	)
 	(segment
-		(start 119.86 63.881)
-		(end 121.285 63.881)
+		(start 117.602 67.564)
+		(end 118.745 66.421)
 		(width 0.2)
 		(layer "F.Cu")
@@
 	)
 	(segment
-		(start 119.86 63.881)
-		(end 118.491 63.881)
+		(start 117.094 67.564)
+		(end 117.094 68.58)
 		(width 0.2)
 		(layer "F.Cu")
@@
 	)
 	(segment
-		(start 117.301 60.405)
-		(end 116.84 60.405)
+		(start 117.094 68.58)
+		(end 118.11 69.596)
 		(width 0.2)
 		(layer "F.Cu")
@@
 	)
 	(segment
-		(start 118.11 61.214)
-		(end 117.301 60.405)
+		(start 118.745 66.421)
+		(end 119.86 66.421)
 		(width 0.2)
 		(layer "F.Cu")

Commit message: zlk drc
Parts:
- added TP17: TestPoint, TestPoint:TestPoint_THTPad_D2.0mm_Drill1.0mm, F.Cu at (58.4, 37.1)
- added TP18: TestPoint, TestPoint:TestPoint_THTPad_D2.0mm_Drill1.0mm, F.Cu at (134.6, 38.4)
- added TP19: TestPoint, TestPoint:TestPoint_THTPad_D2.0mm_Drill1.0mm, F.Cu at (135.9, 72.9)
- moved TP16 0.28 mm to (114.8, 52.2)
- moved D1 0.25 mm to (123.3, 54.1)
- moved C1 0.13 mm to (128.2, 54.2)
- moved C2 0.13 mm to (117.4, 54.2)
- moved R5 0.13 mm to (111.8, 64.9)
Routing:
- net MISO: track 56.4 -> 54.8 mm
- net GND: track 179.7 -> 178.4 mm, vias 57 -> 54
- net SCK: track 65.2 -> 64.1 mm
- net MOSI: track 63.2 -> 62.3 mm
- net VCC: track 47.3 -> 47.9 mm
- net RST: track 64.4 -> 63.9 mm
