File: cpumodul85/cpumodul85.kicad_pcb (KiCad board)
At the start: 2 copper layers, 106 x 80 mm, 22 parts, among them P1 DIN41612_03x16_ABC, U1 74HC14, U2 EP1810, U3 8085AH-2, U4 48Z08, U5 48T08, U6 27512

Commit message: erc+drc
Connections:
- net Cb3 renamed EXT_AD7
- net Cb4 renamed EXT_AD5
- net Cb5 renamed EXT_AD3
- net Cb6 renamed EXT_AD1
- net Cc3 renamed EXT_AD6
- net Cc4 renamed EXT_AD4
- net Cc5 renamed EXT_AD2
- net Cc6 renamed EXT_AD0
- P1 pad a7: Ca7 -> unconnected-(P1A-Pin_a7-Pada7)
- U3 pad 38: HLDA -> unconnected-(U3-HLDA-Pad38)
- U3 pad 4: SOD -> unconnected-(U3-SOD-Pad4)
Other:
- board text added: "GITH"
- board text removed: "GITH :"
