File: cpumodul85/cpumodul85.kicad_sch (KiCad schematic)
At the start: 20 parts, among them P1 DIN41612_03x16_ABC, U1 74HC14, U2 EP1810, U3 8085AH-2, U4 48Z08, U5 48T08, U6 27512

Commit message: match
Parts:
- added C4, C5: VC100NF, Capacitor_THT:C_Axial_L3.8mm_D2.6mm_P7.50mm_Horizontal, symbol Device:C
Connections:
- net A14: no longer R5.1, U2.50 (INP11), U4.1 (A14), U5.1 (A14)
- net A6: now also U2.60 (I/O_40D)
- net AD6: now also U2.62 (I/O_42D); no longer U2.56 (INP16)
- net ALE: now also P1.b7 (Pin_b7)
- net GND: now also C4.2, C5.2
- net INTA: now also P1.c7 (Pin_c7)
- net INTR: now also P1.c8 (Pin_c8)
- net IO/M: now also P1.a11 (Pin_a11)
- net RES_OUT: now also P1.c13 (Pin_c13), U2.54 (INP14)
- net S1: now also U2.56 (INP16)
- net SID: now also P1.b13 (Pin_b13)
- net VCC: now also C4.1, C5.1
- net RST65: now reaches P1.c10 (Pin_c10)
- net RST65: now also U3.8 (RST6_5)
- net RST75: now reaches P1.c11 (Pin_c11)
- net RST75: now also U3.7 (RST7_5)
- net Cc3: now reaches P1.c3 (Pin_c3)
- net Cc3: now also U2.61 (I/O_41D)
- net Cc4: now reaches P1.c4 (Pin_c4)
- net Cc4: now also U2.67 (I/O_47D)
- net Cc5: now reaches P1.c5 (Pin_c5)
- net Cc5: now also U2.6 (I/O_5A)
- net Cc6: now reaches P1.c6 (Pin_c6)
- net Cc6: now also U2.12 (I/O_11A)
- net RST55: now reaches P1.c9 (Pin_c9)
- net RST55: now also U3.9 (RST5_5)
- net at U1.8: now also U1.1
- net Ca13: now reaches U1.13
- net Ca13: now also P1.a13 (Pin_a13)
- net Cb5: now reaches U2.3 (I/O_2A)
- net Cb5: now also P1.b5 (Pin_b5)
- net Ca4: now reaches U2.36 (I/O_25C)
- net Ca4: now also P1.a4 (Pin_a4)
- net Ca5: now reaches U2.37 (I/O_26C)
- net Ca5: now also P1.a5 (Pin_a5)
- net Ca6: now reaches U2.38 (I/O_27C)
- net Ca6: now also P1.a6 (Pin_a6)
- net Ca9: now reaches U2.42 (I/O_31C)
- net Ca9: now also P1.a9 (Pin_a9)
- net Ca8: now reaches U2.43 (I/O_32C)
- net Ca8: now also P1.a8 (Pin_a8)
- net Ca3: now reaches U2.44 (I/O_33C)
- net Ca3: now also P1.a3 (Pin_a3)
- net A14Z: now reaches U2.51 (CLK3/INP12)
- net A14Z: now also R4.1, U4.1 (A14)
- net Cb3: now reaches U2.58 (I/O_38D)
- net Cb3: now also P1.b3 (Pin_b3)
- net Cb4: now reaches U2.64 (I/O_44D)
- net Cb4: now also P1.b4 (Pin_b4)
- net Cb6: now reaches U2.9 (I/O_8A)
- net Cb6: now also P1.b6 (Pin_b6)
- net Ca7: now reaches P1.a7 (Pin_a7)
- net TRAP: now reaches R2.1
- net TRAP: now also U3.6 (TRAP)
- new net A14T: R5.1, U2.50 (INP11), U5.1 (A14)
- no-connect marks 8 -> 13
Other:
- moved on the sheet: P1A, P1B

Commit message: erc+drc
Connections:
- net Ca7: no longer names the net of P1.a7 (Pin_a7)
- net Cb3 renamed EXT_AD7
- net Cb4 renamed EXT_AD5
- net Cb5 renamed EXT_AD3
- net Cb6 renamed EXT_AD1
- net Cc3 renamed EXT_AD6
- net Cc4 renamed EXT_AD4
- net Cc5 renamed EXT_AD2
- net Cc6 renamed EXT_AD0
- net HLDA: no longer names the net of U3.38 (HLDA)
- net SOD: no longer names the net of U3.4 (SOD)
- no-connect marks 13 -> 16
Other:
- moved on the sheet: C1, C2, C3, C4, C5, C6, C7, P1A, P1B, P1C, R1, R2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
