File: Druckeranschluss/Druckeranschluss.kicad_pcb (KiCad board)
At the start: 2 copper layers, 49.5 x 49.5 mm, 11 parts, among them J1 Conn_01x08, J2 DE9_Socket, J3 Conn_01x05, Q1 BC327, Q2 BC337

Commit message: ende drucker und jamma unten
Connections:
- net GND renamed 24VST
- net Net-(J1-Pin_4) renamed +NT5V
- net Net-(J1-Pin_5) renamed 5VGND
- net Net-(J3-Pin_3) renamed /INTX
- net Net-(J3-Pin_4) renamed /INRX
- net Net-(Q1-C) renamed /RX_A
- net Net-(Q2-B) renamed /TX_A
- net RX renamed /RX
- net TX renamed /TX
- J1 pad 1: unconnected-(J1-Pin_1-Pad1) -> +48V
- J1 pad 3: unconnected-(J1-Pin_3-Pad3) -> +12V
- J1 pad 6: unconnected-(J1-Pin_6-Pad6) -> 12VGND
Other:
- board text added: "~sD"
- board text removed: "ADP"
