File: Druckeranschluss/Druckeranschluss.kicad_sch (KiCad schematic)
At the start: 11 parts, among them J1 Conn_01x08, J2 DE9_Socket, J3 Conn_01x05, Q1 BC327, Q2 BC337

Commit message: ende drucker und jamma unten
Connections:
- net 5VGND: now reaches J1.5 (Pin_5), J3.2 (Pin_2), Q2.3 (E), R2.2, R6.1
- net TX_A: now reaches Q2.2 (B), R5.2, R6.2
- net +NT5V: now reaches J1.4 (Pin_4), J3.5 (Pin_5), Q1.3 (E), R1.2
- net INTX: now reaches J3.3 (Pin_3), R4.2
- net INRX: now reaches J3.4 (Pin_4), Q2.1 (C)
- net RX_A: now reaches Q1.1 (C), R2.1, R3.1
- net +48V: now reaches J1.1 (Pin_1)
- net +12V: now reaches J1.3 (Pin_3)
- net 12VGND: now reaches J1.6 (Pin_6)
- net GND renamed 24VST
- no-connect marks 10 -> 7
