File: JAMMA/JAMMA.kicad_sch (KiCad schematic)
At the start: 140 parts, among them P1 Conn_02x30_Counter_Clockwise, P2 Conn_01x05, P3 Conn_01x06, P4 Conn_01x06, P5 Conn_01x08, P6 Conn_01x08, U1 TDA2003, U2 74HC165, U3 74HC165, U4 74HC245, U5 74HC107

Commit message: ende drucker und jamma unten
Connections:
- net GND: now also R61.2
- net INPUTS_COMMON: now reaches R45.2
- net INPUTS_COMMON: now also D1.2 (A), P1.5 (Pin_5), P1.56 (Pin_56), R11.2, R14.2, R17.2, R2.2, R20.2, R23.2, R27.2, R30.2, R33.2, R36.2, R39.2, R42.2, R5.2, R8.2
- net at C22.2, R34.2, R35.2: now also U3.4 (D5)
- net at C28.2, U1.2 (-): now also R51.2
- net at U1.3 (GND): now also C18.2
- net at U1.4: now also C19.2, R50.2
- net at R66.2: now also U5.11 (K)
- net at C21.2, R31.2, R32.2: now also U3.5 (D6)
- net VD: now reaches P2.3 (Pin_3)
- net VD: now also C38.1, C45.1, P3.6 (Pin_6)
- net at C15.2: now also R26.2
- net at R71.1: now also U4.1 (A->B)
- net at R70.1: now also U4.2 (A0)
- net at R58.2: now also U4.3 (A1), U4.5 (A3), U4.6 (A4), U4.7 (A5), U4.8 (A6)
- net VIDEO0: now reaches C37.2, R56.2
- net VIDEO0: now also P4.2 (Pin_2)
- net FVIDEO3: now reaches C2.2, L1.1
- net FVIDEO3: now also P1.39 (Pin_39)
- net at C27.2: now also R48.2, R49.2
- net at C43.1: now also D1.1 (K), P1.9 (Pin_9)
- net at R62.2: now also U3.9 (Q7)
- net FVIDEO0: now reaches C4.2, L4.1
- net FVIDEO0: now also P1.36 (Pin_36)
- net at C28.1: now also R50.1, R52.2
- net at C40.2: now also U5.9 (C)
- net at C20.2, R28.2, R29.2: now also U3.6 (D7)
- net VIDEO1: now reaches P4.4 (Pin_4)
- net VIDEO1: now also C36.2, R55.2
- net VIDEO2: now reaches P4.5 (Pin_5)
- net VIDEO2: now also C35.2, R54.2
- net VIDEO3: now reaches P4.6 (Pin_6)
- net VIDEO3: now also C34.2, R53.2
- net at C38.2: now also R74.1
- net LOAD: now reaches U3.1 (~{PL})
- net LOAD: now also U2.1 (~{PL})
- net CLOCK: now reaches U3.2 (CP)
- net CLOCK: now also C30.1, U2.2 (CP)
- net FVIDEO2: now reaches C3.2, L2.1
- net FVIDEO2: now also P1.38 (Pin_38)
- net at R72.1: now also U4.4 (A2)
- net at P3.3 (Pin_3): now also R73.2, R74.2
- net at L5.1: now also C6.1, P1.57 (Pin_57), P1.58 (Pin_58)
- net at L5.2: now also C29.1
- net at C1.2: now also R26.1
- net at U4.16 (B2): now also R68.2
- net at U4.19 (CE): now also R69.2
- net at R73.1: now also C17.2, C18.1
- net FVIDEO1: now reaches P1.37 (Pin_37)
- net FVIDEO1: now also C5.2, L3.1
- net at C19.1: now also R51.1
- net at R67.2: now also U5.13 (~{R})
- net at U5.1 (J): now also R63.1
- net at C44.2: now also P6.5 (Pin_5)
- no-connect marks 0 -> 3
Other:
- moved on the sheet: C1, C15, C16, C17, C18, C19, C2, C20, C21, C22, C23, C24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
