File: Systemmodul25.2/Systemmodul25.2.kicad_pcb (KiCad board)
At the start: 2 copper layers, 61 x 116.8 mm, 32 parts, among them J1 DIN41612_02x16_AB, J2 DIN41612_02x16_AB, J3 AVR-ISP-6, Q1 12.00J1, U1 W27E040, U2 W27E040, U3 M48T18-100PC1, U4 ATmega8515-16A, U5 MAX690xPA

Commit message: systemmodul reset
Parts:
- added FID3: Fiducial, Fiducial:Fiducial_0.75mm_Mask1.5mm, F.Cu at (138.4, 54.6)
- D1: value D -> BAT85
- FID1, FID2: footprint Fiducial:Fiducial_Cross_0.5mm_Mask2mm -> Fiducial:Fiducial_Cross_1.5mm_Mask2mm
- JP1: value Jumper_2_Bridged -> Sound_4MBit
- JP2: value Jumper_2_Open -> Sound_2MBit
- JP3: value Jumper_2_Open -> Program_2MBit
- JP4: value Jumper_2_Bridged -> Program_4MBit
Connections:
- net NVRAM_E2 renamed /NVRAM_E2
- J3 pad 5: Net-(J3-~{RST}) -> RESET
- R4 pad 2: Net-(U5-~{RESET}) -> RESET
- U4 pad 4: Net-(J3-~{RST}) -> RESET
- U5 pad 4: unconnected-(U5-PFI-Pad4) -> GND
- U5 pad 7: Net-(U5-~{RESET}) -> RESET
Routing:
- net RESET: track 0.00 -> 52.2 mm, vias 0 -> 1
- net Net-(U5-~{RESET}): track 41.8 -> 0.00 mm, vias 1 -> 0
- net Net-(J3-~{RST}): track 9.12 -> 0.00 mm

Commit message: move board
Parts:
- moved C2 72.3 mm to (21.0, 67.3)
- moved C3 72.3 mm to (21.0, 108.0)
- moved C4 72.3 mm to (21.0, 62.2)
- moved C5 72.3 mm to (21.0, 102.9)
- moved C8 72.3 mm to (24.8, 29.2)
- moved C9 72.3 mm to (24.8, 33.0)
- moved D1 72.3 mm to (68.2, 92.7)
- moved FID1 72.3 mm to (70.5, 26.7)
- moved FID3 72.3 mm to (70.5, 29.8)
- moved JP1 72.3 mm to (71.2, 108.0)
- moved LED2 72.3 mm to (60.3, 31.8)
- moved R2 72.3 mm to (21.0, 90.2)
- moved U1 72.3 mm to (64.4, 97.8)
- moved U2 72.3 mm to (64.8, 57.1)
- moved U3 72.3 mm to (59.7, 77.5)
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
Commit message: teilenummern
Parts:
- U5: value MAX690xPA -> MAX690CPA
Changed lines of the file:
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@@
 			)
 		)
+		(property "LCSC" "C5173393"
+			(at 0 0 0)
+			(unlocked yes)
+			(layer "F.Fab")
+			(hide yes)
+			(effects
+				(font
+					(size 1 1)
+					(thickness 0.15)
+				)
+			)
+		)
 		(property ki_fp_filters "DIN41612*2x*")
 		(sheetname "/")
@@
 			)
 		)
+		(property "LCSC" "C5173393"
+			(at 0 0 0)
+			(unlocked yes)
+			(layer "F.Fab")
+			(hide yes)
+			(effects
+				(font
+					(size 1 1)
+					(thickness 0.15)
+				)
+			)
+		)
 		(property ki_fp_filters "DIN41612*2x*")
 		(sheetname "/")
@@
 			)
 		)
+		(property "LCSC" "C127674"
+			(at 0 0 0)
+			(unlocked yes)
+			(layer "F.Fab")
+			(hide yes)
+			(effects
+				(font
+					(size 1 1)
+					(thickness 0.15)
+				)
+			)
+		)
 		(property ki_fp_filters "Crystal*")
 		(sheetname "/")
@@
 			)
 		)
-		(property "Value" "MAX690xPA"
+		(property "Value" "MAX690CPA"
 			(at 3.81 9.95 0)
 			(layer "F.Fab")
@@
 			)
 		)
+		(property "LCSC" "C3688193"
+			(at 0 0 0)
+			(unlocked yes)
+			(layer "F.Fab")
+			(hide yes)
+			(effects
+				(font
+					(size 1 1)
+					(thickness 0.15)
+				)
+			)
+		)
 		(property ki_fp_filters "*DIP*W7.62mm*")
 		(sheetname "/")
@@
 			)
 		)
+		(property "LCSC" "C75774"
+			(at 0 0 0)
+			(unlocked yes)
+			(layer "F.Fab")
+			(hide yes)
+			(effects
+				(font
+					(size 1 1)
+					(thickness 0.15)
+				)
+			)
+		)
 		(property ki_fp_filters "TQFP*10x10mm*P0.8mm*")
 		(sheetname "/")
@@
 		(tags "THT DIP DIL PDIP 2.54mm 15.24mm 600mil Socket")
 		(property "Reference" "U2"
-			(at 3.175 -3.175 180)
+			(at 3.175 -3.175 0)
 			(layer "F.SilkS")
 			(effects
@@
 			)
 		)
+		(property "LCSC" "C72122"
+			(at 0 0 0)
+			(unlocked yes)
+			(layer "F.Fab")
+			(hide yes)
+			(effects
+				(font
+					(size 1 1)
+					(thickness 0.15)
+				)
+			)
+		)
 		(property ki_fp_filters "DIP*W15.24mm* PLCC*")
 		(sheetname "/")
@@
 		(tags "THT DIP DIL PDIP 2.54mm 15.24mm 600mil Socket")
 		(property "Reference" "U1"
-			(at 17.78 4.445 180)
+			(at 17.78 4.445 0)
 			(layer "F.SilkS")
 			(effects
@@
 			)
 		)
+		(property "LCSC" "C72122"
+			(at 0 0 0)
+			(unlocked yes)
+			(layer "F.Fab")
+			(hide yes)
+			(effects
+				(font
+					(size 1 1)
+					(thickness 0.15)
+				)
+			)
+		)
 		(property ki_fp_filters "DIP*W15.24mm* PLCC*")
 		(sheetname "/")
@@
 					(thickness 0.15)
 				)
+			)
+		)
+		(property "LCSC" "C601936"
+			(at 0 0 0)
+			(unlocked yes)
+			(layer "F.Fab")
+			(hide yes)
+			(effects
+				(font
+					(size 1 1)
+					(thickness 0.15)
+				)

Commit message: jumper
Parts:
- JP1, JP2, JP3, JP4: footprint TestPoint:TestPoint_2Pads_Pitch5.08mm_Drill1.3mm -> NSM:NSM_Jumper
- moved JP1 2.55 mm to (71.2, 110.5)
- moved JP2 2.55 mm to (67.9, 110.5)
- moved JP3 2.44 mm to (67.9, 69.8)
- moved JP4 2.44 mm to (71.1, 69.8)

Commit message: sys25 erc
Parts:
- JP1: value Sound_4MBit -> 4MBit
- JP2: value Sound_2MBit -> 2MBit
- JP3: value Program_2MBit -> 2MBit
- JP4: value Program_4MBit -> 4MBit
- moved D1 0.38 mm to (67.8, 92.7)
Routing:
- net VDD: track 64.5 -> 65.1 mm
