File: Systemmodul25.2/Systemmodul25.2.kicad_sch (KiCad schematic)
At the start: 15 parts, among them J1 DIN41612_02x16_AB, J2 DIN41612_02x16_AB, J3 AVR-ISP-6, Q1 12.00J1, U1 W27E040, U2 W27E040, U3 M48Tx2, U4 ATmega8515-16A, U5 MAX690xPA

Commit message: modul
Parts:
- removed U3: M48Tx2, Package_DIP:DIP-24_18.0mmx34.29mm_W15.24mm, symbol Memory_RAM:M48Tx2
- added C2, C3, C6: 223, Capacitor_THT:C_Disc_D4.3mm_W1.9mm_P5.00mm, symbol Device:C
- added C4, C5: C_Polarized, Capacitor_THT:CP_Radial_Tantal_D5.0mm_P5.00mm, symbol Device:C_Polarized
- added C8, C9: 33, Capacitor_THT:C_Disc_D4.3mm_W1.9mm_P5.00mm, symbol Device:C
- added FID1, FID2: Fiducial, Fiducial:Fiducial_Cross_0.5mm_Mask2mm, symbol Mechanical:Fiducial
- added FID3, FID5: Fiducial, symbol Mechanical:Fiducial
- added FID4: Fiducial, Fiducial:Fiducial_0.5mm_Mask1mm, symbol Mechanical:Fiducial
- added H1: MountingHole, MountingHole:MountingHole_4.3mm_M4, symbol Mechanical:MountingHole
- added JP1, JP4: Jumper_2_Bridged, TestPoint:TestPoint_2Pads_Pitch5.08mm_Drill1.3mm, symbol Jumper:Jumper_2_Bridged
- added JP2, JP3: Jumper_2_Open, TestPoint:TestPoint_2Pads_Pitch5.08mm_Drill1.3mm, symbol Jumper:Jumper_2_Open
- added LED2: LED, LED_SMD:LED_1206_3216Metric, symbol Device:LED
- added R4: 220k, Resistor_THT:R_Axial_DIN0207_L6.3mm_D2.5mm_P10.16mm_Horizontal, symbol Device:R
- added U3: M48T18-100PC1, Package_DIP:DIP-28_W15.24mm, symbol NVRAM_ST:M48Tx8
- C1: footprint Capacitor_THT:CP_Radial_D8.0mm_P5.00mm -> Capacitor_THT:CP_Radial_Tantal_D7.0mm_P5.00mm
- R3: value 370 -> 470
Connections:
- net GND: now also C1.2, J2.a16 (Pin_a16), C2.2, C3.2, C4.2, C5.2, C6.2, C8.1, C9.1, U3.14 (V_{SS})
- net VCC: now reaches D1.2 (A)
- net VCC: now also J2.b2 (Pin_b2), J3.2 (VCC), LED1.1 (K), U1.1 (VPP), U1.32 (VCC), U2.1 (VPP), U2.32 (VCC), U4.38 (VCC), U5.2 (VCC), C3.1, C5.1, JP2.2 (B), JP3.2 (B), LED2.1 (K), R4.1
- net at R3.1: now also U4.44 (PB4)
- net at R3.2: now also LED1.2 (A), LED2.2 (A)
- net PRG_CE: now reaches U4.10 (PD4)
- net PRG_CE: now also J2.a6 (Pin_a6), U2.22 (~{CE})
- net at U4.14 (XTAL2): now also Q1.2, C8.2
- net at U4.15 (XTAL1): now also Q1.1, C9.2
- net PRG_D7: now reaches U4.30 (PA7)
- net PRG_D7: now also J2.a5 (Pin_a5), U2.21 (D7), U3.19 (DQ7)
- net PRG_D6: now reaches U4.31 (PA6)
- net PRG_D6: now also J2.a4 (Pin_a4), U2.20 (D6), U3.18 (DQ6)
- net PRG_D5: now reaches U4.32 (PA5)
- net PRG_D5: now also J2.a3 (Pin_a3), U2.19 (D5), U3.17 (DQ5)
- net PRG_D4: now reaches U4.33 (PA4)
- net PRG_D4: now also J2.a2 (Pin_a2), U2.18 (D4), U3.16 (DQ4)
- net PRG_D3: now reaches U4.34 (PA3)
- net PRG_D3: now also J2.a1 (Pin_a1), U2.17 (D3), U3.15 (DQ3)
- net PRG_D2: now reaches U4.35 (PA2)
- net PRG_D2: now also J2.b1 (Pin_b1), U2.15 (D2), U3.13 (DQ2)
- net PRG_D1: now reaches U4.36 (PA1)
- net PRG_D1: now also J2.b3 (Pin_b3), U2.14 (D1), U3.12 (DQ1)
- net PRG_D0: now reaches U4.37 (PA0)
- net PRG_D0: now also J2.b4 (Pin_b4), U2.13 (D0), U3.11 (DQ0)
- net at R1.2: now also U3.1 (~{INT}), U3.26 (E2)
- net PRG_A2: now reaches U2.10 (A2)
- net PRG_A2: now also J2.b7 (Pin_b7), U3.8 (A2)
- net PRG_A1: now reaches U2.11 (A1)
- net PRG_A1: now also J2.b6 (Pin_b6), U3.9 (A1)
- net PRG_A0: now reaches U2.12 (A0)
- net PRG_A0: now also J2.b5 (Pin_b5), U3.10 (A0)
- net PRG_A16: now reaches U2.2 (A16)
- net PRG_A16: now also J2.b16 (Pin_b16)
- net PRG_A10: now reaches U2.23 (A10)
- net PRG_A10: now also J2.a7 (Pin_a7), U3.21 (A10)
- net at U2.24 (~{OE}): now also U3.22 (~{G})
- net PRG_A11: now reaches U2.25 (A11)
- net PRG_A11: now also J2.a9 (Pin_a9), U3.23 (A11)
- net PRG_A9: now reaches U2.26 (A9)
- net PRG_A9: now also J2.a10 (Pin_a10), U3.24 (A9)
- net PRG_A8: now reaches U2.27 (A8)
- net PRG_A8: now also J2.a11 (Pin_a11), U3.25 (A8)
- net PRG_A13: now reaches U2.28 (A13)
- net PRG_A13: now also J2.a12 (Pin_a12)
- net PRG_A14: now reaches U2.29 (A14)
- net PRG_A14: now also J2.b14 (Pin_b14)
- net PRG_A15: now reaches U2.3 (A15)
- net PRG_A15: now also J2.a14 (Pin_a14)
- net PRG_A17: now reaches U2.30 (A17)
- net PRG_A17: now also J2.a15 (Pin_a15)
- net PRG_A18: now reaches U2.31 (A18)
- net PRG_A12: now reaches U2.4 (A12)
- net PRG_A12: now also J2.b13 (Pin_b13), U3.2 (A12)
- net PRG_A7: now reaches U2.5 (A7)
- net PRG_A7: now also J2.b12 (Pin_b12), U3.3 (A7)
- net PRG_A6: now reaches U2.6 (A6)
- net PRG_A6: now also J2.b11 (Pin_b11), U3.4 (A6)
- net PRG_A5: now reaches U2.7 (A5)
- net PRG_A5: now also J2.b10 (Pin_b10), U3.5 (A5)
- net PRG_A4: now reaches U2.8 (A4)
- net PRG_A4: now also J2.b9 (Pin_b9), U3.6 (A4)
- net PRG_A3: now reaches U2.9 (A3)
- net PRG_A3: now also J2.b8 (Pin_b8), U3.7 (A3)
- net SND_D1: now reaches J1.a1 (Pin_a1)
- net SND_D1: now also U1.14 (D1)
- net SND_A11: now reaches J1.a10 (Pin_a10)
- net SND_A11: now also U1.25 (A11)
- net SND_A13: now reaches J1.a11 (Pin_a11)
- net SND_A13: now also U1.28 (A13)
- net SND_A15: now reaches J1.a12 (Pin_a12)
- net SND_A15: now also U1.3 (A15)
- net SND_A17: now reaches J1.a13 (Pin_a13)
- net SND_A17: now also U1.30 (A17)
- net SND_OE: now reaches J1.a14 (Pin_a14)
- net SND_OE: now also U1.24 (~{OE})
- net SND_D2: now reaches J1.a15 (Pin_a15)
- net SND_D2: now also U1.15 (D2)
- net SND_D3: now reaches J1.a2 (Pin_a2)
- net SND_D3: now also U1.17 (D3)
- net SND_D5: now reaches J1.a3 (Pin_a3)
- net SND_D5: now also U1.19 (D5)
- net SND_D7: now reaches J1.a4 (Pin_a4)
- net SND_D7: now also U1.21 (D7)
- net SND_A1: now reaches J1.a5 (Pin_a5)
- net SND_A1: now also U1.11 (A1)
- net SND_A3: now reaches J1.a6 (Pin_a6)
- net SND_A3: now also U1.9 (A3)
- net SND_A5: now reaches J1.a7 (Pin_a7)
- net SND_A5: now also U1.7 (A5)
- net SND_A7: now reaches J1.a8 (Pin_a8)
- net SND_A7: now also U1.5 (A7)
- net SND_A9: now reaches J1.a9 (Pin_a9)
- net SND_A9: now also U1.26 (A9)
- net SND_D0: now reaches J1.b1 (Pin_b1)
- net SND_D0: now also U1.13 (D0)
- net SND_A10: now reaches J1.b10 (Pin_b10)
- net SND_A10: now also U1.23 (A10)
- net SND_A12: now reaches J1.b11 (Pin_b11)
- net SND_A12: now also U1.4 (A12)
- net SND_A14: now reaches J1.b12 (Pin_b12)
- net SND_A14: now also U1.29 (A14)
- net SND_A16: now reaches J1.b13 (Pin_b13)
- net SND_A16: now also U1.2 (A16)
- net SND_A18: now reaches J1.b14 (Pin_b14)
- net SND_A18: now also U1.31 (A18), JP1.2 (B)
- net SND_CE: now reaches J1.b15 (Pin_b15)
- net SND_CE: now also U1.22 (~{CE})
- net at J1.b2 (Pin_b2): now also J2.b15 (Pin_b15)
- net SND_D4: now reaches J1.b3 (Pin_b3)
- net SND_D4: now also U1.18 (D4)
- net SND_D6: now reaches J1.b4 (Pin_b4)
- net SND_D6: now also U1.20 (D6)
- net SND_A0: now reaches J1.b5 (Pin_b5)
- net SND_A0: now also U1.12 (A0)
- net SND_A2: now reaches J1.b6 (Pin_b6)
- net SND_A2: now also U1.10 (A2)
- net SND_A4: now reaches J1.b7 (Pin_b7)
- net SND_A4: now also U1.8 (A4)
- net SND_A6: now reaches J1.b8 (Pin_b8)
- net SND_A6: now also U1.6 (A6)
- net SND_A8: now reaches J1.b9 (Pin_b9)
- net SND_A8: now also U1.27 (A8)
- net at C1.1: now also C6.1
- net at J2.a13 (Pin_a13): now also U3.27 (~{W})
- net at J2.a8 (Pin_a8): now also U3.20 (~{E1})
- net at R2.1: now also U3.28 (V_{CC})
- new net: C2.1, C4.1
- new net: JP1.1 (A), JP2.1 (A)
- new net: JP3.1 (A), JP4.1 (A)
Other:
- moved on the sheet: C1, D1, J1, J2, J3, LED1, Q1, R1, R2, R3, U1, U2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

Commit message: oben
Connections:
- net VCC: now also C2.1, C4.1
- net at D1.1 (K): now also C1.1, C6.1, R1.1, R2.1, U3.28 (V_{CC})
- net at JP4.2 (B): now also J1.b16 (Pin_b16)
- net PRG_OE: now reaches U2.24 (~{OE}), U3.22 (~{G})
- net PRG_OE: now also J1.a16 (Pin_a16)
- net at J2.a8 (Pin_a8), U3.20 (~{E1}): now also R2.2
Other:
- moved on the sheet: C1, C6, D1, JP1, JP2, JP3, JP4, R1, R2

Commit message: modul atmega
Connections:
- net PRG_A10: now also U4.18 (PC0)
- net PRG_A11: now also U4.19 (PC1)
- net PRG_A12: now also U4.20 (PC2)
- net PRG_A13: now also U4.21 (PC3)
- net PRG_A14: now also U4.22 (PC4)
- net PRG_A15: now also U4.23 (PC5)
- net PRG_A16: now also U4.24 (PC6)
- net PRG_A17: now also U4.25 (PC7)
- net PRG_A8: now also U4.5 (PD0)
- net PRG_A9: now also U4.7 (PD1)
- net VDD: now reaches C1.1, C6.1, D1.1 (K), R1.1, R2.1, U3.28 (V_{CC})
- net NVRAM_W: now reaches U4.41 (PB1)
- net NVRAM_W: now also J2.a13 (Pin_a13), U3.27 (~{W}), U4.8 (PD2)
- net NVRAM_E1: now reaches U4.9 (PD3)
- net NVRAM_E1: now also J2.a8 (Pin_a8), R2.2, U3.20 (~{E1})
- net at U5.7 (~{RESET}): now also R4.2
- net NVRAM_E2: now reaches R1.2, U3.1 (~{INT}), U3.26 (E2)
- no-connect marks 0 -> 3
Other:
- moved on the sheet: D1, R1, R2, R4

Commit message: systemmodul fertig
Connections:
- net PRG_A18: now also J1.b16 (Pin_b16), JP4.2 (B); no longer U2.31 (A18)
- net SND_A18: no longer U1.31 (A18)
- net at JP1.1 (A), JP2.1 (A): now also U1.31 (A18)
- net at JP3.1 (A), JP4.1 (A): now also U2.31 (A18)
Other:
- moved on the sheet: JP1, JP2, JP3, JP4

Commit message: systemmodul reset
Parts:
- removed FID5: Fiducial, symbol Mechanical:Fiducial
- D1: value D -> BAT85
- FID1, FID2: footprint Fiducial:Fiducial_Cross_0.5mm_Mask2mm -> Fiducial:Fiducial_Cross_1.5mm_Mask2mm
- FID3: footprint (none) -> Fiducial:Fiducial_0.75mm_Mask1.5mm
- JP1: value Jumper_2_Bridged -> Sound_4MBit
- JP2: value Jumper_2_Open -> Sound_2MBit
- JP3: value Jumper_2_Open -> Program_2MBit
- JP4: value Jumper_2_Bridged -> Program_4MBit
Connections:
- net GND: now also U5.4 (PFI)
- net RESET: now reaches J3.5 (~{RST}), U4.4 (~{RESET})
- net RESET: now also R4.2, U5.7 (~{RESET})
- no-connect marks 3 -> 13
Other:
- moved on the sheet: C1, C2, C3, C4, C5, C6, C8, C9, D1, FID1, FID2, FID3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

Commit message: reset typ
Parts:
- U5: value MAX690xPA -> MAX690CPA
Changed lines of the file:
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@@
 			)
 		)
-		(property "Value" "MAX690xPA"
+		(property "Value" "MAX690CPA"
 			(at 149.4633 81.28 0)
 			(effects

Commit message: jumper
Parts:
- JP1, JP2, JP3, JP4: footprint TestPoint:TestPoint_2Pads_Pitch5.08mm_Drill1.3mm -> NSM:NSM_Jumper
Changed lines of the file:
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@@
 			)
 		)
-		(property "Footprint" "TestPoint:TestPoint_2Pads_Pitch5.08mm_Drill1.3mm"
+		(property "Footprint" "NSM:NSM_Jumper"
 			(at 30.48 152.4 0)
 			(effects
@@
 			)
 		)
-		(property "Footprint" "TestPoint:TestPoint_2Pads_Pitch5.08mm_Drill1.3mm"
+		(property "Footprint" "NSM:NSM_Jumper"
 			(at 96.52 152.4 0)
 			(effects
@@
 			)
 		)
-		(property "Footprint" "TestPoint:TestPoint_2Pads_Pitch5.08mm_Drill1.3mm"
+		(property "Footprint" "NSM:NSM_Jumper"
 			(at 30.48 142.24 0)
 			(effects
@@
 			)
 		)
-		(property "Footprint" "TestPoint:TestPoint_2Pads_Pitch5.08mm_Drill1.3mm"
+		(property "Footprint" "NSM:NSM_Jumper"
 			(at 96.52 142.24 0)
 			(effects

Commit message: sys25 erc
Parts:
- JP1: value Sound_4MBit -> 4MBit
- JP2: value Sound_2MBit -> 2MBit
- JP3: value Program_2MBit -> 2MBit
- JP4: value Program_4MBit -> 4MBit
