File: YMersatz/YMersatz.kicad_pcb (KiCad board)
At the start: 2 copper layers, 53 x 20 mm, 9 parts, among them J1 Conn_01x20, J2 Conn_01x20, U1 74LS574, U2 74LS08, Y1 SG-615

Commit message: ym pins
Parts:
- moved J1 48.3 mm to (70.3, 22.0), turned to -90 degrees
Connections:
- net Net-(J2-Pin_10) renamed /IOB3
- net Net-(J2-Pin_11) renamed /IOB2
- net Net-(J2-Pin_12) renamed /IOB1
- net Net-(J2-Pin_13) renamed /IOB0
- net Net-(J2-Pin_6) renamed /IOB7
- net Net-(J2-Pin_7) renamed /IOB6
- net Net-(J2-Pin_8) renamed /IOB5
- net Net-(J2-Pin_9) renamed /IOB4
- net SO renamed SoundOut_B
- J1 pad 1: +5V -> /IOA0
- J1 pad 10: /D6 -> /D7
- J1 pad 11: /D7 -> /D6
- J1 pad 12: unconnected-(J1-Pin_12-Pad12) -> /D5
- J1 pad 13: +5V -> /D4
- J1 pad 14: unconnected-(J1-Pin_14-Pad14) -> /D3
- J1 pad 15: unconnected-(J1-Pin_15-Pad15) -> /D2
- J1 pad 16: +5V -> /D1
- J1 pad 17: unconnected-(J1-Pin_17-Pad17) -> /D0
- J1 pad 18: unconnected-(J1-Pin_18-Pad18) -> /C
- J1 pad 19: unconnected-(J1-Pin_19-Pad19) -> /TEST1
- J1 pad 2: unconnected-(J1-Pin_2-Pad2) -> /CLOCK
- J1 pad 20: unconnected-(J1-Pin_20-Pad20) -> +5V
- J1 pad 3: unconnected-(J1-Pin_3-Pad3) -> /~{RESET}
- J1 pad 4: /D0 -> /~{A9}
- J1 pad 5: /D1 -> /A8
- J1 pad 6: /D2 -> /SEL
- J1 pad 7: /D3 -> /BDIR
- J1 pad 8: /D4 -> /BC2
- J1 pad 9: /D5 -> /BC1
- J2 pad 14: unconnected-(J2-Pin_14-Pad14) -> /IOA7
- J2 pad 15: unconnected-(J2-Pin_15-Pad15) -> /IOA6
- J2 pad 16: unconnected-(J2-Pin_16-Pad16) -> /IOA5
- J2 pad 17: unconnected-(J2-Pin_17-Pad17) -> /IOA4
- J2 pad 18: unconnected-(J2-Pin_18-Pad18) -> /IOA3
- J2 pad 19: unconnected-(J2-Pin_19-Pad19) -> /IOA2
- J2 pad 20: unconnected-(J2-Pin_20-Pad20) -> /IOA1
- J2 pad 3: unconnected-(J2-Pin_3-Pad3) -> A
Routing:
- net unconnected-(J1-Pin_18-Pad18): track 8.20 -> 0.00 mm
- net /~{RESET}: track 0.00 -> 8.20 mm
- net unconnected-(J1-Pin_3-Pad3): track 7.28 -> 0.00 mm
- net /C: track 0.00 -> 7.28 mm
- net unconnected-(J1-Pin_20-Pad20): track 5.33 -> 0.00 mm
- net /IOA0: track 0.00 -> 5.33 mm
- net unconnected-(J2-Pin_3-Pad3): track 3.89 -> 0.00 mm
- net A: track 0.00 -> 3.89 mm
