File: ArduinoISP/ArduinoISP.kicad_sch (KiCad schematic)
At the start: 11 parts, among them J1 Analog, J2 Digital, J3 AVR-ISP-10, J4 AVR-ISP-6

Commit message: erc
Parts:
- J4: footprint Arduino_MountingHole:IDC-Header_2x03_P2.54mm_Horizontal -> ArduinoISP:IDC-Header_2x03_P2.54mm_Horizontal
Other:
- company: (none) -> sD
- title: (none) -> ArduinoISP
