File: DB512k/DB512k.kicad_sch (KiCad schematic)
At the start: 130 parts, among them J7 Conn_01x04_Socket, J8 DIN41612_03x10_ABC, J9 DIN41612_03x10_ABC, Q1 Q_Photo_NPN_CBE, Q2 Q_Photo_NPN_CBE, Q3 BSS84, Q4 IRF7313, Q5 BC807-40W, Q6 BC846, U1 MC68331, U10 RTC4543, U11 74LS08, U2 AT90S1200A, U3 CY62157, U4 74LS573, U5 74LS245, U6 74LS573, U7 74LS573, U8 74LS245, U9 74LS20, Y1 32.768k

Commit message: weg
Parts:
- removed C35: C, Capacitor_SMD:C_0805_2012Metric, symbol Device:C
- removed D11: BAS28, Package_TO_SOT_SMD:SOT-143, symbol DualDiode:BAS28
- removed R4: 1k, Resistor_SMD:R_0603_1608Metric, symbol Device:R
- removed R8: R, Resistor_SMD:R_0603_1608Metric, symbol Device:R
- removed RN1, RN12, RN3: 330, Resistor_SMD:R_Array_Concave_4x0603, symbol Device:R_Pack04
- removed RN10, RN2: 750, Resistor_SMD:R_Array_Concave_4x0603, symbol Device:R_Pack04
- removed RN11, RN4, RN5, RN9: R_Pack04, Resistor_SMD:R_Array_Concave_4x0603, symbol Device:R_Pack04
- removed RN13, RN6, RN7, RN8: 822, Resistor_SMD:R_Array_Concave_4x0603, symbol Device:R_Pack04
- removed TP12, TP21, TP29, TP30, TP6, TP8: TestPoint, TestPoint:TestPoint_Pad_D1.0mm, symbol Connector:TestPoint
- removed U3: CY62157, Package_SO:TSOP-II-44_10.16x18.41mm_P0.8mm, symbol NXP:CY62157
- added J1: Conn_01x04_Socket, ADP:Deckel, symbol Connector:Conn_01x04_Socket
- added U12, U13, U14, U3: HM628128_TSOP32, Package_SO:TSOP-I-32_18.4x8mm_P0.5mm, symbol Memory_RAM:HM628128_TSOP32
- U2: footprint Package_SO:SSOP-20_5.3x7.2mm_P0.65mm -> Package_SO:SOIC-20W_7.5x12.8mm_P1.27mm
- U4, U5, U6, U7, U8: footprint Package_SO:TSSOP-20_4.4x6.5mm_P0.65mm -> Package_SO:SO-20_12.8x7.5mm_P1.27mm
Connections:
- net A0: no longer U1.115 (A0)
- net A1: now also U12.20 (A0), U13.20 (A0), U14.20 (A0), U3.20 (A0)
- net A10: now also U12.2 (A9), U13.2 (A9), U14.2 (A9), U3.2 (A9)
- net A11: now also U12.31 (A10), U13.31 (A10), U14.31 (A10), U3.31 (A10)
- net A12: now also U12.1 (A11), U13.1 (A11), U14.1 (A11), U3.1 (A11)
- net A13: now also U12.12 (A12), U13.12 (A12), U14.12 (A12), U3.12 (A12)
- net A14: now also U12.4 (A13), U13.4 (A13), U14.4 (A13), U3.4 (A13)
- net A15: now also U12.11 (A14), U13.11 (A14), U14.11 (A14), U3.11 (A14)
- net A16: now also U12.7 (A15), U13.7 (A15), U14.7 (A15), U3.7 (A15)
- net A17: now also U12.10 (A16), U13.10 (A16), U14.10 (A16), U3.10 (A16)
- net A2: now also U12.19 (A1), U13.19 (A1), U14.19 (A1), U3.19 (A1)
- net A3: now also U12.18 (A2), U13.18 (A2), U14.18 (A2), U3.18 (A2)
- net A4: now also U12.17 (A3), U13.17 (A3), U14.17 (A3), U3.17 (A3)
- net A5: now also U12.16 (A4), U13.16 (A4), U14.16 (A4), U3.16 (A4)
- net A6: now also U12.15 (A5), U13.15 (A5), U14.15 (A5), U3.15 (A5)
- net A7: now also U12.14 (A6), U13.14 (A6), U14.14 (A6), U3.14 (A6)
- net A8: now also U12.13 (A7), U13.13 (A7), U14.13 (A7), U3.13 (A7)
- net A9: now also U12.3 (A8), U13.3 (A8), U14.3 (A8), U3.3 (A8)
- net D0: now also U13.21 (I/O0), U14.21 (I/O0)
- net D1: now also U13.22 (I/O1), U14.22 (I/O1)
- net D10: now also U5.4 (A2), U12.23 (I/O2), U3.23 (I/O2); no longer U5.7 (A5)
- net D11: now also U5.5 (A3), U12.25 (I/O3), U3.25 (I/O3); no longer U5.6 (A4)
- net D12: now also U5.6 (A4), U12.26 (I/O4), U3.26 (I/O4); no longer U5.5 (A3)
- net D13: now also U5.7 (A5), U12.27 (I/O5), U3.27 (I/O5); no longer U5.4 (A2)
- net D14: now also U5.8 (A6), U12.28 (I/O6), U3.28 (I/O6); no longer U5.3 (A1)
- net D15: now also U5.9 (A7), U12.29 (I/O7), U3.29 (I/O7); no longer U5.2 (A0)
- net D2: now also U13.23 (I/O2), U14.23 (I/O2)
- net D3: now also U13.25 (I/O3), U14.25 (I/O3)
- net D4: now also U13.26 (I/O4), U14.26 (I/O4)
- net D5: now also U13.27 (I/O5), U14.27 (I/O5)
- net D6: now also U13.28 (I/O6), U14.28 (I/O6)
- net D7: now also U13.29 (I/O7), U14.29 (I/O7)
- net D8: now also U5.2 (A0), U12.21 (I/O0), U3.21 (I/O0); no longer U5.9 (A7)
- net D9: now also U5.3 (A1), U12.22 (I/O1), U3.22 (I/O1); no longer U5.8 (A6)
- net GND: now also U12.24 (GND), U13.24 (GND), U14.24 (GND), U3.24 (GND)
- net VDD: now also U12.8 (VCC), U13.8 (VCC), U14.8 (VCC), U3.8 (VCC)
- net cD10: now also U5.16 (B2); no longer J8.c9 (Pin_c9), U4.14 (Q5), U5.13 (B5)
- net cD11: now also U5.15 (B3); no longer J8.a8 (Pin_a8), U4.15 (Q4), U5.14 (B4)
- net cD12: now also U5.14 (B4); no longer J8.b8 (Pin_b8), U4.16 (Q3), U5.15 (B3)
- net cD13: now also U5.13 (B5); no longer J8.c8 (Pin_c8), U4.17 (Q2), U5.16 (B2)
- net cD14: now also U5.12 (B6); no longer J8.b7 (Pin_b7), U4.18 (Q1), U5.17 (B1)
- net cD15: now also U5.11 (B7); no longer J8.c7 (Pin_c7), U4.19 (Q0), U5.18 (B0)
- net cD8: now also U5.18 (B0); no longer J8.a9 (Pin_a9), U4.12 (Q7), U5.11 (B7)
- net cD9: now also U5.17 (B1); no longer J8.b9 (Pin_b9), U4.13 (Q6), U5.12 (B6)
- net at R12.1, Y1.1: no longer C32.1
- net cPQS3: no longer names the net of J9.b1 (Pin_b1)
- no-connect marks 21 -> 10
Other:
- moved on the sheet: U5

Commit message: rtc
Parts:
- added Y3: Resonator, Crystal:Resonator_SMD-3Pin_7.2x3.0mm, symbol Device:Resonator
- R23, R25, R26, R28: value ~ -> (none)
Connections:
- net A1: now also U6.9 (D7); no longer U6.3 (D1)
- net A2: now also U6.8 (D6); no longer U6.4 (D2)
- net A3: now also U6.7 (D5); no longer U6.5 (D3)
- net A4: now also U6.6 (D4)
- net A5: no longer U6.9 (D7)
- net A6: no longer U6.8 (D6)
- net A7: no longer U6.7 (D5)
- net A8: no longer U6.6 (D4)
- net GND: now also Y3.2
- net MOSI: no longer U10.11 (DATA), U10.6 (WR)
- net SCK: no longer U10.12 (CLK)
- net cA1: now also J9.c3 (Pin_c3), U6.12 (Q7); no longer J9.c4 (Pin_c4), U6.18 (Q1)
- net cA2: now also J9.a2 (Pin_a2), U6.13 (Q6); no longer J9.a3 (Pin_a3), U6.17 (Q2)
- net cA3: now also J9.b2 (Pin_b2), U6.14 (Q5); no longer J9.b3 (Pin_b3), U6.16 (Q3)
- net cA5: no longer J9.c3 (Pin_c3), U6.12 (Q7)
- net cA6: no longer J9.a2 (Pin_a2), U6.13 (Q6)
- net cA7: no longer J9.b2 (Pin_b2), U6.14 (Q5)
- net cA8: no longer J9.c2 (Pin_c2), U6.15 (Q4)
- net cD0: now also U8.18 (B0); no longer U8.11 (B7)
- net cD1: now also U8.17 (B1); no longer U8.12 (B6)
- net cD2: now also U8.16 (B2); no longer U8.13 (B5)
- net cD3: now also U8.15 (B3); no longer U8.14 (B4)
- net cD4: now also U8.14 (B4); no longer U8.15 (B3)
- net cD5: now also U8.13 (B5); no longer U8.16 (B2)
- net cD6: now also U8.12 (B6); no longer U8.17 (B1)
- net cD7: now also U8.11 (B7); no longer U8.18 (B0)
- net at U10.5 (Foe): now also U10.7 (Fsel)
- net RTC_CLK: now reaches U2.11 (PD6)
- net RTC_CLK: now also U10.12 (CLK)
- net RTC_DATA: now reaches U2.2 (PD0)
- net RTC_DATA: now also U10.11 (DATA)
- net at U2.4 (XTAL2): now also Y3.3
- net at U2.5 (XTAL1): now also Y3.1
- net A0: no longer names the net of U6.2 (D0)
- net cA0: no longer names the net of J9.b4 (Pin_b4), U6.19 (Q0)
- new net: J9.c2 (Pin_c2), U6.15 (Q4)
- new net: J9.b3 (Pin_b3), U6.16 (Q3)
- new net: J9.a3 (Pin_a3), U6.17 (Q2)
- new net: J9.c4 (Pin_c4), U6.18 (Q1)
Other:
- moved on the sheet: U2

Commit message: chips
Parts:
- removed C27: C, Capacitor_SMD:C_0805_2012Metric, symbol Device:C
- removed C40: C, Capacitor_SMD:C_1206_3216Metric, symbol Device:C
- removed D4, D5: BAS40-05, Package_TO_SOT_SMD:SOT-23-3, symbol Device:D_Schottky_Dual_CommonCathode_AAK
- removed Q3: BSS84, Package_TO_SOT_SMD:SOT-23, symbol Transistor_FET:BSS84
- removed Q4: IRF7313, Package_SO:SOIC-8_3.9x4.9mm_P1.27mm, symbol Transistor_FET:IRF7309IPBF
- removed Q5: BC807-40W, Package_TO_SOT_SMD:TSOT-23, symbol Transistor_BJT:Q_PNP_BEC
- removed R1: 10, Resistor_SMD:R_0805_2012Metric, symbol Device:R
- removed R2: 1, Resistor_SMD:R_0805_2012Metric, symbol Device:R
- removed R22: 10M, Resistor_SMD:R_1206_3216Metric, symbol Device:R
- removed R23, R26: (no value), Resistor_SMD:R_0603_1608Metric, symbol Device:R
- removed TP10, TP11, TP20, TP28, TP9: TestPoint, TestPoint:TestPoint_Pad_D1.0mm, symbol Connector:TestPoint
- removed TP36: TestPoint, TestPoint:TestPoint_Pad_D1.5mm, symbol Connector:TestPoint
- removed U4: 74LS573, Package_SO:SO-20_12.8x7.5mm_P1.27mm, symbol 74xx:74LS573
- removed U9: 74LS20, Package_SO:TSSOP-14_4.4x5mm_P0.65mm, symbol 74xx:74LS20
- added D4: SM6T6V8A, Diode_SMD:D_SMB, symbol Diode:SM6T6V8A
- added Q3: BSP31, Package_TO_SOT_SMD:SOT-223, symbol Transistor_BJT:Q_PNP_BCEC
- added U15: 74HC10, Package_SO:SO-14_3.9x8.65mm_P1.27mm, symbol 74xx:74LS10
- added U16: TS3704, Package_SO:SO-14_3.9x8.65mm_P1.27mm, symbol Comparator:LM339
- added U4: 74HC245, Package_SO:SO-20_12.8x7.5mm_P1.27mm, symbol 74xx:74HC245
- added U9: MAX691A CSE, Package_SO:SO-16_3.9x9.9mm_P1.27mm, symbol Power_Supervisor:MAX691xWE
- U11: value 74LS08 -> 74HC08; footprint Package_SO:TSSOP-14_4.4x5mm_P0.65mm -> Package_SO:SO-14_3.9x8.65mm_P1.27mm
- U6, U7: value 74LS573 -> 74HC573
- U8: value 74LS245 -> 74HC245
Connections:
- net A21: no longer U11.10, U11.5, U11.9
- net D10: now also U4.7 (A5)
- net D11: now also U4.6 (A4)
- net D12: now also U4.5 (A3)
- net D13: now also U4.4 (A2)
- net D14: now also U4.3 (A1)
- net D15: now also U4.2 (A0)
- net D8: now also U4.9 (A7)
- net D9: now also U4.8 (A6)
- net FC2: no longer U11.12, U11.13, U11.4
- net GND: now also U7.10 (GND), D4.2 (A2), U15.7 (GND), U16.12 (V-), U9.4 (GND)
- net at U11.1: no longer U11.2
- new net: U16.5 (+), U16.6 (-)
