File: VideoEncoder/VideoEncoder.kicad_sch (KiCad schematic)
At the start: 42 parts, among them Q1 SAs, Q2 SAs, U1 LD1086D2M33TR, U10 74LCX245, U11 HD63484_PLCC, U12 AM29F400Bx-xxEx, U13 74LCX573, U14 EPM7032, U15 74AHCT125, U16 HYB514171, U17 MSM5416283, U18 74LVC2G157, U19 74LCX32, U2 74LCX32, U20 74LVC2G157, U21 SAA7105, U22 74LCX573, U3 74LCX14, U4 74HC00, U5 74LCX573, U6 74LCX245, U7 74LCX245, U8 74LCX573, U9 74LCX573, Y1 SG-615

Commit message: jumper
Parts:
- added J1: DE15_Socket_HighDensity_MountingHoles, Connector_Dsub:DSUB-15-HD_Pins_Horizontal_P2.29x1.90mm_EdgePinOffset3.03mm_Housed_MountingHolesOffset4.94mm, symbol Connector:DE15_Socket_HighDensity_MountingHoles
- added J2: Conn_01x06, Connector_Stocko:Stocko_MKS_1656-6-0-606_1x6_P2.50mm_Vertical, symbol Connector_Generic:Conn_01x06
- added JP1, JP2, JP3: SolderJumper_2_Open, Jumper:SolderJumper-2_P1.3mm_Open_Pad1.0x1.5mm, symbol Jumper:SolderJumper_2_Open
- R1, R10, R11, R2, R3, R4, R5, R6, R7, R8, R9: footprint (none) -> Resistor_SMD:R_0805_2012Metric

Commit message: intel
Parts:
- U12: value AM29F400Bx-xxEx -> JS28F640; symbol Memory_Flash:AM29F400Bx-xxEx -> Memory:JS28F640
Connections:
- net R: now reaches J2.1 (Pin_1)
- net G: now reaches J2.2 (Pin_2)
- net B: now reaches J2.3 (Pin_3)
- net GND: now reaches J2.4 (Pin_4)
- net GND: now also U11.17 (GND), U11.18 (GND), U11.35 (GND), U11.54 (GND), U11.55 (GND), U13.10 (GND), U4.7 (GND), U5.10 (GND), U6.10 (GND), U7.10 (GND), U8.10 (GND)
- net SYN: now reaches J2.5 (Pin_5)
- net MAD8: now reaches U6.3 (A1)
- net MAD8: now also U11.48 (MAD8)
- net MAD9: now reaches U6.5 (A3)
- net MAD9: now also U11.47 (MAD9)
- net MAD10: now reaches U6.7 (A5)
- net MAD10: now also U11.46 (MAD10)
- net MAD11: now reaches U6.9 (A7)
- net MAD11: now also U11.45 (MAD11)
- net MAD15: now reaches U11.41 (MAD15)
- net MAD14: now reaches U11.42 (MAD14)
- net MAD13: now reaches U11.43 (MAD13)
- net MAD13: now also U7.5 (A3)
- net MAD12: now reaches U11.44 (MAD12)
- net MAD12: now also U7.3 (A1)
- net MAD7: now reaches U11.49 (MAD7)
- net MAD7: now also U5.9 (D7)
- net MAD6: now reaches U11.50 (MAD6)
- net MAD6: now also U5.8 (D6)
- net MAD5: now reaches U11.51 (MAD5)
- net MAD5: now also U5.7 (D5)
- net MAD4: now reaches U11.61 (MAD4)
- net MAD4: now also U5.6 (D4)
- net MAD3: now reaches U11.62 (MAD3)
- net MAD3: now also U5.5 (D3)
- net MAD2: now reaches U11.63 (MAD2)
- net MAD2: now also U5.4 (D2)
- net MAD1: now reaches U11.64 (MAD1)
- net MAD1: now also U5.3 (D1)
- net MAD0: now reaches U11.65 (MAD0)
- net MAD0: now also U5.2 (D0)
- net at U12.27 (A2): no longer U12.46 (VSS)
- no-connect marks 0 -> 1
Other:
- moved on the sheet: J2, R10, R8, U15A, U15B, U15C, U15D, U15E, U5, U6, U7
