File: SteuereinheitBackgammonMoM/SteuereinheitBackgammonMoM.kicad_sch (KiCad schematic)
At the start: 47 parts, among them J1 Service, J2 Conn_02x05_Odd_Even, J3 Serienplan, J4 Reserve, J9 Netzteil, Q1 BSS100, U1 TDA1308, U10 74HC245, U11 74HC245, U12 74HC273, U13 74LS139, U14 74HC00, U15 74HC74, U16 L4962-A, U18 74HC138, U19 27C512, U2 74HC04, U20 27C512, U22 MP696P, U24 68681, U25 68230, U26 uPD4168C, U27 uPD4168C, U28 MC68000P, U3 74HC04, U4 74HC30, U5 HEF4094B, U6 74HC164, U7 74HC32, U8 74HC245, U9 74HC245, Y1 3.6864MHZ

Commit message: strom
Parts:
- added J5: LAUTSPRECHER, Connector_Stocko:Stocko_MKS_1652-6-0-202_1x2_P2.50mm_Vertical, symbol Connector_Generic:Conn_01x02
- added J6: SERIELL, Connector_Stocko:Stocko_MKS_1658-6-0-808_1x8_P2.50mm_Vertical, symbol Connector_Generic:Conn_01x08
- added RN6: 10K, Resistor_THT:R_Array_SIP9, symbol Device:R_Network08
- added RV1: 10K, Potentiometer_THT:Potentiometer_Piher_PT-10-V10_Vertical, symbol Device:R_Potentiometer
Connections:
- net +12V: now also J6.8 (Pin_8)
- net +24V: now also J6.4 (Pin_4)
- net +48V: now also J6.2 (Pin_2)
- net +5V: now also J6.1 (Pin_1)
- net A17: now also U10.2 (A0)
- net A18: now also U10.3 (A1)
- net A19: now also U10.4 (A2)
- net A20: now also U10.5 (A3)
- net A21: now also U10.6 (A4)
- net A22: now also U10.7 (A5)
- net A23: now also U10.8 (A6)
- net BUS_A1: now also U23.3 (A0), U24.1 (RS1)
- net BUS_A17: now also U10.18 (B0)
- net BUS_A18: now also U10.17 (B1)
- net BUS_A19: now also U10.16 (B2)
- net BUS_A2: now also U24.3 (RS2)
- net BUS_A20: now also U10.15 (B3)
- net BUS_A21: now also U10.14 (B4), U18.1 (A0)
- net BUS_A22: now also U10.13 (B5), U18.2 (A1)
- net BUS_A23: now also U10.12 (B6), U18.3 (A2)
- net BUS_A3: now also U24.5 (RS3)
- net BUS_A4: now also U24.6 (RS4)
- net CLK: now also U14.9, U23.8 (CLK), U25.40 (CLK)
- net D0: now also U21.14 (D0)
- net D1: now also U21.13 (D1)
- net D2: now also U21.12 (D2)
- net D3: now also U21.11 (D3)
- net GND: now also U11.19 (CE), U13.8 (GND), U14.7 (GND), U15.7 (GND), U18.8 (GND), U21.9 (GND), U6.7 (GND), U9.19 (CE), J5.2 (Pin_2), J6.7 (Pin_7)
- net RW: now also U25.43 (R/W), U8.1 (A->B)
- net TS0: now also RN5.4 (R3), U24.7 (IP0)
- net TS1: now also RN5.3 (R2), U24.4 (IP1)
- net TS2: now also RN5.5 (R4)
- net TS3: now also RN5.7 (R6)
- net TS4: now also RN5.6 (R5)
- net TS5: now also RN5.2 (R1)
- net TS6: now also RN5.8 (R7)
- net TS7: now also RN5.9 (R8)
- net TS_A0: no longer U24.6 (RS4)
- net TS_A1: no longer U24.5 (RS3)
- net TS_A2: now also RN6.9 (R8); no longer U24.3 (RS2)
- net TS_A3: now also RN6.7 (R6); no longer U24.1 (RS1)
- net VCC: now reaches U6.14 (VCC)
- net VCC: now also R1.2, R2.2, RN1.1 (common), RN2.1 (common), RN3.1 (common), RN4.1 (common), U10.1 (A->B), U10.20 (VCC), U11.20 (VCC), U12.20 (VCC), U14.10, U14.13, U14.14 (VCC), U15.14 (VCC), U18.16 (VCC), U19.28 (VCC), U20.28 (VCC), U21.18 (VDD), U22.3 (VCC), U23.18 (Vcc), U24.40 (VCC), U25.12 (VCC), U26.28 (V_{CC}), U27.28 (V_{CC}), U28.13 (~{BR}), U28.14 (V_{CC}), U28.49 (V_{CC}), U5.16 (V_{DD}), U7.14 (VCC), U8.20 (VCC), U9.1 (A->B), U9.20 (VCC)
- net IPL0: now reaches U15.8 (~{Q})
- net IPL0: now also U28.25 (~{IPL0})
- net at U18.15 (~{Y0}): now also U4.4
- net TX: now reaches U3.6
- net TX: now also J6.6 (Pin_6)
- net at R1.1: now also U23.7 (~{DTACK})
- net at R2.1: now also U24.21 (IRQ)
- net PC6: now reaches U22.11 (WDI)
- net PC6: now also U25.36 (PC6/PIACK)
- net at U24.27 (OP4): now also RN6.4 (R3)
- net RX: now reaches U24.31 (RXDA)
- net RX: now also J6.3 (Pin_3)
- net IPL2: now reaches U28.23 (~{IPL2})
- net IPL1: now reaches U28.24 (~{IPL1})
- net at U21.10 (~{WR}): now also U15.6 (~{Q})
- net at U21.15 (CS1): now also R4.2
- net at U21.8 (~{RD}): now also U15.5 (Q)
- new net LS: J5.1 (Pin_1)
- no-connect marks 2 -> 3
Other:
- moved on the sheet: R1, R2, R4, RN3, U10, U14C, U14D, U15A, U21, U23
