File: SteuereinheitBackgammonMoM/SteuereinheitBackgammonMoM.kicad_pcb (KiCad board)
At the start: 2 copper layers, 315 x 147.4 mm, 46 parts, among them J1 Service, J2 Conn_02x05_Odd_Even, J3 Serienplan, J4 Reserve, J9 Netzteil, Q1 BSS100, U10 74HC245, U11 74HC245, U12 74HC273, U13 74LS139, U14 74HC00, U15 74HC74, U16 L4962-A, U18 74HC138, U19 27C512, U2 74HC04, U20 27C512, U22 MP696P, U24 68681, U25 68230, U26 uPD4168C, U27 uPD4168C, U28 MC68000P, U3 74HC04, U4 74HC30, U5 HEF4094B, U6 74HC164, U7 74HC32, U8 74HC245, U9 74HC245, Y1 3.6864MHZ

Commit message: rarr
Parts:
- added J5: LAUTSPRECHER, Connector_Stocko:Stocko_MKS_1652-6-0-202_1x2_P2.50mm_Vertical, F.Cu at (354.4, 83.1)
- added J6: SERIELL, Connector_Stocko:Stocko_MKS_1658-6-0-808_1x8_P2.50mm_Vertical, F.Cu at (354.4, 115.1)
- added RN6: 10K, Resistor_THT:R_Array_SIP9, F.Cu at (322.0, 189.4)
- added RV1: 10K, Potentiometer_THT:Potentiometer_Piher_PT-10-V10_Vertical, F.Cu at (289.6, 93.4)
Connections:
- R1 pad 1: unconnected-(R1-Pad1) -> Net-(U23-~{DTACK})
- R1 pad 2: unconnected-(R1-Pad2) -> VCC
- R2 pad 1: unconnected-(R2-Pad1) -> Net-(U24-IRQ)
- R2 pad 2: unconnected-(R2-Pad2) -> VCC
- R4 pad 2: unconnected-(R4-Pad2) -> Net-(U21-CS1)
- RN1 pad 1: unconnected-(RN1-common-Pad1) -> VCC
- RN2 pad 1: unconnected-(RN2-common-Pad1) -> VCC
- RN3 pad 1: unconnected-(RN3-common-Pad1) -> VCC
- RN4 pad 1: unconnected-(RN4-common-Pad1) -> VCC
- RN5 pad 2: unconnected-(RN5-R1-Pad2) -> TS5
- RN5 pad 3: unconnected-(RN5-R2-Pad3) -> TS1
- RN5 pad 4: unconnected-(RN5-R3-Pad4) -> TS0
- RN5 pad 5: unconnected-(RN5-R4-Pad5) -> TS2
- RN5 pad 6: unconnected-(RN5-R5-Pad6) -> TS4
- RN5 pad 7: unconnected-(RN5-R6-Pad7) -> TS3
- RN5 pad 8: unconnected-(RN5-R7-Pad8) -> TS6
- RN5 pad 9: unconnected-(RN5-R8-Pad9) -> TS7
- U10 pad 1: unconnected-(U10-A->B-Pad1) -> VCC
- U10 pad 12: unconnected-(U10-B6-Pad12) -> BUS_A23
- U10 pad 13: unconnected-(U10-B5-Pad13) -> BUS_A22
- U10 pad 14: unconnected-(U10-B4-Pad14) -> BUS_A21
- U10 pad 15: unconnected-(U10-B3-Pad15) -> BUS_A20
- U10 pad 16: unconnected-(U10-B2-Pad16) -> BUS_A19
- U10 pad 17: unconnected-(U10-B1-Pad17) -> BUS_A18
- U10 pad 18: unconnected-(U10-B0-Pad18) -> BUS_A17
- U10 pad 2: unconnected-(U10-A0-Pad2) -> A17
- U10 pad 20: unconnected-(U10-VCC-Pad20) -> VCC
- U10 pad 3: unconnected-(U10-A1-Pad3) -> A18
- U10 pad 4: unconnected-(U10-A2-Pad4) -> A19
- U10 pad 5: unconnected-(U10-A3-Pad5) -> A20
- U10 pad 6: unconnected-(U10-A4-Pad6) -> A21
- U10 pad 7: unconnected-(U10-A5-Pad7) -> A22
- U10 pad 8: unconnected-(U10-A6-Pad8) -> A23
- U11 pad 19: unconnected-(U11-CE-Pad19) -> GND
- U11 pad 20: unconnected-(U11-VCC-Pad20) -> VCC
- U12 pad 20: unconnected-(U12-VCC-Pad20) -> VCC
- U13 pad 8: unconnected-(U13C-GND-Pad8) -> GND
- U14 pad 10: Net-(U14-Pad10) -> VCC
- U14 pad 13: Net-(U14-Pad10) -> VCC
- U14 pad 14: unconnected-(U14E-VCC-Pad14) -> VCC
- U14 pad 7: unconnected-(U14E-GND-Pad7) -> GND
- U14 pad 9: unconnected-(U14-Pad9) -> CLK
- U15 pad 14: unconnected-(U15C-VCC-Pad14) -> VCC
- U15 pad 5: unconnected-(U15A-Q-Pad5) -> Net-(U15A-Q)
- U15 pad 6: unconnected-(U15A-~{Q}-Pad6) -> Net-(U15A-~{Q})
- U15 pad 7: unconnected-(U15C-GND-Pad7) -> GND
- U15 pad 8: unconnected-(U15B-~{Q}-Pad8) -> IPL0
- U18 pad 1: unconnected-(U18-A0-Pad1) -> BUS_A21
- U18 pad 15: unconnected-(U18-~{Y0}-Pad15) -> Net-(U18-~{Y0})
- U18 pad 16: unconnected-(U18-VCC-Pad16) -> VCC
- U18 pad 2: unconnected-(U18-A1-Pad2) -> BUS_A22
- U18 pad 3: unconnected-(U18-A2-Pad3) -> BUS_A23
- U18 pad 8: unconnected-(U18-GND-Pad8) -> GND
- U19 pad 28: unconnected-(U19-VCC-Pad28) -> VCC
- U20 pad 28: unconnected-(U20-VCC-Pad28) -> VCC
- U21 pad 10: unconnected-(U21-~{WR}-Pad10) -> Net-(U15A-~{Q})
- U21 pad 11: unconnected-(U21-D3-Pad11) -> D3
- U21 pad 12: unconnected-(U21-D2-Pad12) -> D2
- U21 pad 13: unconnected-(U21-D1-Pad13) -> D1
- U21 pad 14: unconnected-(U21-D0-Pad14) -> D0
- U21 pad 15: unconnected-(U21-CS1-Pad15) -> Net-(U21-CS1)
- U21 pad 18: unconnected-(U21-VDD-Pad18) -> VCC
- U21 pad 8: unconnected-(U21-~{RD}-Pad8) -> Net-(U15A-Q)
- U21 pad 9: unconnected-(U21-GND-Pad9) -> GND
- U22 pad 11: unconnected-(U22-WDI-Pad11) -> PC6
- U22 pad 3: unconnected-(U22-VCC-Pad3) -> VCC
- U23 pad 18: unconnected-(U23-Vcc-Pad18) -> VCC
- U23 pad 3: unconnected-(U23-A0-Pad3) -> BUS_A1
- U23 pad 7: unconnected-(U23-~{DTACK}-Pad7) -> Net-(U23-~{DTACK})
- U23 pad 8: unconnected-(U23-CLK-Pad8) -> CLK
- U24 pad 1: TS_A3 -> BUS_A1
- U24 pad 21: unconnected-(U24-IRQ-Pad21) -> Net-(U24-IRQ)
- U24 pad 27: unconnected-(U24-OP4-Pad27) -> Net-(RN6-R3)
- U24 pad 3: TS_A2 -> BUS_A2
- U24 pad 31: unconnected-(U24-RXDA-Pad31) -> RX
- U24 pad 4: unconnected-(U24-IP1-Pad4) -> TS1
- U24 pad 40: unconnected-(U24-VCC-Pad40) -> VCC
- U24 pad 5: TS_A1 -> BUS_A3
- U24 pad 6: TS_A0 -> BUS_A4
- U24 pad 7: unconnected-(U24-IP0-Pad7) -> TS0
- U25 pad 12: unconnected-(U25-VCC-Pad12) -> VCC
- U25 pad 36: unconnected-(U25-PC6/PIACK-Pad36) -> PC6
- U25 pad 40: unconnected-(U25-CLK-Pad40) -> CLK
- U25 pad 43: unconnected-(U25-R/W-Pad43) -> RW
- U26 pad 28: unconnected-(U26-V_{CC}-Pad28) -> VCC
- U27 pad 28: unconnected-(U27-V_{CC}-Pad28) -> VCC
- U28 pad 13: unconnected-(U28-~{BR}-Pad13) -> VCC
- U28 pad 14: Net-(U28-V_{CC}-Pad14) -> VCC
- U28 pad 23: unconnected-(U28-~{IPL2}-Pad23) -> IPL2
- U28 pad 24: unconnected-(U28-~{IPL1}-Pad24) -> IPL1
- U28 pad 25: unconnected-(U28-~{IPL0}-Pad25) -> IPL0
- U28 pad 49: Net-(U28-V_{CC}-Pad14) -> VCC
- U3 pad 6: unconnected-(U3-Pad6) -> TX
- U4 pad 4: unconnected-(U4-Pad4) -> Net-(U18-~{Y0})
- U5 pad 16: unconnected-(U5-V_{DD}-Pad16) -> VCC
- U6 pad 14: unconnected-(U6-VCC-Pad14) -> VCC
- U6 pad 7: unconnected-(U6-GND-Pad7) -> GND
- U7 pad 14: unconnected-(U7E-VCC-Pad14) -> VCC
- U8 pad 1: unconnected-(U8-A->B-Pad1) -> RW
- U8 pad 20: unconnected-(U8-VCC-Pad20) -> VCC
- U9 pad 1: unconnected-(U9-A->B-Pad1) -> VCC
- U9 pad 19: unconnected-(U9-CE-Pad19) -> GND
- U9 pad 20: unconnected-(U9-VCC-Pad20) -> VCC
Routing:
- net +24V: track 0.00 -> 523.6 mm
- net GND: track 574.7 -> 992.1 mm, vias 1 -> 7
- net VCC: track 0.00 -> 337.5 mm
- net unconnected-(U12-Q3-Pad9): track 68.5 -> 277.5 mm, vias 0 -> 1
- net CLK: track 203.7 -> 361.5 mm, vias 6 -> 7
- net D4: track 220.4 -> 369.1 mm, vias 5 -> 7
- net IPL0: track 0.00 -> 129.0 mm, vias 0 -> 2
- net unconnected-(U3-Pad6): track 128.4 -> 0.00 mm, vias 1 -> 0
- net TX: track 0.00 -> 128.4 mm, vias 0 -> 1
- net D1: track 252.8 -> 374.7 mm, vias 6 -> 7
- net D3: track 59.9 -> 181.1 mm, vias 3 -> 5
- net Net-(U21-CS1): track 0.00 -> 115.1 mm, vias 0 -> 4
- net Net-(U15A-~{Q}): track 0.00 -> 113.2 mm, vias 0 -> 2
- net D7: track 39.9 -> 143.7 mm, vias 2 -> 4
- net PC6: track 0.00 -> 103.1 mm
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Other:
- board text added: "4245/000101/M011"
