File: ZLKhalter/ZLKhalter.kicad_pcb (KiCad board)
At the start: 2 copper layers, 43.2 x 35.6 mm, 7 parts, among them J1 Conn_02x04_Counter_Clockwise, J2 Conn_01x04_Pin, J3 Conn_02x04_Counter_Clockwise, J4 Conn_02x03_Odd_Even, J6 Conn_02x03_Top_Bottom, J7 Conn_02x03_Top_Bottom

Commit message: einlagig
Parts:
- R1: footprint Resistor_SMD:R_0603_1608Metric_Pad0.98x0.95mm_HandSolder -> Resistor_SMD:R_0805_2012Metric_Pad1.20x1.40mm_HandSolder
- moved R1 2.89 mm to (142.3, 143.8)
Routing:
- net RST: track 55.2 -> 86.1 mm, vias 1 -> 0
- net SOD_MOSI: track 60.0 -> 76.6 mm
- net VCC: track 69.5 -> 84.2 mm
- net GND: track 77.8 -> 81.0 mm
- net +12V: track 19.2 -> 16.4 mm
- net SID_MISO: track 51.2 -> 52.7 mm, vias 1 -> 0
- net SCK: track 56.4 -> 55.0 mm, vias 1 -> 0
Other:
- outline, holes or cut-outs redrawn

Commit message: einseitig+led
Parts:
- added D1: LED, LED_SMD:LED_0805_2012Metric_Pad1.15x1.40mm_HandSolder, F.Cu at (147.3, 143.8)
- added D2: LED, LED_SMD:LED_0805_2012Metric_Pad1.15x1.40mm_HandSolder, F.Cu at (141.0, 148.2)
- added JP1: SolderJumper_3_Open, Jumper:SolderJumper-3_P1.3mm_Open_Pad1.0x1.5mm, F.Cu at (137.6, 140.3)
- added Q1: BSS138, Package_TO_SOT_SMD:SOT-23, F.Cu at (138.8, 150.5)
- added R2: 270, Resistor_SMD:R_0805_2012Metric_Pad1.20x1.40mm_HandSolder, F.Cu at (144.8, 143.8)
- added R3: 270, Resistor_SMD:R_0805_2012Metric_Pad1.20x1.40mm_HandSolder, F.Cu at (139.7, 143.8)
- moved J4 0.63 mm to (142.9, 134.6)
- moved R1 0.09 mm to (142.2, 143.8)
Routing:
- net GND: track 81.0 -> 98.6 mm
- net Net-(JP1-C): track 0.00 -> 9.24 mm
- net SOD_MOSI: track 76.6 -> 85.2 mm
- net VCC: track 84.2 -> 90.3 mm
- net Net-(D2-A): track 0.00 -> 2.92 mm
- net Net-(D1-A): track 0.00 -> 2.54 mm
- net Net-(D2-K): track 0.00 -> 1.80 mm
- net SID_MISO: track 52.7 -> 53.2 mm
