File: ZLKhalter/ZLKhalter.kicad_sch (KiCad schematic)
At the start: 7 parts, among them J1 Conn_02x04_Counter_Clockwise, J2 Conn_01x04_Pin, J3 Conn_02x04_Counter_Clockwise, J4 Conn_02x03_Odd_Even, J6 Conn_02x03_Top_Bottom, J7 Conn_02x03_Top_Bottom

Commit message: einlagig
Parts:
- R1: footprint Resistor_SMD:R_0603_1608Metric_Pad0.98x0.95mm_HandSolder -> Resistor_SMD:R_0805_2012Metric_Pad1.20x1.40mm_HandSolder
Changed lines of the file:
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@@
 			)
 		)
-		(property "Footprint" "Resistor_SMD:R_0603_1608Metric_Pad0.98x0.95mm_HandSolder"
+		(property "Footprint" "Resistor_SMD:R_0805_2012Metric_Pad1.20x1.40mm_HandSolder"
 			(at 127 52.578 90)
 			(hide yes)

Commit message: einseitig+led
Parts:
- added D1, D2: LED, LED_SMD:LED_0805_2012Metric_Pad1.15x1.40mm_HandSolder, symbol Device:LED
- added JP1: SolderJumper_3_Open, Jumper:SolderJumper-3_P1.3mm_Open_Pad1.0x1.5mm, symbol Jumper:SolderJumper_3_Open
- added Q1: BSS138, Package_TO_SOT_SMD:SOT-23, symbol Transistor_FET:BSS138
- added R2, R3: 270, Resistor_SMD:R_0805_2012Metric_Pad1.20x1.40mm_HandSolder, symbol Device:R
Connections:
- net GND: now also D1.1 (K), Q1.2 (S)
- net SID_MISO: now also JP1.1 (A)
- net SOD_MOSI: now also JP1.3 (B)
- net VCC: now also R2.1, R3.1
- new net: D2.1 (K), Q1.3 (D)
- new net: D2.2 (A), R3.2
- new net: D1.2 (A), R2.2
- new net: JP1.2 (C), Q1.1 (G)
