File: GSE14/GSE14.kicad_pcb (KiCad board)
At the start: 2 copper layers, 163 x 249 mm, 161 parts, among them IC5 7404, J1 Seriell, J13 Steckerleiste 13, J15 Steckerleiste 15, J16 Steckerleiste 16, J17 Steckerleiste 17, Q6 BC238B, Q7 BC328, Q8 BC238B, Q9 BF245A, SW1 Reset, SW2 NMI, T1 BDX 53 C, T2 BDX 53 C, T3 BDX 53 C, T4 BDX 53 C, T5 BD 675, U1 4093, U10 74C373/2, U11 74C373/3, U12 74LS123, U13 L7805, U14 4503, U2 74HO32, U3 4069, U4 74LS74, U6 74LS132, U7 74LS155, U8 74HC138, U9 74C373/1, Y1 4MHz

Commit message: pm1
Connections:
- C56 pad 1: /Auszahlung010 -> /Auszahlung1
- C58 pad 1: unconnected-(C58-Pad1) -> /Auszahlung5
- C58 pad 2: unconnected-(C58-Pad2) -> GND
- C60 pad 1: unconnected-(C60-Pad1) -> /Pegelschalter2
- C60 pad 2: unconnected-(C60-Pad2) -> GND
- C61 pad 1: unconnected-(C61-Pad1) -> /Pegelschalter5
- C61 pad 2: unconnected-(C61-Pad2) -> GND
- D8 pad 1: unconnected-(D8-K-Pad1) -> +12V
- EPROM1 pad 14: unconnected-(EPROM1-GND-Pad14) -> GND
- EPROM2 pad 14: unconnected-(EPROM2-GND-Pad14) -> GND
- PIO1 pad 37: ~{M1} -> ~{PM1}
- PIO2 pad 37: ~{M1} -> ~{PM1}
- U15 pad 10: unconnected-(U15-~{WR}-Pad10) -> ~{WR}
- U2 pad 2: unconnected-(U2-Pad2) -> Net-(U2-Pad2)
- U2 pad 3: unconnected-(U2-Pad3) -> Net-(U2-Pad3)
- U3 pad 1: unconnected-(U3-Pad1) -> ~{M1}
- U3 pad 10: unconnected-(U3-Pad10) -> ~{PM1}
- U3 pad 11: unconnected-(U3-Pad11) -> Net-(U2-Pad3)
- U3 pad 4: unconnected-(U3-Pad4) -> Net-(U2-Pad2)
Routing:
- net GND: track 1350.8 -> 1645.9 mm, vias 30 -> 33
- net ~{PM1}: track 0.00 -> 187.6 mm, vias 0 -> 3
- net ~{WR}: track 22.4 -> 166.9 mm, vias 2 -> 3
- net VCC: track 914.2 -> 1056.2 mm, vias 14 -> 15
- net ~{RES}: track 141.1 -> 257.9 mm
- net unconnected-(U15-~{WR}-Pad10): track 104.6 -> 0.00 mm, vias 1 -> 0
- net Net-(PIO2-PA6): track 205.0 -> 292.1 mm
- net ~{M1}: track 234.0 -> 151.4 mm, vias 5 -> 4
- net D1: track 297.0 -> 370.3 mm
- net unconnected-(U16-Z-Pad10): track 146.4 -> 218.3 mm
- net ~{IORQ}: track 136.1 -> 200.2 mm
- net ~{RD}: track 253.2 -> 311.4 mm
- net A1: track 204.1 -> 258.2 mm
- net unconnected-(U3-Pad10): track 51.4 -> 0.00 mm, vias 2 -> 0
- net D0: track 339.5 -> 389.6 mm
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
Commit message: silkscreen
Parts:
- removed JP1, JP2: Jumper_3_Bridged12, Connector_PinHeader_2.54mm:PinHeader_1x03_P2.54mm_Vertical
- B1: value TestPoint_2Pole -> +5V
- B2: value TestPoint_2Pole -> GND
- U11: value 74C373/3 -> 74C373/1
- U15: value ~ -> 8251A
- U9: value 74C373/1 -> 74C373/3
- moved D7 13.2 mm to (191.0, 36.2), turned to -90 degrees
- moved D9 13.0 mm to (194.9, 36.3), turned to -90 degrees
- moved R14 12.6 mm to (187.3, 36.2), turned to -90 degrees
- moved D10 1.17 mm to (231.6, 39.4), turned to 90 degrees
- renumbered D9 to D7, D7 to D9
Connections:
- net Net-(RAM1-~{E}) renamed RAM_CS
- C49 pad 1: VCC -> VCCQ
- C55 pad 1: unconnected-(C55-Pad1) -> GND
- C55 pad 2: unconnected-(C55-Pad2) -> /Auszahlung010
- C62 pad 1: unconnected-(C62-Pad1) -> Net-(J16-Pin_27)
- C63 pad 1: unconnected-(C63-Pad1) -> Net-(J16-Pin_25)
- C64 pad 1: unconnected-(C64-Pad1) -> Net-(J16-Pin_23)
- C65 pad 1: unconnected-(C65-Pad1) -> /SynchronRechts
- C66 pad 1: unconnected-(C66-Pad1) -> /SynchronMitte
- C67 pad 1: unconnected-(C67-Pad1) -> /SynchronLinks
- C68 pad 1: unconnected-(C68-Pad1) -> /MotorlogikClear
- C69 pad 1: unconnected-(C69-Pad1) -> /Motorstromumschaltung
- C70 pad 1: unconnected-(C70-Pad1) -> /RueckgabeTaste
- CPU1 pad 18: Net-(CPU1-~{HALT}) -> unconnected-(CPU1-~{HALT}-Pad18)
- CPU1 pad 25: unconnected-(CPU1-~{BUSREQ}-Pad25) -> Net-(CPU1-~{BUSREQ})
- D10 pad 1: Net-(D10-K) -> GND
- D10 pad 2: VCC -> Net-(D10-A)
- D4 pad 2: unconnected-(D4-A-Pad2) -> Net-(D4-A)
- EPROM1 pad 20: Net-(EPROM1-~{CE}) -> ROM1_CS
- EPROM1 pad 26: unconnected-(EPROM1-NC-Pad26) -> VCC
- EPROM2 pad 20: Net-(EPROM2-~{CE}) -> ROM2_CS
- IC5 pad 13: Net-(IC5-Pad13) -> RES
- J1 pad 10: Net-(J1-Pin_10) -> GND
- J1 pad 4: unconnected-(J1-Pin_4-Pad4) -> Net-(J1-Pin_4)
- J1 pad 5: unconnected-(J1-Pin_5-Pad5) -> SERIAL_CLOCK
- J1 pad 6: Net-(J1-Pin_10) -> GND
- J1 pad 8: Net-(J1-Pin_10) -> GND
- J16 pad 1: GND -> /MotorimpulseLinks
- J16 pad 10: /SynchronRechts -> Net-(J16-Pin_10)
- J16 pad 11: /SynchronMitte -> /RueckgabeTaste
- J16 pad 12: /SynchronMitte -> /RueckgabeTaste
- J16 pad 13: /SynchronLinks -> /Motorstromumschaltung
- J16 pad 14: /SynchronLinks -> /Motorstromumschaltung
- J16 pad 17: /Motorstromumschaltung -> /SynchronLinks
- J16 pad 18: /Motorstromumschaltung -> /SynchronLinks
- J16 pad 19: /RueckgabeTaste -> /SynchronMitte
- J16 pad 2: GND -> /MotorimpulseLinks
- J16 pad 20: /RueckgabeTaste -> /SynchronMitte
- J16 pad 21: Net-(J16-Pin_21) -> /SynchronRechts
- J16 pad 22: Net-(J16-Pin_21) -> /SynchronRechts
- J16 pad 25: /MotorimpulseMitte -> Net-(J16-Pin_25)
- J16 pad 26: /MotorimpulseMitte -> Net-(J16-Pin_25)
- J16 pad 27: /MotorimpulseRechts -> Net-(J16-Pin_27)
- J16 pad 28: /MotorimpulseRechts -> Net-(J16-Pin_27)
- J16 pad 29: /MotorimpulseLinks -> GND
- J16 pad 3: Net-(J16-Pin_3) -> /MotorimpulseRechts
- J16 pad 30: /MotorimpulseLinks -> GND
- J16 pad 4: Net-(J16-Pin_3) -> /MotorimpulseRechts
- J16 pad 5: Net-(J16-Pin_5) -> /MotorimpulseMitte
- J16 pad 6: Net-(J16-Pin_5) -> /MotorimpulseMitte
- J16 pad 9: /SynchronRechts -> Net-(J16-Pin_10)
- PIO2 pad 27: Net-(J16-Pin_3) -> Net-(J16-Pin_27)
- PIO2 pad 28: Net-(J16-Pin_5) -> Net-(J16-Pin_25)
- PIO2 pad 29: Net-(J16-Pin_7) -> Net-(J16-Pin_23)
- Q6 pad 2: Net-(PIO2-PA0) -> Net-(Q6-B)
- Q6 pad 3: Net-(D10-K) -> Net-(D10-A)
- Q8 pad 2: unconnected-(Q8-B-Pad2) -> Net-(Q8-B)
- Q8 pad 3: unconnected-(Q8-C-Pad3) -> GND
- R19 pad 2: Net-(CPU1-~{HALT}) -> Net-(CPU1-~{BUSREQ})
- R2 pad 1: unconnected-(R2-Pad1) -> Net-(D4-A)
- R22 pad 2: unconnected-(R22-Pad2) -> Net-(Q6-B)
- R24 pad 1: Net-(PIO1-PB1) -> Net-(T2-B)
- R24 pad 2: Net-(T2-B) -> Net-(PIO1-PB1)
- R4 pad 1: unconnected-(R4-Pad1) -> Net-(Q8-B)
- R7 pad 1: unconnected-(R7-Pad1) -> Net-(D4-A)
- U1 pad 13: unconnected-(U1-Pad13) -> Net-(PIO2-PA0)
- U1 pad 14: VCC -> VCCQ
- U11 pad 1: GND -> Net-(U11-OE)
- U11 pad 11: Net-(U11-LE) -> VCC
- U11 pad 13: /EXT_A4 -> /D_I4
- U11 pad 14: /EXT_A5 -> /D_I5
- U11 pad 17: /EXT_A6 -> /D_I6
- U11 pad 18: /EXT_A7 -> /D_I7
- U11 pad 3: /EXT_A0 -> /D_I0
- U11 pad 4: /EXT_A1 -> /D_I1
- U11 pad 7: /EXT_A2 -> /D_I2
- U11 pad 8: /EXT_A3 -> /D_I3
- U12 pad 1: unconnected-(U12A-A-Pad1) -> Net-(U12A-A)
- U12 pad 5: unconnected-(U12B-Q-Pad5) -> Net-(U12A-A)
- U14 pad 12: Net-(J16-Pin_23) -> Net-(J16-Pin_7)
- U14 pad 7: Net-(J16-Pin_21) -> Net-(J16-Pin_10)
- U15 pad 11: unconnected-(U15-~{CS}-Pad11) -> UART_CS
- U15 pad 12: unconnected-(U15-C/~{D}-Pad12) -> A0
- U15 pad 21: unconnected-(U15-RESET-Pad21) -> RES
- U15 pad 22: unconnected-(U15-~{DSR}-Pad22) -> Net-(J1-Pin_4)
- U15 pad 25: Net-(U15-~{RxC}) -> SERIAL_CLOCK
- U15 pad 9: Net-(U15-~{RxC}) -> SERIAL_CLOCK
- U16 pad 10: unconnected-(U16-Z-Pad10) -> SERIAL_CLOCK
- U2 pad 11: Net-(U9-LE) -> Net-(U11-OE)
- U3 pad 6: Net-(U11-LE) -> Net-(U9-LE)
- U4 pad 4: unconnected-(U4A-~{S}-Pad4) -> VCC
- U6 pad 10: Net-(IC5-Pad13) -> RES
- U6 pad 11: Net-(IC5-Pad13) -> RES
- U7 pad 10: Net-(EPROM1-~{CE}) -> ROM2_CS
- U7 pad 13: Net-(JP2-C) -> A13
- U7 pad 3: Net-(JP1-C) -> A14
- U7 pad 9: Net-(EPROM2-~{CE}) -> ROM1_CS
- U8 pad 16: unconnected-(U8-VCC-Pad16) -> VCC
- U8 pad 7: unconnected-(U8-~{Y7}-Pad7) -> UART_CS
- U9 pad 12: /D_I4 -> /EXT_A4
- U9 pad 15: /D_I5 -> /EXT_A5
- U9 pad 16: /D_I6 -> /EXT_A6
- U9 pad 19: /D_I7 -> /EXT_A7
- U9 pad 2: /D_I0 -> /EXT_A0
- U9 pad 5: /D_I1 -> /EXT_A1
- U9 pad 6: /D_I2 -> /EXT_A2
- U9 pad 9: /D_I3 -> /EXT_A3
Routing:
- net GND: track 1645.9 -> 2024.2 mm, vias 33 -> 40
- net SERIAL_CLOCK: track 0.00 -> 370.3 mm, vias 0 -> 4
- net RES: track 0.00 -> 327.0 mm, vias 0 -> 5
- net VCC: track 1056.2 -> 1299.9 mm, vias 15 -> 14
- net unconnected-(U16-Z-Pad10): track 218.3 -> 0.00 mm, vias 1 -> 0
- net Net-(U11-OE): track 0.00 -> 199.0 mm, vias 0 -> 2
- net /RueckgabeTaste: track 0.00 -> 173.5 mm, vias 0 -> 4
- net unconnected-(U15-RESET-Pad21): track 165.2 -> 0.00 mm, vias 3 -> 0
- net D7: track 250.4 -> 411.6 mm, vias 3 -> 5
- net Net-(PIO2-PA0): track 0.00 -> 159.7 mm, vias 0 -> 2
- net Net-(J1-Pin_4): track 0.00 -> 158.6 mm, vias 0 -> 1
- net Net-(U9-LE): track 0.00 -> 155.6 mm, vias 0 -> 1
- net Net-(IC5-Pad13): track 153.8 -> 0.00 mm, vias 2 -> 0
- net UART_CS: track 0.00 -> 142.7 mm, vias 0 -> 2
- net Net-(D4-A): track 0.00 -> 137.4 mm
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
Commit message: dicker
Parts:
- added AE1: Antenna, TestPoint:TestPoint_Bridge_Pitch6.35mm_Drill1.3mm, F.Cu at (122.7, 31.8)
- added AE2: Antenna, TestPoint:TestPoint_Bridge_Pitch6.35mm_Drill1.3mm, F.Cu at (255.9, 31.5)
- added J2: Conn_01x04, Connector_PinHeader_2.54mm:PinHeader_2x04_P2.54mm_Vertical, F.Cu at (222.9, 88.9)
- Q1: renamed from Y1; value 4MHz -> 4M
- RAM1: value MB8416-20L -> 6116
- U11: value 74C373/1 -> 74C373/3
- U16: value ~ -> HD-4702
- U9: value 74C373/3 -> 74C373/1
- moved TA1 1.69 mm to (218.4, 38.5)
- moved R40 1.52 mm to (215.3, 51.3)
- moved C51 1.43 mm to (178.2, 73.5)
- moved C71 1.31 mm to (212.5, 38.0)
- moved R32 1.24 mm to (179.3, 84.2)
- moved C72 1.09 mm to (212.2, 45.5)
- moved R20 1.03 mm to (240.0, 61.5)
- moved R41 0.77 mm to (215.3, 55.5)
- moved R31 0.76 mm to (215.3, 59.2)
- moved J17 0.63 mm to (114.3, 231.1)
- moved C3 0.53 mm to (247.7, 226.7)
- moved R26 0.49 mm to (142.2, 112.4)
- moved T2 0.48 mm to (141.6, 120.7)
- moved C1 0.44 mm to (212.1, 234.3)
- moved D8 0.44 mm to (232.4, 220.3)
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- renumbered U1 to IC1, U2 to IC2, U3 to IC3, SW1 to TA1, SW2 to TA2
Connections:
- net Net-(J1-Pin_2) renamed ~{DTR}
- net Net-(J1-Pin_4) renamed ~{DSR}
- net VCCQ renamed VCMOS
- C51 pad 1: unconnected-(C51-Pad1) -> Net-(C51-Pad1)
- C51 pad 2: unconnected-(C51-Pad2) -> GND
- IC1 pad 8: Net-(R11-Pad1) -> Net-(C51-Pad1)
- IC1 pad 9: Net-(R11-Pad1) -> Net-(C51-Pad1)
- IC5 pad 3: Net-(U4B-Q) -> Net-(U4A-C)
- J1 pad 1: unconnected-(J1-Pin_1-Pad1) -> ~{CTS}
- J1 pad 3: unconnected-(J1-Pin_3-Pad3) -> ~{RTS}
- J1 pad 7: unconnected-(J1-Pin_7-Pad7) -> RxD
- J1 pad 9: unconnected-(J1-Pin_9-Pad9) -> TxD
- PIO2 pad 14: unconnected-(PIO2-PA1-Pad14) -> RxRDY
- R11 pad 1: Net-(R11-Pad1) -> Net-(C51-Pad1)
- R12 pad 2: Net-(R11-Pad1) -> Net-(C51-Pad1)
- R28 pad 2: unconnected-(R28-Pad2) -> /Pegelschalter2
- R29 pad 2: unconnected-(R29-Pad2) -> /Pegelschalter5
- U15 pad 14: unconnected-(U15-RxRDY-Pad14) -> RxRDY
- U15 pad 17: unconnected-(U15-~{CTS}-Pad17) -> ~{CTS}
- U15 pad 19: unconnected-(U15-TxD-Pad19) -> TxD
- U15 pad 23: unconnected-(U15-~{RTS}-Pad23) -> ~{RTS}
- U15 pad 3: unconnected-(U15-RxD-Pad3) -> RxD
- U16 pad 11: unconnected-(U16-S3-Pad11) -> Net-(J2-Pin_7)
- U16 pad 12: unconnected-(U16-S2-Pad12) -> Net-(J2-Pin_5)
- U16 pad 13: unconnected-(U16-S1-Pad13) -> Net-(J2-Pin_3)
- U16 pad 14: unconnected-(U16-S0-Pad14) -> Net-(J2-Pin_1)
- U4 pad 1: unconnected-(U4A-~{R}-Pad1) -> VCC
- U4 pad 3: unconnected-(U4A-C-Pad3) -> Net-(U4A-C)
- U4 pad 9: Net-(U4B-Q) -> Net-(U4A-C)
Routing:
- net ~{CTS}: track 0.00 -> 208.5 mm
- net Net-(C51-Pad1): track 0.00 -> 202.5 mm, vias 0 -> 4
- net ~{RTS}: track 0.00 -> 188.6 mm, vias 0 -> 1
- net RxD: track 0.00 -> 173.5 mm, vias 0 -> 1
- net TxD: track 0.00 -> 171.9 mm, vias 0 -> 3
- net Net-(R11-Pad1): track 160.1 -> 0.00 mm, vias 4 -> 0
- net unconnected-(J1-Pin_7-Pad7): track 149.7 -> 0.00 mm, vias 1 -> 0
- net unconnected-(J1-Pin_9-Pad9): track 126.7 -> 0.00 mm, vias 2 -> 0
- net RxRDY: track 0.00 -> 84.5 mm, vias 0 -> 1
- net Net-(AE1-A): track 110.7 -> 180.3 mm, vias 1 -> 0
- net unconnected-(U15-RxRDY-Pad14): track 68.6 -> 0.00 mm, vias 1 -> 0
- net GND: track 2024.2 -> 1966.6 mm, vias 40 -> 76
- net Net-(U4A-C): track 0.00 -> 44.7 mm
- net Net-(U4B-Q): track 42.7 -> 0.00 mm
- net unconnected-(U15-~{CTS}-Pad17): track 40.8 -> 0.00 mm
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- added copper zone on F.Cu, net GND
Other:
- board text added: "82 007"
- board text added: "GSD-1.4"
